File: LoRa_Board.kicad_sch (KiCad schematic)
At the start: 97 parts, among them J1 Conn_01x08_Pin, J11 Power Select Jumpers, J13 USART1 Connector, J14 LPUART1 Connector, J15 Power Select Jumpers, J16 USB_B_Micro, J17 BOOT0_Jumper, J19 SMA PCB END LAUNCH JACK ROUND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, J2 Speaker Board Header, J3 Debug_Pins, J4 Conn_01x08, J5 User Button Jumper, J6 Power Pins, J7 GPIO_Pins, J8 Power Pins, J9 LCD_I2C3_Connector, U1 STM32WL55CCU6, U3 USBLC6-2SC6, U5 BGS12WN6E6327, U7 FT230XS, Y1 Clock_ECS-327MVATX-7-CN-TR, Y3 ABM3B-32.000MHZ-8-R30-B1U-T

Commit message: Update
Parts:
- removed C2: 100n, symbol Device:C
- removed C4, C6: 330p, symbol Device:C
- removed J1: Conn_01x08_Pin, symbol Connector:Conn_01x08_Pin
- removed J13: USART1 Connector, Connector_PinHeader_2.54mm:PinHeader_1x04_P2.54mm_Vertical, symbol Connector:Conn_01x04_Pin
- removed J14: LPUART1 Connector, Connector_PinHeader_2.54mm:PinHeader_1x04_P2.54mm_Vertical, symbol Connector:Conn_01x04_Pin
- removed J2: Speaker Board Header, symbol Connector:Conn_01x05_Socket
- removed J4: Conn_01x08, symbol Connector_Generic:Conn_01x08
- removed J7: GPIO_Pins, symbol Connector:Conn_01x15_Pin
- removed J8: Power Pins, symbol Connector_Generic:Conn_01x04
- removed J9: LCD_I2C3_Connector, Connector_PinHeader_2.54mm:PinHeader_1x04_P2.54mm_Vertical, symbol Connector:Conn_01x04_Pin
- removed R3, R4, R5, R6: 100R, Resistor_SMD:R_0805_2012Metric_Pad1.20x1.40mm_HandSolder, symbol Device:R
- added BH1: Battery_Holder_1060TR, Personal_Project:Battery_Holder_1060TR, symbol Personal_Projects:Battery_Holder_1060TR
- added C19: 100n, Capacitor_SMD:C_0603_1608Metric_Pad1.08x0.95mm_HandSolder, symbol Device:C
- added J10: SPI1_Headers, symbol Connector_Generic:Conn_01x06
- added J2: LPUART1_Headers, symbol Connector_Generic:Conn_01x04
- added J4: Coin Battery Jumper, Connector_PinHeader_2.54mm:PinHeader_1x03_P2.54mm_Vertical, symbol Connector_Generic:Conn_01x03
- added J8: Pin_Headers, symbol Connector_Generic:Conn_02x05_Odd_Even
- added J9: I2C1_Headers, symbol Connector_Generic:Conn_01x04
- added R12, R13, R14, R15, R16, R17, R18, R19: 100R, Resistor_SMD:R_0805_2012Metric_Pad1.20x1.40mm_HandSolder, symbol Device:R
- U2, U6: footprint (none) -> Personal_Project:Button_KMR231GLFS
Connections:
- net PA12_SPI1_MOSI is gone; now on net PA12_USART1_RTS: U1.35 (PA12)
- net PA15_SPI1_NSS is gone; now on net PA15: U1.43 (PA15)
- net PA1_USART2_RTS is gone; now on net PA11_USART1_CTS: U7.6 (~{CTS})
- net PA2_USART2_TX is gone; now on net PA10_USART1_RX: U7.4 (RXD)
- net PA3_USART2_RX is gone; now on net PB6_USART1_TX: U7.1 (TXD)
- net PB6_I2C1_SCL is gone; now on net PB6_USART1_TX: U1.4 (PB6)
- net +3.3V: now also J10.1 (Pin_1), J2.1 (Pin_1), J4.1 (Pin_1), J9.1 (Pin_1); no longer U1.37 (VBAT)
- net GND: now also BH1.2 (-), C19.2, J10.2 (Pin_2), J2.2 (Pin_2), J9.2 (Pin_2)
- net PA0: now also J8.1 (Pin_1)
- net PA15: now also J8.6 (Pin_6)
- net PA1_SPI1_SCK: now also R16.1
- net PA2_LPUART1_TX: now also R12.1
- net PA3_LPUART1_RX: now also R13.1
- net PA5: now also J8.2 (Pin_2)
- net PA7: now also J8.3 (Pin_3)
- net PA8_MCO: now also J8.4 (Pin_4)
- net PA9: now also J8.5 (Pin_5)
- net PB0: now also J8.7 (Pin_7)
- net PB12: now also J8.10 (Pin_10)
- net PB2: now also J8.8 (Pin_8)
- net PB4: now also J8.9 (Pin_9)
- net PB7_I2C1_SDA: now also R14.1
- net PA0_USART2_CTS renamed PA12_USART1_RTS
- net PA10 renamed PA10_USART1_RX
- net PA11_SPI1_MISO renamed PA11_USART1_CTS
- net PA4 renamed PA4_SPI1_NSS
- net PA4_SPI1_NSS: now also R17.1
- net PA6 renamed PA6_SPI1_MISO
- net PA6_SPI1_MISO: now also R18.1
- net PB5 renamed PB5_SPI1_MOSI
- net PB5_SPI1_MOSI: now also R19.1
- net PB8 renamed PB8_I2C1_SCL
- net PB8_I2C1_SCL: now also R15.1
- new net: J10.3 (Pin_3), R16.2
- new net: J9.3 (Pin_3), R14.2
- new net: J10.6 (Pin_6), R19.2
- new net: J2.4 (Pin_4), R13.2
- new net: J2.3 (Pin_3), R12.2
- new net: BH1.1 (+), J4.3 (Pin_3)
- new net: J9.4 (Pin_4), R15.2
- new net: J10.4 (Pin_4), R17.2
- new net: J10.5 (Pin_5), R18.2
- new net VBAT: C19.1, J4.2 (Pin_2), U1.37 (VBAT)
- no-connect marks 9 -> 10
Other:
- note added: "EP is optional adhesive zone"
- note added: "Placed 100 Ohm resistors on the UART, SPI, andd I2C lines to reduce ringing. PA8 MCO is to be used during intial setup to choose HSE load capacitors Then it is meant to be used as button input Decided to use ESDALC6V1W5 as ESD protection Is not ideal but should work for both 3.3V and 5V pins and has low capacitance (Used by ST)"
- note removed: "Add ground"
- note removed: "DAC_OUT1 to PA10"
- note removed: "PA8 MCO is to be used during intial setup to choose HSE load capacitors Then it is meant to be used as button input Decided to use ESDALC6V1W5 as ESD protection Is not ideal but should work for both 3.3V and 5V pins and has low capacitance (Used by ST)"
- moved on the sheet: C1, C10, C11, C12, C13, C14, C15, C16, C17, C18, C3, C40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

Commit message: Update
Parts:
- removed C17: 33p_GJM0335C1E330JB01D_MURATA, symbol Device:C
- removed J8: Pin_Headers, symbol Connector_Generic:Conn_02x05_Odd_Even
- removed L4: 15u_MLZ2012M150W_TDK, Inductor_SMD:L_0805_2012Metric_Pad1.15x1.40mm_HandSolder, symbol Device:L
- added J1: Pin_Headers, Connector_PinHeader_2.54mm:PinHeader_2x06_P2.54mm_Vertical, symbol Connector_Generic:Conn_02x06_Odd_Even
- added L1: 15u_MLZ2012M150W_TDK, Inductor_SMD:L_0805_2012Metric_Pad1.15x1.40mm_HandSolder, symbol Device:L
- C1, C10, C11, C12, C13, C15, C3, C41, C42, C43, C46, C47, C48, C49, C5, C50, C53, C54, C55, C56, C57, C58, C59, C60, C61, C62, C63, C64, C65, C66, C67, C7, C8, C9, FB3: footprint (none) -> Capacitor_SMD:C_0805_2012Metric_Pad1.18x1.45mm_HandSolder
- C19: footprint Capacitor_SMD:C_0603_1608Metric_Pad1.08x0.95mm_HandSolder -> Capacitor_SMD:C_0805_2012Metric_Pad1.18x1.45mm_HandSolder
- C51: value 33p_GJM0335C1E330JB01D_MURATA -> 100n_FCC0402KRX7R7BB104; footprint (none) -> Capacitor_SMD:C_0805_2012Metric_Pad1.18x1.45mm_HandSolder
- FB1: value FCM1608KF-601T03TAI-TECH -> ILB1206ER700V_1206; footprint (none) -> Capacitor_SMD:C_1206_3216Metric_Pad1.33x1.80mm_HandSolder
- J10: footprint (none) -> Connector_PinHeader_2.54mm:PinHeader_1x06_P2.54mm_Vertical
- J2, J6, J9: footprint (none) -> Connector_PinHeader_2.54mm:PinHeader_1x04_P2.54mm_Vertical
- J5: footprint (none) -> Connector_PinHeader_2.54mm:PinHeader_1x02_P2.54mm_Vertical
- L10, L5, L6, L7, L8, L9: footprint (none) -> Inductor_SMD:L_0603_1608Metric_Pad1.05x0.95mm_HandSolder
- R1, R10, R11, R9: footprint (none) -> Resistor_SMD:R_0805_2012Metric_Pad1.20x1.40mm_HandSolder
Connections:
- net VDDRF1V55 is gone; now on net VFBSMPS: C53.1, U1.29 (VDDRF1V55)
- net GND: now also J1.12 (Pin_12)
- net PA0: now also J1.1 (Pin_1)
- net PA15: now also J1.6 (Pin_6)
- net PA5: now also J1.2 (Pin_2)
- net PA7: now also J1.3 (Pin_3)
- net PA8_MCO: now also J1.4 (Pin_4)
- net PA9: now also J1.5 (Pin_5)
- net PB0: now also J1.7 (Pin_7)
- net PB12: now also J1.10 (Pin_10)
- net PB2: now also J1.8 (Pin_8)
- net PB4: now also J1.9 (Pin_9)
- net PC15-OSC32_OUT: now also J1.11 (Pin_11)
- net USB_D+: now also U3.4 (I/O2); no longer U3.6 (I/O1)
- net USB_D-: now also U3.6 (I/O1); no longer U3.4 (I/O2)
- net USB_D2+: now also U3.3 (I/O2); no longer U3.1 (I/O1)
- net USB_D2-: now also U3.1 (I/O1); no longer U3.3 (I/O2)
- net VFBSMPS: now also L1.1
- net VLXSMPS: now also L1.2
- net MCO_OSC_IN (ST_LINK) renamed PH0-OSC_IN
- no-connect marks 10 -> 9
Other:
- note added: "70R@100MHz"
- note added: "FCM1608KF-601T03TAI-TECH"
- note added: "Place near VDDPA pin"
- note added: "Placed 100 Ohm resistors on the UART, SPI, andd I2C lines to reduce ringing. PA8 MCO is to be used during intial setup to choose HSE load capacitors Then it is meant to be used as button input Decided to use ESDALC6V1W5 as ESD protection Is not ideal but should work for both 3.3V and 5V pins and has low capacitance (Used by ST) VDDPA Supply Input supply for PA regulator Transmit high output power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"
- note added: "Regulated PA supply output"
- note added: "VDDPA Supply Input supply for PA regulator"
- note removed: "600R@100MHz"
- note removed: "Placed 100 Ohm resistors on the UART, SPI, andd I2C lines to reduce ringing. PA8 MCO is to be used during intial setup to choose HSE load capacitors Then it is meant to be used as button input Decided to use ESDALC6V1W5 as ESD protection Is not ideal but should work for both 3.3V and 5V pins and has low capacitance (Used by ST)"
- moved on the sheet: C51, U3

Commit message: Update
Parts:
- added C17: 1uF, Capacitor_SMD:C_0805_2012Metric_Pad1.18x1.45mm_HandSolder, symbol Device:C
- added C2, C20, C21, C22, C27, C28: 100n, Capacitor_SMD:C_0805_2012Metric_Pad1.18x1.45mm_HandSolder, symbol Device:C
- added C23, C26, C4: 4u7, Capacitor_SMD:C_0805_2012Metric_Pad1.18x1.45mm_HandSolder, symbol Device:C
- added C24: 33p_GJM0335C1E330JB01D_MURATA, Capacitor_SMD:C_0805_2012Metric_Pad1.18x1.45mm_HandSolder, symbol Device:C
- added C25: 100n_FCC0402KRX7R7BB104, Capacitor_SMD:C_0805_2012Metric_Pad1.18x1.45mm_HandSolder, symbol Device:C
- added C29, C30: 47p, Capacitor_SMD:C_0805_2012Metric_Pad1.18x1.45mm_HandSolder, symbol Device:C
- added C31: 10p, Capacitor_SMD:C_0805_2012Metric_Pad1.18x1.45mm_HandSolder, symbol Device:C
- added C6: 1u, Capacitor_SMD:C_0805_2012Metric_Pad1.18x1.45mm_HandSolder, symbol Device:C
- added FB2: ILB1206ER700V_1206, Capacitor_SMD:C_1206_3216Metric_Pad1.33x1.80mm_HandSolder, symbol Device:FerriteBead
- added FB4: Part # MI0805K601R-10, Capacitor_SMD:C_0805_2012Metric_Pad1.18x1.45mm_HandSolder, symbol Device:FerriteBead
- added J7: BOOT0_Jumper, Connector_PinHeader_2.54mm:PinHeader_1x03_P2.54mm_Vertical, symbol Connector:Conn_01x03_Pin
- added J8: USB_B_Micro, Connector_USB:USB_Micro-B_Molex-105017-0001, symbol Connector:USB_B_Micro
- added R3: 1k, Resistor_SMD:R_0805_2012Metric_Pad1.20x1.40mm_HandSolder, symbol Device:R
- added R4, R5: 27, Resistor_SMD:R_0805_2012Metric_Pad1.20x1.40mm_HandSolder, symbol Device:R
- added R6: 100k, Resistor_SMD:R_0805_2012Metric_Pad1.20x1.40mm_HandSolder, symbol Device:R
- added U4: ~, Personal_Project:Button_KMR231GLFS, symbol Personal_Projects:Button_KMR231GLFS
- added U8: FT230XS, Package_SO:SSOP-16_3.9x4.9mm_P0.635mm, symbol Interface_USB:FT230XS
- added U9: USBLC6-2SC6, Package_TO_SOT_SMD:SOT-23-6, symbol Power_Protection:USBLC6-2SC6
Connections:
- net +3.3V: now also C20.1, C21.1, C22.1, C23.1, C24.1, C25.1, C6.1, FB2.2, J7.1 (Pin_1)
- net +3.3VA: now also C2.1, C4.1, FB2.1
- net BOOT0J: now also J7.2 (Pin_2), R3.1
- net GND: now also C17.1, C2.2, C24.2, C25.2, C26.2, C27.2, C28.2, C29.2, C30.2, C31.2, C4.2, C6.2, J7.3 (Pin_3), J8.5 (GND), J8.6 (Shield), R6.1, U4.3, U4.4, U4.5 (GND), U8.13 (GND), U8.5 (GND), U9.2 (GND)
- net NRST: now also C17.2, U4.1, U4.2
- net PA10_USART1_RX: now also U8.4 (RXD)
- net PA11_USART1_CTS: now also U8.6 (~{CTS})
- net PA12_USART1_RTS: now also U8.2 (~{RTS})
- net PB6_USART1_TX: now also U8.1 (TXD)
- net USBDM: now also R10.2, R4.2, U8.9 (USBDM); no longer R11.2
- net USBDP: now also R11.2, R5.2, U8.8 (USBDP); no longer R10.2
- net USB_D+: now also C30.1, R4.1, U9.4 (I/O2)
- net USB_D-: now also C29.1, R5.1, U9.6 (I/O1)
- net USB_D2+: now also J8.3 (D+), U9.3 (I/O2)
- net USB_D2-: now also J8.2 (D-), U9.1 (I/O1)
- net VBUS_5V: now also C31.1, FB4.1, J8.1 (VBUS), U9.5 (VBUS)
- net VBUS_5V_FB: now also C26.1, C27.1, FB4.2, U8.12 (VCC)
- new net: C28.1, U8.10 (3V3OUT), U8.11 (~{RESET}), U8.3 (VCCIO)
- new net: C20.2, C21.2, C22.2, C23.2
- new net: J8.4 (ID), R6.2
- no-connect marks 9 -> 13
Other:
- moved on the sheet: C65, U7

Commit message: Update
Parts:
- removed C17: 1uF, Capacitor_SMD:C_0805_2012Metric_Pad1.18x1.45mm_HandSolder, symbol Device:C
- removed C2, C20, C21, C22, C27, C28: 100n, Capacitor_SMD:C_0805_2012Metric_Pad1.18x1.45mm_HandSolder, symbol Device:C
- removed C23, C26, C4: 4u7, Capacitor_SMD:C_0805_2012Metric_Pad1.18x1.45mm_HandSolder, symbol Device:C
- removed C24: 33p_GJM0335C1E330JB01D_MURATA, Capacitor_SMD:C_0805_2012Metric_Pad1.18x1.45mm_HandSolder, symbol Device:C
- removed C25: 100n_FCC0402KRX7R7BB104, Capacitor_SMD:C_0805_2012Metric_Pad1.18x1.45mm_HandSolder, symbol Device:C
- removed C29, C30: 47p, Capacitor_SMD:C_0805_2012Metric_Pad1.18x1.45mm_HandSolder, symbol Device:C
- removed C31: 10p, Capacitor_SMD:C_0805_2012Metric_Pad1.18x1.45mm_HandSolder, symbol Device:C
- removed C6: 1u, Capacitor_SMD:C_0805_2012Metric_Pad1.18x1.45mm_HandSolder, symbol Device:C
- removed FB2: ILB1206ER700V_1206, Capacitor_SMD:C_1206_3216Metric_Pad1.33x1.80mm_HandSolder, symbol Device:FerriteBead
- removed FB4: Part # MI0805K601R-10, Capacitor_SMD:C_0805_2012Metric_Pad1.18x1.45mm_HandSolder, symbol Device:FerriteBead
- removed J7: BOOT0_Jumper, Connector_PinHeader_2.54mm:PinHeader_1x03_P2.54mm_Vertical, symbol Connector:Conn_01x03_Pin
- removed J8: USB_B_Micro, Connector_USB:USB_Micro-B_Molex-105017-0001, symbol Connector:USB_B_Micro
- removed R3: 1k, Resistor_SMD:R_0805_2012Metric_Pad1.20x1.40mm_HandSolder, symbol Device:R
- removed R4, R5: 27, Resistor_SMD:R_0805_2012Metric_Pad1.20x1.40mm_HandSolder, symbol Device:R
- removed R6: 100k, Resistor_SMD:R_0805_2012Metric_Pad1.20x1.40mm_HandSolder, symbol Device:R
- removed U4: ~, Personal_Project:Button_KMR231GLFS, symbol Personal_Projects:Button_KMR231GLFS
- removed U8: FT230XS, Package_SO:SSOP-16_3.9x4.9mm_P0.635mm, symbol Interface_USB:FT230XS
- removed U9: USBLC6-2SC6, Package_TO_SOT_SMD:SOT-23-6, symbol Power_Protection:USBLC6-2SC6
Connections:
- no-connect marks 13 -> 9
Other:
- moved on the sheet: C14, C16, C3, C63, C64, C65, C66, C67, C9, ESD1, ESD2, FB3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

Commit message: Update
Parts:
- FB1: value ILB1206ER700V_1206 -> BLM21PG601SN1D_0805; footprint Capacitor_SMD:C_1206_3216Metric_Pad1.33x1.80mm_HandSolder -> Capacitor_SMD:C_0805_2012Metric_Pad1.18x1.45mm_HandSolder
Changed lines of the file:
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@@
 	)
 	(symbol
-		(lib_id "Device:FerriteBead")
-		(at 193.04 87.63 90)
-		(unit 1)
-		(exclude_from_sim no)
-		(in_bom yes)
-		(on_board yes)
-		(dnp no)
-		(fields_autoplaced yes)
-		(property "Reference" "FB1"
-			(at 192.9892 80.01 90)
-			(effects
-				(font
-					(size 1.27 1.27)
-				)
-			)
-		)
-		(property "Value" "ILB1206ER700V_1206"
-			(at 192.9892 82.55 90)
-			(effects
-				(font
-					(size 1.27 1.27)
-				)
-			)
-		)
-		(property "Footprint" "Capacitor_SMD:C_1206_3216Metric_Pad1.33x1.80mm_HandSolder"
-			(at 193.04 89.408 90)
-			(effects
-				(font
-					(size 1.27 1.27)
-				)
-				(hide yes)
-			)
-		)
-		(property "Datasheet" "~"
-			(at 193.04 87.63 0)
-			(effects
-				(font
-					(size 1.27 1.27)
-				)
-				(hide yes)
-			)
-		)
-		(property "Description" "Ferrite bead"
-			(at 193.04 87.63 0)
-			(effects
-				(font
-					(size 1.27 1.27)
-				)
-				(hide yes)
-			)
-		)
-		(pin "1"
-		)
-		(pin "2"
-		)
-		(instances
-			(project "LoRa_Board"
-				(path "/34ccaf76-212c-4f8e-9afa-bb7eea5015e3"
-					(reference "FB1")
-					(unit 1)
-				)
-			)
-		)
-	)
-	(symbol
 		(lib_id "Device:C")
 		(at 132.08 55.88 0)
@@
 					(unit 1)
 				)
+			)
+		)
+	)
+	(symbol
+		(lib_id "Device:FerriteBead")
+		(at 193.04 87.63 90)
+		(unit 1)
+		(exclude_from_sim no)
+		(in_bom yes)
+		(on_board yes)
+		(dnp no)
+		(property "Reference" "FB1"
+			(at 188.976 85.852 90)
+			(effects
+				(font
+					(size 1.27 1.27)
+				)
+			)
+		)
+		(property "Value" "BLM21PG601SN1D_0805"
+			(at 197.104 91.694 90)
+			(effects
+				(font
+					(size 1.27 1.27)
+				)
+			)
+		)
+		(property "Footprint" "Capacitor_SMD:C_0805_2012Metric_Pad1.18x1.45mm_HandSolder"
+			(at 193.04 89.408 90)
+			(effects
+				(font
+					(size 1.27 1.27)
+				)
+				(hide yes)
+			)
+		)
+		(property "Datasheet" "~"
+			(at 193.04 87.63 0)
+			(effects
+				(font
+					(size 1.27 1.27)
+				)
+				(hide yes)
+			)
+		)
+		(property "Description" "Ferrite bead"
+			(at 193.04 87.63 0)
+			(effects
+				(font
+					(size 1.27 1.27)
+				)
+				(hide yes)
+			)
+		)
+		(pin "1"
+		)
+		(pin "2"
+		)
+		(instances
+			(project "LoRa_Board"
+				(path "/34ccaf76-212c-4f8e-9afa-bb7eea5015e3"
+					(reference "FB1")
+					(unit 1)
+				)

Commit message: Update
Parts:
- removed C56: 10p, Capacitor_SMD:C_0805_2012Metric_Pad1.18x1.45mm_HandSolder, symbol Device:C
- removed C57: 1n, Capacitor_SMD:C_0805_2012Metric_Pad1.18x1.45mm_HandSolder, symbol Device:C
- removed J1: Pin_Headers, Connector_PinHeader_2.54mm:PinHeader_2x06_P2.54mm_Vertical, symbol Connector_Generic:Conn_02x06_Odd_Even
- removed L8: 51n_LQW18AN51NG0Z, Inductor_SMD:L_0603_1608Metric_Pad1.05x0.95mm_HandSolder, symbol Device:L
- removed R1, R9: 100R, Resistor_SMD:R_0805_2012Metric_Pad1.20x1.40mm_HandSolder, symbol Device:R
- removed U5: BGS12WN6E6327, Package_LGA:Infineon_PG-TSNP-6-10_0.7x1.1mm_0.7x1.1mm_P0.4mm, symbol RF_Switch:BGS12WN6E6327
- added C2, C38: 220p_GRM1555C2A221GE01, Capacitor_SMD:C_0805_2012Metric, symbol Device:C
- added C33: 47n_Murata_GCM155R71E473KA55, Capacitor_SMD:C_0805_2012Metric, symbol Device:C
- added C34: 68p_Murata_GCM1555C1H680JA16, Capacitor_SMD:C_0805_2012Metric, symbol Device:C
- added C35, C39: 18p_GJM1555C1H180FB01, Capacitor_SMD:C_0805_2012Metric, symbol Device:C
- added C36: 20p_GJM1555C1H200GB01, Capacitor_SMD:C_0805_2012Metric, symbol Device:C
- added C37: 30p_GJM1555C1H300FB01, Capacitor_SMD:C_0805_2012Metric, symbol Device:C
- added C52, C68: 10p, Capacitor_SMD:C_0805_2012Metric, symbol Device:C
- added C69: 1n, Capacitor_SMD:C_0805_2012Metric, symbol Device:C
- added IC1: RF_Switch_PE42440MLBB-Z, Personal_Project:PE42440_QFN50P300X300X80-17N, symbol Personal_Projects:RF_Switch_PE42440MLBB-Z
- added J8: Conn_02x05_Odd_Even, Connector_PinHeader_2.54mm:PinHeader_2x05_P2.54mm_Vertical, symbol Connector_Generic:Conn_02x05_Odd_Even
- added L14: 6n8_LQW18AN6N8C00, Inductor_SMD:L_0603_1608Metric_Pad1.05x0.95mm_HandSolder, symbol Device:L
- added L15: 160n_LQW18ANR16G00, Inductor_SMD:L_0603_1608Metric_Pad1.05x0.95mm_HandSolder, symbol Device:L
- added L16: 12n_LQW18AN12NG0Z, Inductor_SMD:L_0603_1608Metric_Pad1.05x0.95mm_HandSolder, symbol Device:L
- added L17, L2: 51n_LQW18AN51NG0Z, Inductor_SMD:L_0603_1608Metric_Pad1.05x0.95mm_HandSolder, symbol Device:L
- added L18: 47n_LQW15AN47NJ00, Inductor_SMD:L_0603_1608Metric_Pad1.05x0.95mm_HandSolder, symbol Device:L
- added R20, R5, R6: 100R, Resistor_SMD:R_0805_2012Metric, symbol Device:R
- added SW1, SW2: Switch_NX3L1T3157GM,115, Personal_Project:Switch_NX3L1T3157GM115, symbol Personal_Projects:Switch_NX3L1T3157GM,115
- C1, C10, C11, C12, C13, C14, C15, C16, C18, C19, C3, C40, C41, C42, C43, C46, C47, C48, C5, C50, C51, C53, C58, C59, C60, C61, C62, C63, C64, C65, C66, C67, C7, C8, C9, FB1, FB3: footprint Capacitor_SMD:C_0805_2012Metric_Pad1.18x1.45mm_HandSolder -> Capacitor_SMD:C_0805_2012Metric
- C44: value 47n -> 33p_CC0402GRNPO9BN330; footprint Capacitor_SMD:C_0805_2012Metric_Pad1.18x1.45mm_HandSolder -> Capacitor_SMD:C_0805_2012Metric
- C45: value 68p -> 1n; footprint Capacitor_SMD:C_0805_2012Metric_Pad1.18x1.45mm_HandSolder -> Capacitor_SMD:C_0805_2012Metric
- C49: value 220p_GRM1555C2A221GE01 -> 33p_CC0402GRNPO9BN330; footprint Capacitor_SMD:C_0805_2012Metric_Pad1.18x1.45mm_HandSolder -> Capacitor_SMD:C_0805_2012Metric
- C54: value 10p -> 1n; footprint Capacitor_SMD:C_0805_2012Metric_Pad1.18x1.45mm_HandSolder -> Capacitor_SMD:C_0805_2012Metric
- C55: value 1n -> 10p; footprint Capacitor_SMD:C_0805_2012Metric_Pad1.18x1.45mm_HandSolder -> Capacitor_SMD:C_0805_2012Metric
- L6: value 160n_LQW18ANR16G00 -> 33n_LQW15AN33NG00
- R10, R11, R12, R13, R14, R15, R16, R17, R18, R19, R2, R7, R8: footprint Resistor_SMD:R_0805_2012Metric_Pad1.20x1.40mm_HandSolder -> Resistor_SMD:R_0805_2012Metric
Connections:
- net +3.3V: now also R5.1, SW1.5 (VCC), SW2.3 (Y0), SW2.5 (VCC); no longer U1.25 (VDDPA)
- net GND: now also C44.1, C49.1, C54.2, C55.2, C33.2, C34.2, C35.1, C37.1, C39.1, C52.2, C68.2, C69.2, IC1.1 (GND_1), IC1.10 (GND_5), IC1.12 (GND_6), IC1.14 (GND_7), IC1.17 (EP), IC1.5 (GND_2), IC1.7 (GND_3), IC1.9 (GND_4), SW1.2 (GND), SW2.2 (GND); no longer C44.2, C54.1, C55.1
- net PA0: now also J8.1 (Pin_1)
- net PA15: now also J8.6 (Pin_6)
- net PA5: now also J8.2 (Pin_2)
- net PA7: now also J8.3 (Pin_3)
- net PA8_MCO: now also J8.4 (Pin_4)
- net PA9: now also J8.5 (Pin_5)
- net PB12: now also J8.8 (Pin_8)
- net PB4: now also J5.2 (Pin_2), J8.7 (Pin_7)
- net PC13: now also J8.10 (Pin_10)
- net PC15-OSC32_OUT: now also J8.9 (Pin_9)
- net RF1: now also IC1.8 (RF3)
- net RF2_1: now also C39.2, IC1.6 (RF4), L17.2; no longer C49.2, C50.2
- net RF2_2: now also C38.2, L17.1; no longer C49.1
- net RF2_3: now also C36.2, C37.2, C38.1, L16.2; no longer C46.2, C48.2, L7.2
- net RF2_4: now also C35.2, C36.1, L14.2, L16.1, L18.1; no longer C46.1, C47.2, L5.2, L6.2, L7.1
- net RFIN: now also IC1.11 (RFC)
- net VDD: now also C45.1, C68.1, IC1.2 (VDD), R5.2; no longer C54.2, C55.2
- net VFBSMPS: now also SW2.1 (Y1)
- net VR_PA: now also C33.1, C34.1, L15.1; no longer C44.1, C45.1, L6.1
- net RFO_LP: now reaches U1.22 (RFO_LP)
- net RFO_LP: now also L14.1
- net PB0 renamed PB0_CTRL1
- net PB0_CTRL1: now also R20.1, SW1.6 (S), SW2.6 (S); no longer J5.2 (Pin_2)
- net PB2 renamed PB2_CTRL2
- net PB2_CTRL2: now also R6.1
- new net: L15.2, SW1.4 (Z)
- new net RF1_1: C50.2, IC1.13 (RF1), L2.2
- new net RF1_2: C2.2, L2.1
- new net RF1_3: C2.1, C46.2, C48.2, L7.2
- new net RF1_4: C46.1, C47.2, L5.2, L6.2, L7.1
- new net V1: C55.1, C69.1, IC1.4 (V1), R20.2
- new net V2: C52.1, C54.1, IC1.3 (V2), R6.2
- new net VDDPA: SW2.4 (Z), U1.25 (VDDPA)
- new net Y0: C44.2, L6.1, SW1.3 (Y0)
- new net Y1: C49.2, L18.2, SW1.1 (Y1)
Other:
- note added: "CTRL LOGIC CTRL1=LOW, CTRL2=LOW VDDPA=VDDSMPS, RF_HP, ANT=RF_HP CTRL1=HIGH, CTRL2=LOW VDDPA=FBSMPS, RF_LP, ANT=RFI (RF3) CTRL1=HIGH, CTRL2=HIGH VDDPA=FBSMPS, RF_LP, ANT=RF_LP(RF4)"
- note added: "STM32MP157FAD1 2x STM32WB55CGU6 2x STM32WB5MMGH6TR STM32MP135DAF7 STM32H7S7L8H6H STSPIN958TR STM32H7S3I8T6 LSM6DSV16XTR ISM330BXTR STM32WL55CCU6 STM32WL55JCI6 2x AGVLB.25B.07.0060A Connector: I-PEX MHF® I (U.FL Compatible) GW.52.A153 2.4/5.8/7.1GHZ Hinged RP-SMA (M) Connector TI.96.A113 900-940MHZ Connector: SMA(M)"
- note added: "VDDPA Power Amplifier voltage depends on the chosenn power transmission (HP or LP)"
- note removed: "Placed 100 Ohm resistors on the UART, SPI, andd I2C lines to reduce ringing. PA8 MCO is to be used during intial setup to choose HSE load capacitors Then it is meant to be used as button input Decided to use ESDALC6V1W5 as ESD protection Is not ideal but should work for both 3.3V and 5V pins and has low capacitance (Used by ST) VDDPA Supply Input supply for PA regulator Transmit high output power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"
- note removed: "STM32MP157FAD1 2x STM32WB55CGU6 2x STM32WB5MMGH6TR STM32MP135DAF7 STM32H7S7L8H6H STSPIN958TR STM32H7S3I8T6 LSM6DSV16XTR ISM330BXTR STM32WL55CCU6 STM32WL55JCI6 2x"
- moved on the sheet: C1, C10, C11, C12, C13, C14, C15, C16, C18, C3, C40, C41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
