File: LoRa_Board.kicad_sch (KiCad schematic)
At the start: 113 parts, among them IC1 RF_Switch_PE42440MLBB-Z, J10 SPI1_Headers, J11 Power Select Jumpers, J15 Power Select Jumpers, J16 USB_B_Micro, J17 BOOT0_Jumper, J19 SMA PCB END LAUNCH JACK ROUND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, J2 LPUART1_Headers, J3 Debug_Pins, J4 Coin Battery Jumper, J5 User Button Jumper, J6 Power Pins, J8 Conn_02x05_Odd_Even, J9 I2C1_Headers, SW1 Switch_NX3L1T3157GM,115, SW2 Switch_NX3L1T3157GM,115, U1 STM32WL55CCU6, U3 USBLC6-2SC6, U7 FT230XS, Y1 Clock_ECS-327MVATX-7-CN-TR, Y3 ABM3B-32.000MHZ-8-R30-B1U-T

Commit message: Update
Parts:
- removed C53: 33p_GJM0335C1E330JB01D_MURATA, Capacitor_SMD:C_0805_2012Metric, symbol Device:C
- removed C7: 100n, Capacitor_SMD:C_0805_2012Metric, symbol Device:C
- removed Y1: Clock_ECS-327MVATX-7-CN-TR, Personal_Project:Clock_ECS327MVATX7CNTR, symbol Personal_Projects:Clock_ECS-327MVATX-7-CN-TR
- removed Y3: ABM3B-32.000MHZ-8-R30-B1U-T, Personal_Project:XTAL_ABM3B-32.000MHZ-10-R30-B1U-T, symbol Personal_Projects:ABM3B-32.000MHZ-10-R30-B1U-T
- added C17: 1p2_GJM1555C1H1R2WB01D, Capacitor_SMD:C_0805_2012Metric, symbol Device:C
- added C20, C21: 33p_NMC0603NPO330J50TRPF, Capacitor_SMD:C_0603_1608Metric, symbol Device:C
- added C22: 3p3_GRM1885C1H3R3CA01D, Capacitor_SMD:C_0603_1608Metric, symbol Device:C
- added C4: 10n, Capacitor_SMD:C_0805_2012Metric, symbol Device:C
- added C6: 10p, Capacitor_SMD:C_0805_2012Metric, symbol Device:C
- added FB2: Murata_BLM21AG102SZ1D, Capacitor_SMD:C_0805_2012Metric, symbol Device:FerriteBead
- added OS1: Oscillator_ECS-327MVATX-3-CN-TR, Personal_Project:Oscillator_ECS327MVATX3CNTR, symbol Personal_Projects:Oscillator_ECS-327MVATX-3-CN-TR
- added OS2: Oscillator_ECS-TXO-32CSMV-320-AN-TR, Personal_Project:Oscillator_ECSTXO32CSMV320ANTR, symbol Personal_Projects:Oscillator_ECS-TXO-32CSMV-320-AN-TR
- added R1: 220R, Resistor_SMD:R_0805_2012Metric, symbol Device:R
- C2: value 220p_GRM1555C2A221GE01 -> 68p_GRM1555C2A221GE01
- C43: value 33p_GJM0335C1E330JB01D_MURATA -> 100n_CL21B104KCFNNNE
- C46: value 20p_GJM1555C1H200GB01 -> 2p2_GJM1555C1H200GB01
- C47: value 18p_GJM1555C1H180FB01 -> 1p2_GJM1555C1H180FB01
- C48: value 30p_GJM1555C1H300FB01 -> 5p6_GJM1555C1H300FB01
- C5: value 33p_GJM0335C1E330JB01D_MURATA -> 33p_NMC0603NPO330J50TRPF; footprint Capacitor_SMD:C_0805_2012Metric -> Capacitor_SMD:C_0603_1608Metric
- C51: value 100n_FCC0402KRX7R7BB104 -> 47p_KGQ21HCG2D470JT
- L2: value 51n_LQW18AN51NG0Z -> 8n7_LQW18AN51NG0Z
- L7: value 12n_LQW18AN12NG0Z -> 3n6_LQW18AN12NG0Z
Connections:
- net +3.3V: now also C22.1, OS1.4 (VDD); no longer C43.1, C51.1
- net GND: now also C17.2, C20.2, C21.2, C22.2, C4.1, OS1.2 (GND), OS2.1 (GND_1), OS2.2 (GND_2)
- net PB4: no longer U1.2 (PB4)
- net PH0-OSC_IN: now also C6.2
- net VDDPA: now also C20.1
- net VFBSMPS: now also C21.1
- net VR_PA: now also C17.1
- net at R2.1: now also OS1.3 (OUTPUT)
- net PB0_CTRL1 renamed PB4_CTRL1
- net PB4_CTRL1: now also U1.2 (PB4); no longer U1.30 (PB0)
- new net: OS2.3 (OUTPUT), R1.1
- new net: C4.2, FB2.2, OS2.4 (VDD)
- new net: C6.1, R1.2
- new net PB0_VDD_TCXO: C43.1, C51.1, FB2.1, U1.30 (PB0)
- no-connect marks 9 -> 10
Other:
- note added: "Clipped Sine Wave Oscillator - Series C eliminates DC component - MCU acciepots clock above zero so the clock signal gets biased (increased) inside the MCU."
- note added: "Internal pullup resistor allows active output if pin 1 is NC"
- note added: "Reference design: BLM15HG102SN1"
- note removed: "Capacitors inside MCU Set registers"
- note removed: "Place near VDDPA pin"
- note removed: "The devices include internal programmable capacitances that can be used to tune the crystal frequency in order to compensate the PCB parasitic one. Load capacitors are located in the MCU and can be set using SUBGHZ_HSEINTRIMR and SUBGHZ_HSEOUTTRIMR registers minimum value ~11.3 pF maximum capacitor value ~33.4 pF The HSE32 frequency can be measured by outputting the HSE32 clock on the MCO when in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"
- moved on the sheet: C1, C14, C16, C43, C51, ESD1, J11, LDO1

Commit message: Update
Parts:
- removed J11, J15: Power Select Jumpers, Personal_Project:PinHeader_2x03_P2.54mm_Vertical_PINS, symbol Connector_Generic:Conn_02x03_Top_Bottom
- added J1: 3V_Selection_Header, Connector_PinHeader_2.54mm:PinHeader_1x03_P2.54mm_Vertical, symbol Connector_Generic:Conn_01x03
- added J7: 5V_Selection_Header, Connector_PinHeader_2.54mm:PinHeader_1x03_P2.54mm_Vertical, symbol Connector_Generic:Conn_01x03
- added SHLD1: RFShield_OnePiece, Personal_Project:RF_Shield_MS631-10F, symbol Device:RFShield_OnePiece
- C50: value 18p_GJM1555C1H180FB01 -> 1p2_GJM1555C1H180FB01
- C58: value 220p_GRM1555C2A221GE01 -> 33p_GRM1555C2A221GE01
- C59, C60: value 22p_GJM1555C1H220FB01 -> 3p3_GJM1555C1H220FB01
- C61: value 15p_GJM1555C1H150FB01 -> 3p6_GJM1555C1H150FB01
- C62: value 18p_GJM1555C1H120FB01 -> 2p7_GJM1555C1H120FB01
- L10: value 120n_LQW18ANR12G00 -> 11n_LQW18ANR12G00
- L9: value 47n_LQW18AN47NG0Z -> 8n7_LQW18AN47NG0Z
Connections:
- net +3.3V: now also J1.2 (Pin_2)
- net +5V: now also J7.2 (Pin_2)
- net GND: now also J3.1 (Pin_1), J3.7 (Pin_7), SHLD1.1 (Shield)
- net LD_OUT_3V3: now also J1.3 (Pin_3)
- net VBUS_5V: now also ESD1.5 (I/O4), J7.3 (Pin_3); no longer ESD1.4 (I/O3)
- net 3V3_SW renamed EXT_3V
- net EXT_3V: now also J6.3 (Pin_3), J1.1 (Pin_1); no longer J3.7 (Pin_7)
- net 5V_SW: no longer names the net of ESD1.1 (I/O1)
- net 5V_SW: no longer J3.1 (Pin_1)
- net PC_3V3: no longer names the net of ESD2.1 (I/O1)
- net PC_3V3: no longer J6.3 (Pin_3)
- net PC_5V renamed EXT_5V
- net EXT_5V: now also ESD1.4 (I/O3), J7.1 (Pin_1); no longer ESD1.5 (I/O4)
- no-connect marks 10 -> 12
