File: LoRa_Board.kicad_sch (KiCad schematic)
At the start: 120 parts, among them IC1 RF_Switch_PE42440MLBB-Z, J1 3V_Selection_Header, J10 SPI1_Headers, J16 USB_B_Micro, J17 BOOT0_Jumper, J19 SMA PCB END LAUNCH JACK ROUND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, J2 LPUART1_Headers, J3 Debug_Pins, J4 Coin Battery Jumper, J5 User Button Jumper, J6 Power Pins, J7 5V_Selection_Header, J8 Conn_02x05_Odd_Even, J9 I2C1_Headers, SW1 Switch_NX3L1T3157GM,115, SW2 Switch_NX3L1T3157GM,115, U1 STM32WL55CCU6, U3 USBLC6-2SC6, U7 FT230XS

Commit message: Update
Parts:
- removed ESD2: ESDALC6V1W5, Personal_Project:SOT323-5L_STM-L, symbol Personal_Projects:ESDALC6V1W5
- removed J10: SPI1_Headers, Connector_PinHeader_2.54mm:PinHeader_1x06_P2.54mm_Vertical, symbol Connector_Generic:Conn_01x06
- removed J2: LPUART1_Headers, Connector_PinHeader_2.54mm:PinHeader_1x04_P2.54mm_Vertical, symbol Connector_Generic:Conn_01x04
- removed J9: I2C1_Headers, Connector_PinHeader_2.54mm:PinHeader_1x04_P2.54mm_Vertical, symbol Connector_Generic:Conn_01x04
- removed R14, R15, R17, R18, R19: 100R, Resistor_SMD:R_0805_2012Metric, symbol Device:R
- added J11: SPI1_Headers, Connector_PinHeader_2.54mm:PinHeader_2x05_P2.54mm_Horizontal, symbol Connector_Generic:Conn_02x05_Odd_Even
- added J2: I2C1_Headers, Connector_PinHeader_2.54mm:PinHeader_2x03_P2.54mm_Horizontal, symbol Connector_Generic:Conn_02x03_Odd_Even
- added J9: LPUART1_Headers, Connector_PinHeader_2.54mm:PinHeader_2x03_P2.54mm_Horizontal, symbol Connector_Generic:Conn_02x03_Odd_Even
- added R3, R4, R9: 33R, Resistor_SMD:R_0805_2012Metric, symbol Device:R
- J3: footprint Connector_PinHeader_2.54mm:PinHeader_2x04_P2.54mm_Vertical -> Connector_PinHeader_2.54mm:PinHeader_2x04_P2.54mm_Horizontal
- J8: footprint Connector_PinHeader_2.54mm:PinHeader_2x05_P2.54mm_Vertical -> Connector_PinHeader_2.54mm:PinHeader_2x05_P2.54mm_Horizontal
- R12, R13, R16: value 100R -> 33R
Connections:
- net +3.3V: now also J11.1 (Pin_1), J2.1 (Pin_1), J9.6 (Pin_6)
- net EXT_3V: now also ESD1.4 (I/O3), J1.3 (Pin_3); no longer J1.1 (Pin_1)
- net EXT_5V: now also ESD1.3 (I/O2); no longer ESD1.4 (I/O3)
- net GND: now also J8.1 (Pin_1), J8.3 (Pin_3), J8.5 (Pin_5), J8.7 (Pin_7), J8.9 (Pin_9), J11.10 (Pin_10), J11.2 (Pin_2), J11.4 (Pin_4), J11.6 (Pin_6), J11.8 (Pin_8), J2.2 (Pin_2), J2.4 (Pin_4), J2.6 (Pin_6), J9.1 (Pin_1), J9.3 (Pin_3), J9.5 (Pin_5)
- net LD_OUT_3V3: now also J1.1 (Pin_1); no longer J1.3 (Pin_3)
- net NRST: now also J3.6 (Pin_6); no longer J3.8 (Pin_8)
- net PA0: now also J8.2 (Pin_2); no longer J8.1 (Pin_1)
- net PA13_SWDIO: now also J3.8 (Pin_8); no longer J3.2 (Pin_2)
- net PA14_SWCLK: now also J3.2 (Pin_2); no longer J3.4 (Pin_4)
- net PA4_SPI1_NSS: now also R3.1
- net PB3_SWO: now also J3.4 (Pin_4); no longer J3.6 (Pin_6)
- net PB5_SPI1_MOSI: now also R9.1
- net PB7_I2C1_SDA: now also J2.3 (Pin_3)
- net PB8_I2C1_SCL: now also J2.5 (Pin_5)
- net PC15-OSC32_OUT: no longer J8.9 (Pin_9)
- net at R16.2: now also J11.3 (Pin_3)
- net at R13.2: now also J9.2 (Pin_2)
- net at R12.2: now also J9.4 (Pin_4)
- net PA5 renamed PA5_INOUTRF
- net PA5_INOUTRF: now also R6.1; no longer J8.2 (Pin_2)
- net PA6_SPI1_MISO: no longer names the net of U1.14 (PA6)
- net PA7 renamed PA7_HPLP_CTRL
- net PA7_HPLP_CTRL: now also R20.1, SW1.6 (S); no longer J8.3 (Pin_3)
- net PA9: no longer names the net of U1.17 (PA9)
- net PA9: no longer J8.5 (Pin_5)
- net PB12 renamed PB12_USR_BTN
- net PB12_USR_BTN: now also J5.2 (Pin_2)
- net PB2_CTRL2 renamed PB2_RFVCTRL
- net PB2_RFVCTRL: now also SW2.6 (S); no longer R6.1
- removed net PB4: J5.2 (Pin_2), J8.7 (Pin_7)
- removed net PB4_CTRL1: R20.1, SW1.6 (S), SW2.6 (S), U1.2 (PB4)
- new net: J11.7 (Pin_7), R4.2
- new net: J11.5 (Pin_5), R3.2
- new net: J11.9 (Pin_9), R9.2
- new net PB4_SPI1_MISO: R4.1, U1.2 (PB4)
Other:
- moved on the sheet: ESD1, J1, J7, R16

Commit message: Update
Parts:
- removed ESD1: ESDALC6V1W5, Personal_Project:SOT323-5L_STM-L, symbol Personal_Projects:ESDALC6V1W5
- removed J1: 3V_Selection_Header, Connector_PinHeader_2.54mm:PinHeader_1x03_P2.54mm_Vertical, symbol Connector_Generic:Conn_01x03
- removed J11: SPI1_Headers, Connector_PinHeader_2.54mm:PinHeader_2x05_P2.54mm_Horizontal, symbol Connector_Generic:Conn_02x05_Odd_Even
- removed J5: User Button Jumper, Connector_PinHeader_2.54mm:PinHeader_1x02_P2.54mm_Vertical, symbol Connector_Generic:Conn_01x02
- removed J7: 5V_Selection_Header, Connector_PinHeader_2.54mm:PinHeader_1x03_P2.54mm_Vertical, symbol Connector_Generic:Conn_01x03
- removed J8: Conn_02x05_Odd_Even, Connector_PinHeader_2.54mm:PinHeader_2x05_P2.54mm_Horizontal, symbol Connector_Generic:Conn_02x05_Odd_Even
- removed R16, R4, R9: 33R, Resistor_SMD:R_0805_2012Metric, symbol Device:R
- added ESD2: ESDALC6V1W5, Personal_Project:SOT323-5L_STM-L, symbol Personal_Projects:ESDALC6V1W5
- added J1: SPI1_Headers, Connector_PinHeader_2.54mm:PinHeader_2x04_P2.54mm_Horizontal, symbol Connector_Generic:Conn_02x04_Odd_Even
- added J10: 3V_Selection_Header, Connector_PinHeader_2.54mm:PinHeader_1x03_P2.54mm_Vertical, symbol Connector_Generic:Conn_01x03
- added J12: 5V_Selection_Header, Connector_PinHeader_2.54mm:PinHeader_1x03_P2.54mm_Vertical, symbol Connector_Generic:Conn_01x03
- added J5: General_Pin_Header, Connector_PinHeader_2.54mm:PinHeader_2x03_P2.54mm_Horizontal, symbol Connector_Generic:Conn_02x03_Odd_Even
- added R14, R15: 33R, Resistor_SMD:R_0805_2012Metric, symbol Device:R
- added S1: Switch_WS-SLSU SMT Mini Slide, Personal_Project:Switch_WS-SLSU SMT Mini Slide, symbol Personal_Projects:Switch_WS-SLSU SMT Mini Slide
Connections:
- net +3.3V: now also J9.1 (Pin_1), J1.1 (Pin_1), S1.2; no longer J9.6 (Pin_6)
- net +5V: now also J12.2 (Pin_2)
- net EXT_3V: now also ESD2.4 (I/O3), J10.3 (Pin_3)
- net EXT_5V: now also ESD2.3 (I/O2), J12.1 (Pin_1)
- net GND: now also J2.3 (Pin_3), J9.2 (Pin_2), J9.6 (Pin_6), ESD2.2 (GND), J1.2 (Pin_2), J1.3 (Pin_3), J1.6 (Pin_6), J1.7 (Pin_7), J5.1 (Pin_1), J5.4 (Pin_4), J5.5 (Pin_5); no longer J2.4 (Pin_4), J9.1 (Pin_1), J9.5 (Pin_5)
- net LD_OUT_3V3: now also J10.1 (Pin_1)
- net PA0: now also J5.6 (Pin_6)
- net PA1_SPI1_SCK: now also R15.2
- net PA2_LPUART1_TX: now also R14.2; no longer R12.1
- net PA4_SPI1_NSS: now also J5.3 (Pin_3); no longer R3.1
- net PA8_MCO: now also J5.2 (Pin_2)
- net PB12_USR_BTN: now also C3.2, U6.1, U6.2
- net PB4_SPI1_MISO: now also R12.2
- net PB5_SPI1_MOSI: now also R3.1
- net PB7_I2C1_SDA: now also J2.4 (Pin_4); no longer J2.3 (Pin_3)
- net VBUS_5V: now also ESD2.5 (I/O4), J12.3 (Pin_3)
- net at R3.2: now also J1.5 (Pin_5)
- net at R13.2: now also J9.5 (Pin_5); no longer J9.2 (Pin_2)
- net at J9.4 (Pin_4): now also R14.1; no longer R12.2
- net PA15: no longer names the net of U1.43 (PA15)
- net PC13: no longer names the net of U1.38 (PC13)
- new net: J1.4 (Pin_4), R12.1
- new net: J1.8 (Pin_8), R15.1
- new net: J10.2 (Pin_2), S1.1
- no-connect marks 12 -> 19
Other:
- note added: "Chip Select pin on general pin header"
- note added: "ON/OFF Switch"
- note added: "STM32MP157FAD1 TFBGA257 Pitch 0.5 2x STM32WB55CGU6 2x STM32WB5MMGH6TR STM32MP135DAF7 TFBGA320 Pitch 0.5 STM32H7S7L8H6H STSPIN958TR STM32H7S3I8T6 LSM6DSV16XTR ISM330BXTR STM32WL55CCU6 STM32WL55JCI6 2x AGVLB.25B.07.0060A Connector: I-PEX MHF® I (U.FL Compatible) GW.52.A153 2.4/5.8/7.1GHZ Hinged RP-SMA (M) Connector TI.96.A113 900-940MHZ Connector: SMA(M) CS5381K-KSZ IC 120DB 192KHZ MULTI-BIT ADC 2x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"
- note removed: "STM32MP157FAD1 2x STM32WB55CGU6 2x STM32WB5MMGH6TR STM32MP135DAF7 STM32H7S7L8H6H STSPIN958TR STM32H7S3I8T6 LSM6DSV16XTR ISM330BXTR STM32WL55CCU6 STM32WL55JCI6 2x AGVLB.25B.07.0060A Connector: I-PEX MHF® I (U.FL Compatible) GW.52.A153 2.4/5.8/7.1GHZ Hinged RP-SMA (M) Connector TI.96.A113 900-940MHZ Connector: SMA(M)"
- moved on the sheet: BH1, C14, C16, C19, C3, J2, J4, J6, LDO1, R13, R3, U6

Commit message: update
Parts:
- removed C1: 4u7, Capacitor_SMD:C_0805_2012Metric, symbol Device:C
- removed ESD2: ESDALC6V1W5, Personal_Project:SOT323-5L_STM-L, symbol Personal_Projects:ESDALC6V1W5
- removed J10: 3V_Selection_Header, Connector_PinHeader_2.54mm:PinHeader_1x03_P2.54mm_Vertical, symbol Connector_Generic:Conn_01x03
- removed J6: Power Pins, Connector_PinHeader_2.54mm:PinHeader_1x04_P2.54mm_Vertical, symbol Connector_Generic:Conn_01x04
- added C23: 4u7, Capacitor_SMD:C_0603_1608Metric_Pad1.08x0.95mm_HandSolder, symbol Device:C
- added D1: BZX84C4V3LT1G, Package_TO_SOT_SMD:SOT-23, symbol Diode:BZX84Cxx
- added D2: BZX84C6V2LT1G, Package_TO_SOT_SMD:SOT-23, symbol Diode:BZX84Cxx
- added J10: Power_Selector_Jumper, Connector_PinHeader_2.54mm:PinHeader_2x03_P2.54mm_Vertical, symbol Connector_Generic:Conn_02x03_Odd_Even
- added J6: JST_XH_2.54_Plug, Personal_Project:Connector_Power2pin_SHDRRA2W80P0X250_1X2_740X1150X610P, symbol Personal_Projects:Connector_Power2pin_JST_XH_2.54_Plug
- added Q2: MOSFET_SI2333DDS-T1-BE3, Personal_Project:MOSFET_ SI2333DDS_SOT_DS-T1-BE3_VIS, symbol Personal_Projects:MOSFET_SI2333DDS-T1-BE3
- added R4: 100k, Resistor_SMD:R_0603_1608Metric_Pad0.98x0.95mm_HandSolder, symbol Device:R
- added Z2: Diode_BZX84C6V2-7-F, Personal_Project:Diode_BZX84C6V2_SOT96P240X110-3N, symbol Personal_Projects:Diode_BZX84C6V2-7-F
- J12: value 5V_Selection_Header -> 3V_Selection_Header
Connections:
- net GND: now also C23.2, D1.1 (A), D2.1 (A), J6.1 (POWER-), R4.2
- net LD_OUT_3V3: now also J12.3 (Pin_3)
- net VBUS_5V: now also D2.3 (K), J10.5 (Pin_5); no longer J12.3 (Pin_3)
- net POWER_3V3: now reaches S1.1
- net POWER_3V3: now also J12.2 (Pin_2), C23.1
- net +5V renamed LDO_IN
- net LDO_IN: now also J10.4 (Pin_4), J10.6 (Pin_6); no longer J12.2 (Pin_2)
- net EXT_5V renamed EXT_POWER+_NOLDO
- net EXT_POWER+_NOLDO: now also J10.2 (Pin_2)
- new net EXT_POWER+: J6.2 (POWER+), Q2.3 (D)
- new net EXT_POWER+_PP: D1.3 (K), J10.1 (Pin_1), J10.3 (Pin_3), Q2.2 (S), Z2.3 (K)
- new net MOSFET_GATE: Q2.1 (G), R4.1, Z2.1 (A)
- no-connect marks 19 -> 18
Other:
- note added: "4u7 capacitor added near poower output"
- note added: "Input voltage range: 1.45V to 5.5V"
- note added: "Overvoltage protection for the PMOSFET VGS (VGS max is 8V)"
- note added: "Polarity Protection"
- moved on the sheet: C14, C16, LDO1

Commit message: Update
Parts:
- removed C23: 4u7, Capacitor_SMD:C_0603_1608Metric_Pad1.08x0.95mm_HandSolder, symbol Device:C
- removed D1: BZX84C4V3LT1G, Package_TO_SOT_SMD:SOT-23, symbol Diode:BZX84Cxx
- removed D2: BZX84C6V2LT1G, Package_TO_SOT_SMD:SOT-23, symbol Diode:BZX84Cxx
- removed J1: SPI1_Headers, Connector_PinHeader_2.54mm:PinHeader_2x04_P2.54mm_Horizontal, symbol Connector_Generic:Conn_02x04_Odd_Even
- removed J10: Power_Selector_Jumper, Connector_PinHeader_2.54mm:PinHeader_2x03_P2.54mm_Vertical, symbol Connector_Generic:Conn_02x03_Odd_Even
- removed J12: 3V_Selection_Header, Connector_PinHeader_2.54mm:PinHeader_1x03_P2.54mm_Vertical, symbol Connector_Generic:Conn_01x03
- removed J16: USB_B_Micro, Connector_USB:USB_Micro-B_Molex-105017-0001, symbol Connector:USB_B_Micro
- removed J18: ~, Personal_Project:SMA Clip Mount Adapter (bottom), symbol Personal_Projects:SMA_PCB_END_JACK_(BOTTOM)
- removed J6: JST_XH_2.54_Plug, Personal_Project:Connector_Power2pin_SHDRRA2W80P0X250_1X2_740X1150X610P, symbol Personal_Projects:Connector_Power2pin_JST_XH_2.54_Plug
- removed J9: LPUART1_Headers, Connector_PinHeader_2.54mm:PinHeader_2x03_P2.54mm_Horizontal, symbol Connector_Generic:Conn_02x03_Odd_Even
- removed Q2: MOSFET_SI2333DDS-T1-BE3, Personal_Project:MOSFET_ SI2333DDS_SOT_DS-T1-BE3_VIS, symbol Personal_Projects:MOSFET_SI2333DDS-T1-BE3
- removed R12, R13, R14, R15: 33R, Resistor_SMD:R_0805_2012Metric, symbol Device:R
- removed R4: 100k, Resistor_SMD:R_0603_1608Metric_Pad0.98x0.95mm_HandSolder, symbol Device:R
- removed S1: Switch_WS-SLSU SMT Mini Slide, Personal_Project:Switch_WS-SLSU SMT Mini Slide, symbol Personal_Projects:Switch_WS-SLSU SMT Mini Slide
- removed Z2: Diode_BZX84C6V2-7-F, Personal_Project:Diode_BZX84C6V2_SOT96P240X110-3N, symbol Personal_Projects:Diode_BZX84C6V2-7-F
- added C1: 4u7, Capacitor_SMD:C_0805_2012Metric, symbol Device:C
- added D3: ESD_TSD05DYFR, Personal_Project:ESD_TSD05DYFR_SOD2613X100N, symbol Personal_Projects:ESD_TSD05DYFR
- added D4: ESD_TSD03DYFR, Personal_Project:ESD_TSD05DYFR_SOD2613X100N, symbol Personal_Projects:ESD_TSD05DYFR
- added J1: JST_XH_2.54_Plug, Personal_Project:Connector_Power2pin_SHDRRA2W80P0X250_1X2_740X1150X610P, symbol Personal_Projects:Connector_Power2pin_JST_XH_2.54_Plug
- added J11: I2C1_Headers, Connector_PinHeader_2.54mm:PinHeader_2x03_P2.54mm_Horizontal, symbol Connector_Generic:Conn_02x03_Odd_Even
- added J13: SPI1_Headers, Connector_PinHeader_2.54mm:PinHeader_2x03_P2.54mm_Horizontal, symbol Connector_Generic:Conn_02x03_Odd_Even
- added J7: LPUART1_Headers, Connector_PinHeader_2.54mm:PinHeader_2x03_P2.54mm_Horizontal, symbol Connector_Generic:Conn_02x03_Odd_Even
- added J8: USB_B_Micro, Connector_USB:USB_Micro-B_XKB_U254-051T-4BH83-F1S, symbol Connector:USB_B_Micro
- added J9: 3V_Selection_Header, Connector_PinHeader_2.54mm:PinHeader_1x03_P2.54mm_Vertical, symbol Connector_Generic:Conn_01x03
- added Q1: MOSFET_SI2333DDS-T1-BE3, Personal_Project:MOSFET_ SI2333DDS_SOT_DS-T1-BE3_VIS, symbol Personal_Projects:MOSFET_SI2333DDS-T1-BE3
- added R16, R17, R18, R25, R9: 33R, Resistor_SMD:R_0805_2012Metric, symbol Device:R
- added S2: Switch_WS-SLSU SMT Mini Slide, Personal_Project:Switch_WS-SLSU SMT Mini Slide, symbol Personal_Projects:Switch_WS-SLSU SMT Mini Slide
- added Z1: Diode_BZX84C6V2-7-F, Personal_Project:Diode_BZX84C6V2_SOT96P240X110-3N, symbol Personal_Projects:Diode_BZX84C6V2-7-F
- IC1: footprint Personal_Project:PE42440_QFN50P300X300X80-17N -> Personal_Project:RF_SWITCH_PE42440_QFN50P300X300X80-17N
- J2: value I2C1_Headers -> Power_Selector_Jumper; footprint Connector_PinHeader_2.54mm:PinHeader_2x03_P2.54mm_Horizontal -> Connector_PinHeader_2.54mm:PinHeader_2x03_P2.54mm_Vertical
- R3: value 33R -> 100k
Connections:
- net +3.3V: now also S2.2; no longer J2.1 (Pin_1)
- net EXT_POWER+: now also J1.2 (POWER+), Q1.3 (D)
- net EXT_POWER+_NOLDO: now also J2.2 (Pin_2), D4.1 (K), J9.1 (Pin_1)
- net EXT_POWER+_PP: now also J2.1 (Pin_1), J2.3 (Pin_3), D3.1 (K), Q1.2 (S), Z1.3 (K)
- net GND: now also R3.2, C1.2, D3.2 (A), D4.2 (A), J1.1 (POWER-), J11.2 (Pin_2), J11.3 (Pin_3), J11.4 (Pin_4), J11.6 (Pin_6), J13.2 (Pin_2), J13.3 (Pin_3), J13.6 (Pin_6), J7.2 (Pin_2), J7.3 (Pin_3), J7.4 (Pin_4), J7.6 (Pin_6), J8.5 (GND), J8.6 (Shield); no longer J2.2 (Pin_2), J2.3 (Pin_3), J2.6 (Pin_6)
- net LDO_IN: now also J2.4 (Pin_4), J2.6 (Pin_6)
- net LD_OUT_3V3: now also J9.3 (Pin_3)
- net MOSFET_GATE: now also R3.1, Q1.1 (G), Z1.1 (A)
- net PA1_SPI1_SCK: now also R18.1
- net PA2_LPUART1_TX: now also R9.2
- net PA3_LPUART1_RX: now also R16.1
- net PB4_SPI1_MISO: now also R17.1
- net PB5_SPI1_MOSI: now also R25.2; no longer R3.1
- net PB7_I2C1_SDA: now also J11.1 (Pin_1); no longer J2.4 (Pin_4)
- net PB8_I2C1_SCL: now also J11.5 (Pin_5); no longer J2.5 (Pin_5)
- net POWER_3V3: now also C1.1, J9.2 (Pin_2), S2.1
- net USB_D2+: now also J8.3 (D+)
- net USB_D2-: now also J8.2 (D-)
- net VBUS_5V: now also J2.5 (Pin_5), J8.1 (VBUS)
- net at R7.2: now also J8.4 (ID)
- net VBUS_5V_FB renamed +5V_VBUS_FB
- new net: J13.1 (Pin_1), R17.2
- new net: J13.4 (Pin_4), R25.1
- new net: J13.5 (Pin_5), R18.2
- new net: J7.1 (Pin_1), R9.1
- new net: J7.5 (Pin_5), R16.2
Other:
- note added: "5.5V Max Voltage of the LDO"
- note added: "LDO Input voltage range: 1.45V to 5.5V Abs Max Vin is 6V"
- moved on the sheet: C63, C64, C65, C66, C67, C9, FB3, J5, R10, R11, U3, U7

Commit message: Update
Other:
- note removed: "STM32MP157FAD1 TFBGA257 Pitch 0.5 2x STM32WB55CGU6 2x STM32WB5MMGH6TR STM32MP135DAF7 TFBGA320 Pitch 0.5 STM32H7S7L8H6H STSPIN958TR STM32H7S3I8T6 LSM6DSV16XTR ISM330BXTR STM32WL55CCU6 STM32WL55JCI6 2x AGVLB.25B.07.0060A Connector: I-PEX MHF® I (U.FL Compatible) GW.52.A153 2.4/5.8/7.1GHZ Hinged RP-SMA (M) Connector TI.96.A113 900-940MHZ Connector: SMA(M) CS5381K-KSZ IC 120DB 192KHZ MULTI-BIT ADC 2x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"
Changed lines of the file:
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@@
-		)
-	)
-	(text "STM32MP157FAD1 TFBGA257 Pitch 0.5 2x\nSTM32WB55CGU6 2x\nSTM32WB5MMGH6TR\nSTM32MP135DAF7 TFBGA320 Pitch 0.5\nSTM32H7S7L8H6H\n\nSTSPIN958TR\nSTM32H7S3I8T6\nLSM6DSV16XTR\nISM330BXTR\nSTM32WL55CCU6\nSTM32WL55JCI6 2x\n\nAGVLB.25B.07.0060A Connector: I-PEX MHF® I (U.FL Compatible)\nGW.52.A153 2.4/5.8/7.1GHZ Hinged RP-SMA (M) Connector\nTI.96.A113 900-940MHZ Connector: SMA(M)\n\nCS5381K-KSZ IC 120DB 192KHZ MULTI-BIT ADC 2x\n\nR9A07G044L28GBG#BC0 551-LFBGA (21x21) pitch 0.8mm"
-		(exclude_from_sim no)
-		(at -45.72 26.162 0)
-		(effects
-			(font
-				(size 1 1)
-			)
-			(justify left)
 		)
 	)

Commit message: Update
Parts:
- removed BH1: Battery_Holder_1060TR, Personal_Project:Battery_Holder_1060TR, symbol Personal_Projects:Battery_Holder_1060TR
- removed C1, C13, C41, C67: 4u7, Capacitor_SMD:C_0805_2012Metric, symbol Device:C
- removed C10, C11, C12, C19, C42, C65, C66: 100n, Capacitor_SMD:C_0805_2012Metric, symbol Device:C
- removed C14, C15, C16: 1u, Capacitor_SMD:C_0805_2012Metric, symbol Device:C
- removed C17: 1p2_GJM1555C1H1R2WB01D, Capacitor_SMD:C_0805_2012Metric, symbol Device:C
- removed C18, C4: 10n, Capacitor_SMD:C_0805_2012Metric, symbol Device:C
- removed C2: 68p_GRM1555C2A221GE01, Capacitor_SMD:C_0805_2012Metric, symbol Device:C
- removed C20, C21, C5: 33p_NMC0603NPO330J50TRPF, Capacitor_SMD:C_0603_1608Metric, symbol Device:C
- removed C22: 3p3_GRM1885C1H3R3CA01D, Capacitor_SMD:C_0603_1608Metric, symbol Device:C
- removed C3, C8: 1uF, Capacitor_SMD:C_0805_2012Metric, symbol Device:C
- removed C33: 47n_Murata_GCM155R71E473KA55, Capacitor_SMD:C_0805_2012Metric, symbol Device:C
- removed C34: 68p_Murata_GCM1555C1H680JA16, Capacitor_SMD:C_0805_2012Metric, symbol Device:C
- removed C35, C39: 18p_GJM1555C1H180FB01, Capacitor_SMD:C_0805_2012Metric, symbol Device:C
- removed C36: 20p_GJM1555C1H200GB01, Capacitor_SMD:C_0805_2012Metric, symbol Device:C
- removed C37: 30p_GJM1555C1H300FB01, Capacitor_SMD:C_0805_2012Metric, symbol Device:C
- removed C38: 220p_GRM1555C2A221GE01, Capacitor_SMD:C_0805_2012Metric, symbol Device:C
- removed C40: 470n, Capacitor_SMD:C_0805_2012Metric, symbol Device:C
- removed C43: 100n_CL21B104KCFNNNE, Capacitor_SMD:C_0805_2012Metric, symbol Device:C
- removed C44, C49: 33p_CC0402GRNPO9BN330, Capacitor_SMD:C_0805_2012Metric, symbol Device:C
- removed C45, C54, C69: 1n, Capacitor_SMD:C_0805_2012Metric, symbol Device:C
- removed C46: 2p2_GJM1555C1H200GB01, Capacitor_SMD:C_0805_2012Metric, symbol Device:C
- removed C47, C50: 1p2_GJM1555C1H180FB01, Capacitor_SMD:C_0805_2012Metric, symbol Device:C
- removed C48: 5p6_GJM1555C1H300FB01, Capacitor_SMD:C_0805_2012Metric, symbol Device:C
- removed C51: 47p_KGQ21HCG2D470JT, Capacitor_SMD:C_0805_2012Metric, symbol Device:C
- removed C52, C55, C6, C68, C9: 10p, Capacitor_SMD:C_0805_2012Metric, symbol Device:C
- removed C58: 33p_GRM1555C2A221GE01, Capacitor_SMD:C_0805_2012Metric, symbol Device:C
- removed C59, C60: 3p3_GJM1555C1H220FB01, Capacitor_SMD:C_0805_2012Metric, symbol Device:C
- removed C61: 3p6_GJM1555C1H150FB01, Capacitor_SMD:C_0805_2012Metric, symbol Device:C
- removed C62: 2p7_GJM1555C1H120FB01, Capacitor_SMD:C_0805_2012Metric, symbol Device:C
- removed C63, C64: 47p, Capacitor_SMD:C_0805_2012Metric, symbol Device:C
- removed D3: ESD_TSD05DYFR, Personal_Project:ESD_TSD05DYFR_SOD2613X100N, symbol Personal_Projects:ESD_TSD05DYFR
- removed D4: ESD_TSD03DYFR, Personal_Project:ESD_TSD05DYFR_SOD2613X100N, symbol Personal_Projects:ESD_TSD05DYFR
- removed FB1: BLM21PG601SN1D_0805, Capacitor_SMD:C_0805_2012Metric, symbol Device:FerriteBead
- removed FB2: Murata_BLM21AG102SZ1D, Capacitor_SMD:C_0805_2012Metric, symbol Device:FerriteBead
- removed FB3: Part # MI0805K601R-10, Capacitor_SMD:C_0805_2012Metric, symbol Device:FerriteBead
- removed H1, H2, H3, H4: MountingHole_Pad, MountingHole:MountingHole_3.2mm_M3_Pad, symbol Mechanical:MountingHole_Pad
- removed IC1: RF_Switch_PE42440MLBB-Z, Personal_Project:RF_SWITCH_PE42440_QFN50P300X300X80-17N, symbol Personal_Projects:RF_Switch_PE42440MLBB-Z
- removed J1: JST_XH_2.54_Plug, Personal_Project:Connector_Power2pin_SHDRRA2W80P0X250_1X2_740X1150X610P, symbol Personal_Projects:Connector_Power2pin_JST_XH_2.54_Plug
- removed J11: I2C1_Headers, Connector_PinHeader_2.54mm:PinHeader_2x03_P2.54mm_Horizontal, symbol Connector_Generic:Conn_02x03_Odd_Even
- removed J13: SPI1_Headers, Connector_PinHeader_2.54mm:PinHeader_2x03_P2.54mm_Horizontal, symbol Connector_Generic:Conn_02x03_Odd_Even
- removed J17: BOOT0_Jumper, Connector_PinHeader_2.54mm:PinHeader_1x03_P2.54mm_Vertical, symbol Connector:Conn_01x03_Pin
- removed J19: SMA PCB END LAUNCH JACK ROUND PO, Personal_Project:SMA Clip Mount Adapter (top), symbol Personal_Projects:SMA PCB END LAUNCH JACK ROUND PO
- removed J2: Power_Selector_Jumper, Connector_PinHeader_2.54mm:PinHeader_2x03_P2.54mm_Vertical, symbol Connector_Generic:Conn_02x03_Odd_Even
- removed J3: Debug_Pins, Connector_PinHeader_2.54mm:PinHeader_2x04_P2.54mm_Horizontal, symbol Connector_Generic:Conn_02x04_Odd_Even
- removed J4: Coin Battery Jumper, Connector_PinHeader_2.54mm:PinHeader_1x03_P2.54mm_Vertical, symbol Connector_Generic:Conn_01x03
- removed J5: General_Pin_Header, Connector_PinHeader_2.54mm:PinHeader_2x03_P2.54mm_Horizontal, symbol Connector_Generic:Conn_02x03_Odd_Even
- removed J7: LPUART1_Headers, Connector_PinHeader_2.54mm:PinHeader_2x03_P2.54mm_Horizontal, symbol Connector_Generic:Conn_02x03_Odd_Even
- removed J8: USB_B_Micro, Connector_USB:USB_Micro-B_XKB_U254-051T-4BH83-F1S, symbol Connector:USB_B_Micro
- removed J9: 3V_Selection_Header, Connector_PinHeader_2.54mm:PinHeader_1x03_P2.54mm_Vertical, symbol Connector_Generic:Conn_01x03
- removed L1: 15u_MLZ2012M150W_TDK, Inductor_SMD:L_0805_2012Metric_Pad1.15x1.40mm_HandSolder, symbol Device:L
- removed L10: 11n_LQW18ANR12G00, Inductor_SMD:L_0603_1608Metric_Pad1.05x0.95mm_HandSolder, symbol Device:L
- removed L14, L5: 6n8_LQW18AN6N8C00, Inductor_SMD:L_0603_1608Metric_Pad1.05x0.95mm_HandSolder, symbol Device:L
- removed L15: 160n_LQW18ANR16G00, Inductor_SMD:L_0603_1608Metric_Pad1.05x0.95mm_HandSolder, symbol Device:L
- removed L16: 12n_LQW18AN12NG0Z, Inductor_SMD:L_0603_1608Metric_Pad1.05x0.95mm_HandSolder, symbol Device:L
- removed L17: 51n_LQW18AN51NG0Z, Inductor_SMD:L_0603_1608Metric_Pad1.05x0.95mm_HandSolder, symbol Device:L
- removed L18: 47n_LQW15AN47NJ00, Inductor_SMD:L_0603_1608Metric_Pad1.05x0.95mm_HandSolder, symbol Device:L
- removed L2: 8n7_LQW18AN51NG0Z, Inductor_SMD:L_0603_1608Metric_Pad1.05x0.95mm_HandSolder, symbol Device:L
- removed L6: 33n_LQW15AN33NG00, Inductor_SMD:L_0603_1608Metric_Pad1.05x0.95mm_HandSolder, symbol Device:L
- removed L7: 3n6_LQW18AN12NG0Z, Inductor_SMD:L_0603_1608Metric_Pad1.05x0.95mm_HandSolder, symbol Device:L
- removed L9: 8n7_LQW18AN47NG0Z, Inductor_SMD:L_0603_1608Metric_Pad1.05x0.95mm_HandSolder, symbol Device:L
- removed LDO1: LDO_TLV75733PDBVR, Personal_Project:LDO_SOT95P280X145-5N, symbol Personal_Projects:LDO_TLV75733PDBVR
- removed OS1: Oscillator_ECS-327MVATX-3-CN-TR, Personal_Project:Oscillator_ECS327MVATX3CNTR, symbol Personal_Projects:Oscillator_ECS-327MVATX-3-CN-TR
- removed OS2: Oscillator_ECS-TXO-32CSMV-320-AN-TR, Personal_Project:Oscillator_ECSTXO32CSMV320ANTR, symbol Personal_Projects:Oscillator_ECS-TXO-32CSMV-320-AN-TR
- removed Q1: MOSFET_SI2333DDS-T1-BE3, Personal_Project:MOSFET_ SI2333DDS_SOT_DS-T1-BE3_VIS, symbol Personal_Projects:MOSFET_SI2333DDS-T1-BE3
- removed R1: 220R, Resistor_SMD:R_0805_2012Metric, symbol Device:R
- removed R10, R11: 27, Resistor_SMD:R_0805_2012Metric, symbol Device:R
- removed R16, R17, R18, R25, R9: 33R, Resistor_SMD:R_0805_2012Metric, symbol Device:R
- removed R2: 10R, Resistor_SMD:R_0805_2012Metric, symbol Device:R
- removed R20, R5, R6: 100R, Resistor_SMD:R_0805_2012Metric, symbol Device:R
- removed R3, R7: 100k, Resistor_SMD:R_0805_2012Metric, symbol Device:R
- removed R8: 1k, Resistor_SMD:R_0805_2012Metric, symbol Device:R
- removed S2: Switch_WS-SLSU SMT Mini Slide, Personal_Project:Switch_WS-SLSU SMT Mini Slide, symbol Personal_Projects:Switch_WS-SLSU SMT Mini Slide
- removed SHLD1: RFShield_OnePiece, Personal_Project:RF_Shield_MS631-10F, symbol Device:RFShield_OnePiece
- removed SW1, SW2: Switch_NX3L1T3157GM,115, Personal_Project:Switch_NX3L1T3157GM115, symbol Personal_Projects:Switch_NX3L1T3157GM,115
- removed U1: STM32WL55CCU6, Package_DFN_QFN:QFN-48-1EP_7x7mm_P0.5mm_EP5.6x5.6mm, symbol MCU_ST_STM32WL:STM32WL55CCUx
- removed U2, U6: ~, Personal_Project:Button_KMR231GLFS, symbol Personal_Projects:Button_KMR231GLFS
- removed U3: USBLC6-2SC6, Package_TO_SOT_SMD:SOT-23-6, symbol Power_Protection:USBLC6-2SC6
- removed U7: FT230XS, Package_SO:SSOP-16_3.9x4.9mm_P0.635mm, symbol Interface_USB:FT230XS
- removed Z1: Diode_BZX84C6V2-7-F, Personal_Project:Diode_BZX84C6V2_SOT96P240X110-3N, symbol Personal_Projects:Diode_BZX84C6V2-7-F
Connections:
- no-connect marks 18 -> 0
Other:
- added sheet Interfaces (Interfaces.kicad_sch)
- added sheet Power_Management (Power_Management.kicad_sch)
- added sheet RF_ANT (RF_ANT.kicad_sch)
- added sheet STM32WL55CCU6 (STM32WL55CCU6.kicad_sch)
- added sheet USB (USB.kicad_sch)
- note removed: "100 nF for each VDD or VDDIO2 (Ceramic capacitors)"
- note removed: "10uF could be 4u7"
- note removed: "4u7 capacitor added near poower output"
- note removed: "5.5V Max Voltage of the LDO"
- note removed: "70R@100MHz"
- note removed: "BOOT0 Switch HIGH enables UART or I2C too allow programminng of the MCU"
- note removed: "Band pass filter for around 900 MHz"
- note removed: "CTRL LOGIC CTRL1=LOW, CTRL2=LOW VDDPA=VDDSMPS, RF_HP, ANT=RF_HP CTRL1=HIGH, CTRL2=LOW VDDPA=FBSMPS, RF_LP, ANT=RFI (RF3) CTRL1=HIGH, CTRL2=HIGH VDDPA=FBSMPS, RF_LP, ANT=RF_LP(RF4)"
- note removed: "Can be used as GPIO"
- note removed: "Chip Select pin on general pin header"
- note removed: "Clipped Sine Wave Oscillator - Series C eliminates DC component - MCU acciepots clock above zero so the clock signal gets biased (increased) inside the MCU."
- note removed: "Clock Output"
- note removed: "EP is optional adhesive zone"
- note removed: "FCM1608KF-601T03TAI-TECH"
- note removed: "FT230XS as close as possible to USB port"
- note removed: "For highest RF power"
- note removed: "For the UFQFPN48 package, VREF+ is internally connected to VDDA"
- note removed: "If shutdown capability is not required, connect EN to IN."
- note removed: "Input voltage range: 1.45V to 5.5V"
- note removed: "Internal pullup resistor allows active output if pin 1 is NC"
- note removed: "LDO Input voltage range: 1.45V to 5.5V Abs Max Vin is 6V"
- note removed: "ON/OFF Switch"
- note removed: "Ordered: STM32WL55CCU6 x1 48-UFQFN Exposed Pad STM32WL55JCI6 x2"
- note removed: "Overvoltage protection for the PMOSFET VGS (VGS max is 8V)"
- note removed: "PIN1 NC = Oscillation"
- note removed: "PWR_FLG tells KiCad that this is power source"
- note removed: "Peripherals: 1. EEPROM memory chips (SPI or I2C) 2. Bluetooth 3. GPS 4. Orientation sensor (MEMS) 5. USB 6. Ethernet (Maybe) 7. A set of user buttons (maybe 4)"
- note removed: "Place 33p Capacitors near the MCU"
- note removed: "Polarity Protection"
- note removed: "Reference design: BLM15HG102SN1"
- note removed: "Regulated PA supply output"
- note removed: "ST-LINK Connections: VCP_TX, SWCLK, SWDIO, VCP_RX, NRST"
- note removed: "These capacitors must be placed as close as possible to (or below) the appropriate pins on the underside of the PCB"
- note removed: "This 3.3V is from digital power rail"
- note removed: "VBUS is the voltage from the USB connector (5V)"
- note removed: "VDDA feeds ADC and DAC pins, and it needs more filtering"
- note removed: "VDDPA Power Amplifier voltage depends on the chosenn power transmission (HP or LP)"
- note removed: "VDDPA Supply Input supply for PA regulator"

Commit message: Update
Other:
- sheet Interfaces ports: added I2C1_SCL_HDR, I2C1_SDA_HDR, I2C2_SCL_HDR, I2C2_SDA_HDR, I/O_HDR0, I/O_HDR1, I/O_HDR2, I/O_HDR3, I/O_HDR4, I/O_HDR5, NRST, SPI_CLK, SPI_CS, SPI_MISO, SPI_MOSI, SWCLK, SWDIO, SWO, UART1_TX/RX, USR_BTN; removed none
- sheet Power_Management ports: added *RST; removed none
- sheet RF_ANT ports: added PA5_INOUTRF, PA7_HPLP_CTRL, RFI_N, RFI_P, RFO_HP, RFO_LP, VR_PA; removed none
- sheet STM32WL55CCU6 ports: added NRST, PA0_DEBUG_PWR-REGLP1S, PA10_DEBUG_RF-HSE32RDY, PA11_DEBUG_RF-NRESET, PA12_I2C2_SCL, PA13_SWDIO, PA14_SWCLK, PA15_I2C2_SDA, PA1_SPI1_SCK, PA2_LPUART1_TX, PA3_LPUART1_RX, PA4_SPI1_NSS, PA5_INOUTRF, PA6_LPUART1_CTS, PA7_HPLP_CTRL, PA8_MCO, PA9_USR_BTN, PB12_LPUART1_RTS, PB2_RFVCTRL, PB3_SWO, PB4_SPI1_MISO, PB5_SPI1_MOSI, PB6_USART1_TX, PB7_I2C1_SDA, PB8_I2C1_SCL, PC15-OSC32_OUT, RFI_N, RFI_P, RFO_HP, RFO_LP, VR_PA; removed none
- sheet USB ports: added UART_CTS, UART_RTS, UART_RX, UART_TX; removed none

Commit message: Update
Other:
- sheet RF_ANT renamed Antenna
Changed lines of the file:
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@@
 			(color 0 255 255 1.0000)
 		)
-		(property "Sheetname" "RF_ANT"
+		(property "Sheetname" "Antenna"
 			(at 29.21 23.4184 0)
 			(effects
