File: LoRa_Board.kicad_sch (KiCad schematic)
At the start: 0 parts

Commit message: PCB Layout
Other:
- sheet STM32WL55CCU6_GPIO ports: added BOOT0_EXTCTR, BOOT0_GPIO; removed none
- sheet STM32WL55CCU6_PWR ports: added NX3L1T3_RFVCTRL_S; removed PB2_RFVCTRL
- sheet STM32WL55CCU6_RF ports: added NX3L1T3_RF_S, SKY13414_V2, SKY13414_V3; removed PA5_INOUTRF, PA7_HPLP_CTRL
- sheet USB ports: added CP2102N_NRST, GPIO.1_RXT, UART_RXD, UART_TXD; removed UART_RX, UART_TX

Commit message: Power domain update
Connections:
- no-connect marks 0 -> 3
Other:
- sheet Interfaces ports: added I/O_HDR10, I/O_HDR6, I/O_HDR7, I/O_HDR8, I/O_HDR9; removed none
- sheet Power_Management ports: added BFR_RST, TPS62740_PG; removed *RST
