File: LoRa_Board.kicad_pcb (KiCad board)
At the start: 4 copper layers, 96 parts, among them J1 Pin_Headers, J10 SPI1_Headers, J11 Power Select Jumpers, J15 Power Select Jumpers, J16 USB_B_Micro, J17 BOOT0_Jumper, J19 SMA PCB END LAUNCH JACK ROUND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, J2 LPUART1_Headers, J3 Debug_Pins, J4 Coin Battery Jumper, J5 User Button Jumper, J6 Power Pins, J9 I2C1_Headers, U1 STM32WL55CCU6, U3 USBLC6-2SC6, U5 BGS12WN6E6327, U7 FT230XS, Y1 Clock_ECS-327MVATX-7-CN-TR, Y3 ABM3B-32.000MHZ-8-R30-B1U-T

Commit message: Update
Parts:
- moved C19 13.8 mm to (150.9, 60.6)
- moved C45 11.5 mm to (162.3, 74.7)
- moved C44 10.9 mm to (160.1, 74.7)
- moved J4 10.9 mm to (145.5, 56.7)
- moved C18 10.4 mm to (146.3, 62.7), turned to 0 degrees
- moved R9 10.3 mm to (180.0, 69.6)
- moved R1 8.54 mm to (181.1, 82.8)
- moved L6 7.70 mm to (168.1, 72.8)
- moved C57 6.61 mm to (183.1, 70.5), turned to -90 degrees
- moved R8 6.24 mm to (161.1, 86.4)
- moved U5 6.17 mm to (185.3, 77.5)
- moved C47 5.79 mm to (167.5, 75.8), turned to -90 degrees
- moved C55 5.08 mm to (184.2, 83.7), turned to 90 degrees
- moved C56 5.01 mm to (185.2, 70.5), turned to -90 degrees
- moved C58 4.87 mm to (188.5, 77.5), turned to 180 degrees
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Connections:
- R10 pad 2: /USBDP -> /USBDM
- R11 pad 2: /USBDM -> /USBDP
Routing:
- net /PC15-OSC32_OUT: track 0.00 -> 20.2 mm, vias 0 -> 1
- net +3.3V: track 0.00 -> 19.6 mm
- net /PA13_SWDIO: track 0.00 -> 19.0 mm, vias 0 -> 1
- net /PA14_SWCLK: track 0.00 -> 15.8 mm, vias 0 -> 1
- net +3.3VA: track 0.00 -> 10.6 mm
- net /PH1-OSC_OUT: track 0.00 -> 10.3 mm
- net /PC13: track 0.00 -> 9.74 mm
- net /VBAT: track 0.00 -> 8.83 mm
- net /PB2: track 0.00 -> 8.80 mm, vias 0 -> 1
- net /PB12: track 0.00 -> 8.74 mm, vias 0 -> 1
- net /PB0: track 0.00 -> 8.63 mm, vias 0 -> 1
- net /PA11_USART1_CTS: track 0.00 -> 8.36 mm
- net /PA10_USART1_RX: track 0.00 -> 8.30 mm
- net /PA12_USART1_RTS: track 0.00 -> 8.20 mm
- net /PH0-OSC_IN: track 0.00 -> 7.50 mm
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
Commit message: Update
Parts:
- FB1: value ILB1206ER700V_1206 -> BLM21PG601SN1D_0805; footprint Capacitor_SMD:C_1206_3216Metric_Pad1.33x1.80mm_HandSolder -> Capacitor_SMD:C_0805_2012Metric_Pad1.18x1.45mm_HandSolder
Changed lines of the file:
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@@
 		)
 	)
-	(footprint "Capacitor_SMD:C_1206_3216Metric_Pad1.33x1.80mm_HandSolder"
+	(footprint "Capacitor_SMD:C_0805_2012Metric_Pad1.18x1.45mm_HandSolder"
 		(layer "F.Cu")
 		(at 140.2 75.7 180)
-		(descr "Capacitor SMD 1206 (3216 Metric), square (rectangular) end terminal, IPC_7351 nominal with elongated pad for handsoldering. (Body size source: IPC-SM-782 page 76, https://www.pcb-3d.com/wordpress/wp-content/uploads/ipc-sm-782a_amendment_1_and_2.pdf), generated with kicad-footprint-generator")
+		(descr "Capacitor SMD 0805 (2012 Metric), square (rectangular) end terminal, IPC_7351 nominal with elongated pad for handsoldering. (Body size source: IPC-SM-782 page 76, https://www.pcb-3d.com/wordpress/wp-content/uploads/ipc-sm-782a_amendment_1_and_2.pdf, https://docs.google.com/spreadsheets/d/1BsfQQcO9C6DZCsRaXUlFlo91Tg2WpOkGARC1WS5S8t0/edit?usp=sharing), generated with kicad-footprint-generator")
 		(tags "capacitor handsolder")
 		(property "Reference" "FB1"
-			(at 0 -1.85 0)
+			(at 0 -1.68 180)
 			(layer "F.SilkS")
 			(effects
@@
 			)
 		)
-		(property "Value" "ILB1206ER700V_1206"
-			(at 0 1.85 0)
+		(property "Value" "BLM21PG601SN1D_0805"
+			(at 0 1.68 180)
 			(layer "F.Fab")
 			(effects
@@
 			)
 		)
-		(property "Footprint" "Capacitor_SMD:C_1206_3216Metric_Pad1.33x1.80mm_HandSolder"
+		(property "Footprint" "Capacitor_SMD:C_0805_2012Metric_Pad1.18x1.45mm_HandSolder"
 			(at 0 0 180)
 			(unlocked yes)
@@
 		(attr smd)
 		(fp_line
-			(start -0.711252 0.91)
-			(end 0.711252 0.91)
+			(start -0.261252 0.735)
+			(end 0.261252 0.735)
 			(stroke
 				(width 0.12)
@@
 		)
 		(fp_line
-			(start -0.711252 -0.91)
-			(end 0.711252 -0.91)
+			(start -0.261252 -0.735)
+			(end 0.261252 -0.735)
 			(stroke
 				(width 0.12)
@@
 		)
 		(fp_line
-			(start 2.48 1.15)
-			(end -2.48 1.15)
+			(start 1.88 0.98)
+			(end -1.88 0.98)
 			(stroke
 				(width 0.05)
@@
 		)
 		(fp_line
-			(start 2.48 -1.15)
-			(end 2.48 1.15)
+			(start 1.88 -0.98)
+			(end 1.88 0.98)
 			(stroke
 				(width 0.05)
@@
 		)
 		(fp_line
-			(start -2.48 1.15)
-			(end -2.48 -1.15)
+			(start -1.88 0.98)
+			(end -1.88 -0.98)
 			(stroke
 				(width 0.05)
@@
 		)
 		(fp_line
-			(start -2.48 -1.15)
-			(end 2.48 -1.15)
+			(start -1.88 -0.98)
+			(end 1.88 -0.98)
 			(stroke
 				(width 0.05)
@@
 		)
 		(fp_line
-			(start 1.6 0.8)
-			(end -1.6 0.8)
+			(start 1 0.625)
+			(end -1 0.625)
 			(stroke
 				(width 0.1)
@@
 		)
 		(fp_line
-			(start 1.6 -0.8)
-			(end 1.6 0.8)
+			(start 1 -0.625)
+			(end 1 0.625)
 			(stroke
 				(width 0.1)
@@
 		)
 		(fp_line
-			(start -1.6 0.8)
-			(end -1.6 -0.8)
+			(start -1 0.625)
+			(end -1 -0.625)
 			(stroke
 				(width 0.1)
@@
 		)
 		(fp_line
-			(start -1.6 -0.8)
-			(end 1.6 -0.8)
+			(start -1 -0.625)
+			(end 1 -0.625)
 			(stroke
 				(width 0.1)
@@
 		)
 		(fp_text user "${REFERENCE}"
-			(at 0 0 0)
+			(at 0 0 180)
 			(layer "F.Fab")
 			(effects
 				(font
-					(size 0.8 0.8)
-					(thickness 0.12)
+					(size 0.5 0.5)
+					(thickness 0.08)
 				)
 			)
 		)
 		(pad "1" smd roundrect
-			(at -1.5625 0 180)
-			(size 1.325 1.8)
+			(at -1.0375 0 180)
+			(size 1.175 1.45)
 			(layers "F.Cu" "F.Paste" "F.Mask")
-			(roundrect_rratio 0.188679)
+			(roundrect_rratio 0.212766)
 			(net 8 "+3.3VA")
 			(pintype "passive")
 		)
 		(pad "2" smd roundrect
-			(at 1.5625 0 180)
-			(size 1.325 1.8)
+			(at 1.0375 0 180)
+			(size 1.175 1.45)
 			(layers "F.Cu" "F.Paste" "F.Mask")
-			(roundrect_rratio 0.188679)
+			(roundrect_rratio 0.212766)
 			(net 4 "+3.3V")
 			(pintype "passive")
 		)
-		(model "${KICAD8_3DMODEL_DIR}/Capacitor_SMD.3dshapes/C_1206_3216Metric.wrl"
+		(model "${KICAD8_3DMODEL_DIR}/Capacitor_SMD.3dshapes/C_0805_2012Metric.wrl"
 			(offset
 				(xyz 0 0 0)
@@
 		(tags "capacitor handsolder")
 		(property "Reference" "C18"
-			(at 0 -1.68 360)
+			(at 0 -1.68 0)
 			(layer "F.SilkS")
 			(effects
@@
 		)
 		(property "Value" "10n"
-			(at 0 1.68 360)
+			(at 0 1.68 0)
 			(layer "F.Fab")
 			(effects
@@
 		)
 		(fp_text user "${REFERENCE}"
-			(at 0 0 360)
+			(at 0 0 0)
 			(layer "F.Fab")
 			(effects

Commit message: Update
Parts:
- removed C56: 10p, Capacitor_SMD:C_0805_2012Metric_Pad1.18x1.45mm_HandSolder
- removed C57: 1n, Capacitor_SMD:C_0805_2012Metric_Pad1.18x1.45mm_HandSolder
- removed J1: Pin_Headers, Connector_PinHeader_2.54mm:PinHeader_2x06_P2.54mm_Vertical
- removed L8: 51n_LQW18AN51NG0Z, Inductor_SMD:L_0603_1608Metric_Pad1.05x0.95mm_HandSolder
- removed R1, R9: 100R, Resistor_SMD:R_0805_2012Metric_Pad1.20x1.40mm_HandSolder
- removed U5: BGS12WN6E6327, Package_LGA:Infineon_PG-TSNP-6-10_0.7x1.1mm_0.7x1.1mm_P0.4mm
- added C2: 220p_GRM1555C2A221GE01, Capacitor_SMD:C_0805_2012Metric, F.Cu at (175.2, 76.8)
- added C33: 47n_Murata_GCM155R71E473KA55, Capacitor_SMD:C_0805_2012Metric, F.Cu at (147.8, 92.2)
- added C34: 68p_Murata_GCM1555C1H680JA16, Capacitor_SMD:C_0805_2012Metric, F.Cu at (147.7, 94.7)
- added C35: 18p_GJM1555C1H180FB01, Capacitor_SMD:C_0805_2012Metric, F.Cu at (168.5, 86.0)
- added C36: 20p_GJM1555C1H200GB01, Capacitor_SMD:C_0805_2012Metric, F.Cu at (171.6, 87.0)
- added C37: 30p_GJM1555C1H300FB01, Capacitor_SMD:C_0805_2012Metric, F.Cu at (175.3, 87.2)
- added C38: 220p_GRM1555C2A221GE01, Capacitor_SMD:C_0805_2012Metric, F.Cu at (175.2, 85.0)
- added C39: 18p_GJM1555C1H180FB01, Capacitor_SMD:C_0805_2012Metric, F.Cu at (181.9, 86.0)
- added C52: 10p, Capacitor_SMD:C_0805_2012Metric, F.Cu at (210.9, 101.0)
- added C68: 10p, Capacitor_SMD:C_0805_2012Metric, F.Cu at (174.7, 79.7)
- added C69: 1n, Capacitor_SMD:C_0805_2012Metric, F.Cu at (216.1, 111.5)
- added IC1: RF_Switch_PE42440MLBB-Z, Personal_Project:PE42440_QFN50P300X300X80-17N, F.Cu at (182.2, 81.0)
- added J8: Conn_02x05_Odd_Even, Connector_PinHeader_2.54mm:PinHeader_2x05_P2.54mm_Vertical, F.Cu at (220.6, 100.2)
- added L14: 6n8_LQW18AN6N8C00, Inductor_SMD:L_0603_1608Metric_Pad1.05x0.95mm_HandSolder, F.Cu at (165.5, 85.2)
- added L15: 160n_LQW18ANR16G00, Inductor_SMD:L_0603_1608Metric_Pad1.05x0.95mm_HandSolder, F.Cu at (151.8, 92.5)
- added L16: 12n_LQW18AN12NG0Z, Inductor_SMD:L_0603_1608Metric_Pad1.05x0.95mm_HandSolder, F.Cu at (171.5, 85.0)
- added L17: 51n_LQW18AN51NG0Z, Inductor_SMD:L_0603_1608Metric_Pad1.05x0.95mm_HandSolder, F.Cu at (178.8, 85.1)
- added L18: 47n_LQW15AN47NJ00, Inductor_SMD:L_0603_1608Metric_Pad1.05x0.95mm_HandSolder, F.Cu at (169.7, 83.2)
- added L2: 51n_LQW18AN51NG0Z, Inductor_SMD:L_0603_1608Metric_Pad1.05x0.95mm_HandSolder, F.Cu at (178.9, 76.8)
- added R20: 100R, Resistor_SMD:R_0805_2012Metric, F.Cu at (220.5, 120.1)
- added R5: 100R, Resistor_SMD:R_0805_2012Metric, F.Cu at (220.5, 114.2)
- added R6: 100R, Resistor_SMD:R_0805_2012Metric, F.Cu at (220.5, 117.2)
- added SW1: Switch_NX3L1T3157GM,115, Personal_Project:Switch_NX3L1T3157GM115, F.Cu at (163.9, 80.8)
- added SW2: Switch_NX3L1T3157GM,115, Personal_Project:Switch_NX3L1T3157GM115, F.Cu at (154.2, 65.7)
- C1, C10, C11, C12, C13, C14, C15, C16, C18, C19, C3, C40, C41, C42, C43, C46, C47, C48, C5, C50, C51, C53, C58, C59, C60, C61, C62, C63, C64, C65, C66, C67, C7, C8, C9, FB1, FB3: footprint Capacitor_SMD:C_0805_2012Metric_Pad1.18x1.45mm_HandSolder -> Capacitor_SMD:C_0805_2012Metric
- C44: value 47n -> 33p_CC0402GRNPO9BN330; footprint Capacitor_SMD:C_0805_2012Metric_Pad1.18x1.45mm_HandSolder -> Capacitor_SMD:C_0805_2012Metric
- C45: value 68p -> 1n; footprint Capacitor_SMD:C_0805_2012Metric_Pad1.18x1.45mm_HandSolder -> Capacitor_SMD:C_0805_2012Metric
- C49: value 220p_GRM1555C2A221GE01 -> 33p_CC0402GRNPO9BN330; footprint Capacitor_SMD:C_0805_2012Metric_Pad1.18x1.45mm_HandSolder -> Capacitor_SMD:C_0805_2012Metric
- C54: value 10p -> 1n; footprint Capacitor_SMD:C_0805_2012Metric_Pad1.18x1.45mm_HandSolder -> Capacitor_SMD:C_0805_2012Metric
- C55: value 1n -> 10p; footprint Capacitor_SMD:C_0805_2012Metric_Pad1.18x1.45mm_HandSolder -> Capacitor_SMD:C_0805_2012Metric
- L6: value 160n_LQW18ANR16G00 -> 33n_LQW15AN33NG00
- R10, R11, R12, R13, R14, R15, R16, R17, R18, R19, R2, R7, R8: footprint Resistor_SMD:R_0805_2012Metric_Pad1.20x1.40mm_HandSolder -> Resistor_SMD:R_0805_2012Metric
- moved H1 52.0 mm to (105.0, 58.0)
- moved H3 51.5 mm to (105.0, 100.0)
- moved R7 48.9 mm to (106.3, 85.2), turned to 90 degrees
- moved FB3 46.0 mm to (109.8, 84.6), turned to 90 degrees
- moved J16 41.9 mm to (104.9, 78.2), turned to -90 degrees
- moved C67 41.7 mm to (119.8, 84.3), turned to -90 degrees
- moved C66 41.3 mm to (122.3, 84.2), turned to -90 degrees
- moved C63 40.9 mm to (116.2, 83.0), turned to -90 degrees
- moved U3 36.2 mm to (112.2, 78.0), turned to 0 degrees
- moved R10 35.8 mm to (117.3, 79.7), turned to 0 degrees
- moved C9 33.3 mm to (108.9, 73.7), turned to 90 degrees
- moved U7 32.1 mm to (123.0, 77.8), turned to -90 degrees
- moved R11 31.7 mm to (117.3, 76.7), turned to 0 degrees
- moved H2 31.1 mm to (197.0, 59.0)
- moved H4 28.9 mm to (197.0, 100.0)
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Connections:
- net /RF2_3 renamed /RF1_3
- net /RF2_4 renamed /RF1_4
- C44 pad 1: /VR_PA -> GND
- C44 pad 2: GND -> /Y0
- C45 pad 1: /VR_PA -> /VDD
- C49 pad 1: /RF2_2 -> GND
- C49 pad 2: /RF2_1 -> /Y1
- C50 pad 2: /RF2_1 -> /RF1_1
- C54 pad 1: GND -> /V2
- C54 pad 2: /VDD -> GND
- C55 pad 1: GND -> /V1
- C55 pad 2: /VDD -> GND
- J5 pad 2: /PB0 -> /PB4
- L6 pad 1: /VR_PA -> /Y0
- U1 pad 22: unconnected-(U1-RFO_LP-Pad22) -> /RFO_LP
- U1 pad 25: +3.3V -> /VDDPA
- U1 pad 30: /PB0 -> /PB0_CTRL1
- U1 pad 31: /PB2 -> /PB2_CTRL2
Routing:
- net /PB2_CTRL2: track 0.00 -> 8.80 mm, vias 0 -> 1
- net /PB2: track 8.80 -> 0.00 mm, vias 1 -> 0
- net /PB0_CTRL1: track 0.00 -> 8.63 mm, vias 0 -> 1
- net /PB0: track 8.63 -> 0.00 mm, vias 1 -> 0
- net /VR_PA: track 4.42 -> 0.00 mm
- net /RF1_1: track 0.00 -> 1.62 mm
- net /VDD: track 0.00 -> 0.70 mm
- net /RF1: track 0.00 -> 0.50 mm
Other:
- board outline added: 100 x 50 mm

Commit message: Update
Parts:
- removed C53: 33p_GJM0335C1E330JB01D_MURATA, Capacitor_SMD:C_0805_2012Metric
- removed C7: 100n, Capacitor_SMD:C_0805_2012Metric
- removed Y1: Clock_ECS-327MVATX-7-CN-TR, Personal_Project:Clock_ECS327MVATX7CNTR
- removed Y3: ABM3B-32.000MHZ-8-R30-B1U-T, Personal_Project:XTAL_ABM3B-32.000MHZ-10-R30-B1U-T
- added C17: 1p2_GJM1555C1H1R2WB01D, Capacitor_SMD:C_0805_2012Metric, B.Cu at (162.8, 70.5)
- added C20: 33p_NMC0603NPO330J50TRPF, Capacitor_SMD:C_0603_1608Metric, B.Cu at (156.8, 73.4)
- added C21: 33p_NMC0603NPO330J50TRPF, Capacitor_SMD:C_0603_1608Metric, F.Cu at (153.9, 72.6)
- added C22: 3p3_GRM1885C1H3R3CA01D, Capacitor_SMD:C_0603_1608Metric, B.Cu at (153.2, 71.7)
- added C4: 10n, Capacitor_SMD:C_0805_2012Metric, F.Cu at (158.9, 66.2)
- added C6: 10p, Capacitor_SMD:C_0805_2012Metric, F.Cu at (155.9, 72.6)
- added FB2: Murata_BLM21AG102SZ1D, Capacitor_SMD:C_0805_2012Metric, F.Cu at (161.2, 66.2)
- added OS1: Oscillator_ECS-327MVATX-3-CN-TR, Personal_Project:Oscillator_ECS327MVATX3CNTR, F.Cu at (145.4, 71.3)
- added OS2: Oscillator_ECS-TXO-32CSMV-320-AN-TR, Personal_Project:Oscillator_ECSTXO32CSMV320ANTR, F.Cu at (155.2, 66.3)
- added R1: 220R, Resistor_SMD:R_0805_2012Metric, F.Cu at (155.1, 69.6)
- BH1, C11, C33, C34, C41, C42, L15: moved to B.Cu
- C43: value 33p_GJM0335C1E330JB01D_MURATA -> 100n_CL21B104KCFNNNE; moved to B.Cu
- C5: value 33p_GJM0335C1E330JB01D_MURATA -> 33p_NMC0603NPO330J50TRPF; footprint Capacitor_SMD:C_0805_2012Metric -> Capacitor_SMD:C_0603_1608Metric; moved to B.Cu
- C51: value 100n_FCC0402KRX7R7BB104 -> 47p_KGQ21HCG2D470JT; moved to B.Cu
- moved BH1 103.6 mm to (127.2, 34.3), turned to -90 degrees
- moved R5 62.8 mm to (169.1, 78.2)
- moved J8 61.8 mm to (176.3, 57.2), turned to -90 degrees
- moved C14 54.0 mm to (123.7, 60.5)
- moved C16 54.0 mm to (123.7, 66.6)
- moved LDO1 54.0 mm to (123.3, 63.8)
- moved C8 53.7 mm to (118.0, 100.4)
- moved U2 53.7 mm to (111.2, 101.7)
- moved J6 44.2 mm to (104.9, 63.8)
- moved R6 43.5 mm to (185.1, 91.9)
- moved J3 42.3 mm to (107.0, 93.1)
- moved J11 41.2 mm to (113.5, 64.7)
- moved R20 41.1 mm to (194.1, 88.7)
- moved J15 39.1 mm to (114.4, 91.3)
- moved C1 34.7 mm to (100.3, 81.5)
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Connections:
- C43 pad 1: +3.3V -> /PB0_VDD_TCXO
- C51 pad 1: +3.3V -> /PB0_VDD_TCXO
- R20 pad 1: /PB0_CTRL1 -> /PB4_CTRL1
- SW1 pad 6: /PB0_CTRL1 -> /PB4_CTRL1
- SW2 pad 6: /PB0_CTRL1 -> /PB4_CTRL1
- U1 pad 2: /PB4 -> /PB4_CTRL1
- U1 pad 30: /PB0_CTRL1 -> /PB0_VDD_TCXO
Routing:
- net +3.3V: track 19.6 -> 61.9 mm, vias 0 -> 4
- net /PB0_VDD_TCXO: track 0.00 -> 24.8 mm, vias 0 -> 2
- net /VR_PA: track 0.00 -> 15.8 mm, vias 0 -> 1
- net /PA15: track 0.00 -> 13.7 mm
- net /VDDPA: track 0.00 -> 13.5 mm, vias 0 -> 2
- net /PH1-OSC_OUT: track 10.3 -> 0.00 mm
- net /PC15-OSC32_OUT: track 20.2 -> 10.6 mm
- net /PB0_CTRL1: track 8.63 -> 0.00 mm, vias 1 -> 0
- net /PA13_SWDIO: track 19.0 -> 10.9 mm
- net /Y1: track 0.00 -> 6.06 mm
- net /Y0: track 0.00 -> 6.06 mm
- net /PB2_CTRL2: track 8.80 -> 3.60 mm, vias 1 -> 0
- net /PB12: track 8.74 -> 3.66 mm, vias 1 -> 0
- net Net-(OS2-VDD): track 0.00 -> 4.90 mm
- net /VLXSMPS: track 0.00 -> 4.66 mm
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- added copper zone on B.Cu, net GND
- added copper zone on F.Cu, net GND
- added copper zone on In1.Cu, net GND
- added copper zone on In2.Cu, net GND
Other:
- outline, holes or cut-outs redrawn

Commit message: Update
Parts:
- removed J11, J15: Power Select Jumpers, Personal_Project:PinHeader_2x03_P2.54mm_Vertical_PINS
- added J1: 3V_Selection_Header, Connector_PinHeader_2.54mm:PinHeader_1x03_P2.54mm_Vertical, F.Cu at (114.2, 90.5)
- added J7: 5V_Selection_Header, Connector_PinHeader_2.54mm:PinHeader_1x03_P2.54mm_Vertical, F.Cu at (113.5, 61.5)
- added SHLD1: RFShield_OnePiece, Personal_Project:RF_Shield_MS631-10F, F.Cu at (148.3, 67.5)
- C2: value 220p_GRM1555C2A221GE01 -> 68p_GRM1555C2A221GE01
- C46: value 20p_GJM1555C1H200GB01 -> 2p2_GJM1555C1H200GB01
- C47, C50: value 18p_GJM1555C1H180FB01 -> 1p2_GJM1555C1H180FB01
- C48: value 30p_GJM1555C1H300FB01 -> 5p6_GJM1555C1H300FB01
- C58: value 220p_GRM1555C2A221GE01 -> 33p_GRM1555C2A221GE01
- C59, C60: value 22p_GJM1555C1H220FB01 -> 3p3_GJM1555C1H220FB01
- C61: value 15p_GJM1555C1H150FB01 -> 3p6_GJM1555C1H150FB01
- C62: value 18p_GJM1555C1H120FB01 -> 2p7_GJM1555C1H120FB01
- FB3: moved to B.Cu
- L10: value 120n_LQW18ANR12G00 -> 11n_LQW18ANR12G00
- L2: value 51n_LQW18AN51NG0Z -> 8n7_LQW18AN51NG0Z
- L7: value 12n_LQW18AN12NG0Z -> 3n6_LQW18AN12NG0Z
- L9: value 47n_LQW18AN47NG0Z -> 8n7_LQW18AN47NG0Z
- moved J8 54.3 mm to (139.4, 96.9)
- moved BH1 45.8 mm to (130.7, 80.0)
- moved J17 36.7 mm to (121.9, 94.3)
- moved R8 31.2 mm to (124.8, 91.0)
- moved J4 27.3 mm to (120.0, 66.4), turned to 180 degrees
- moved C1 20.9 mm to (117.2, 93.8), turned to -90 degrees
- moved ESD2 20.8 mm to (111.4, 86.2)
- moved J5 19.5 mm to (120.6, 57.5), turned to 90 degrees
- moved C3 18.9 mm to (117.4, 57.5)
- moved ESD1 17.1 mm to (108.9, 64.8), turned to 180 degrees
- moved U6 16.9 mm to (110.5, 59.1)
- moved J10 15.2 mm to (147.6, 100.3)
- moved R16 15.2 mm to (151.8, 96.2)
- moved R18 15.2 mm to (157.7, 96.2)
- moved R19 15.2 mm to (160.6, 96.2)
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Connections:
- ESD1 pad 1: /5V_SW -> unconnected-(ESD1-I/O1-Pad1)
- ESD1 pad 4: /VBUS_5V -> /EXT_5V
- ESD1 pad 5: /PC_5V -> /VBUS_5V
- ESD2 pad 1: /PC_3V3 -> unconnected-(ESD2-I/O1-Pad1)
- ESD2 pad 4: /3V3_SW -> /EXT_3V
- J3 pad 1: /5V_SW -> GND
- J3 pad 7: /3V3_SW -> GND
- J6 pad 1: /PC_5V -> /EXT_5V
- J6 pad 3: /PC_3V3 -> /EXT_3V
Routing:
- net /VFBSMPS: track 9.06 -> 67.5 mm, vias 0 -> 2
- net /PB6_USART1_TX: track 0.00 -> 40.9 mm, vias 0 -> 2
- net /PA10_USART1_RX: track 8.30 -> 35.8 mm, vias 0 -> 4
- net /PA11_USART1_CTS: track 8.53 -> 34.8 mm, vias 0 -> 2
- net /PA12_USART1_RTS: track 8.62 -> 30.5 mm, vias 0 -> 2
- net /VBUS_5V: track 0.00 -> 17.0 mm, vias 0 -> 2
- net /VBUS_5V_FB: track 0.00 -> 15.3 mm, vias 0 -> 1
- net +5V: track 0.00 -> 13.0 mm
- net /RFIN_2: track 0.00 -> 11.3 mm
- net Net-(U7-3V3OUT): track 0.00 -> 10.6 mm
- net Net-(J5-Pin_1): track 0.00 -> 7.78 mm
- net /EXT_5V: track 0.00 -> 7.23 mm
- net /PB2_CTRL2: track 3.60 -> 10.6 mm
- net /PB12: track 3.66 -> 10.4 mm
- net GND: track 2.39 -> 8.93 mm, vias 0 -> 18
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Other:
- board text added: "3V3/VBAT/BAT"
- board text added: "5V/GN/3V3/GN"
- board text added: "EX3V3/LDO"
- board text added: "EX5V/VBS"
- board text added: "NR/SWO/CL/SWD"
- board text added: "NRST"
- board text added: "PC5V"
- board text added: "USR BTN"

Commit message: Update
Parts:
- removed ESD2: ESDALC6V1W5, Personal_Project:SOT323-5L_STM-L
- removed J10: SPI1_Headers, Connector_PinHeader_2.54mm:PinHeader_1x06_P2.54mm_Vertical
- removed R14, R15, R17, R18, R19: 100R, Resistor_SMD:R_0805_2012Metric
- added J11: SPI1_Headers, Connector_PinHeader_2.54mm:PinHeader_2x05_P2.54mm_Horizontal, F.Cu at (175.1, 97.8)
- added R3: 33R, Resistor_SMD:R_0805_2012Metric, B.Cu at (171.0, 93.0)
- added R4: 33R, Resistor_SMD:R_0805_2012Metric, B.Cu at (173.5, 93.0)
- added R9: 33R, Resistor_SMD:R_0805_2012Metric, B.Cu at (176.0, 93.0)
- C10, C12, C13, C15, C45, C52, C54, C55, C68, C69, FB1, R20, R5, R6: moved to B.Cu
- C11: moved to F.Cu
- J2: value LPUART1_Headers -> I2C1_Headers; footprint Connector_PinHeader_2.54mm:PinHeader_1x04_P2.54mm_Vertical -> Connector_PinHeader_2.54mm:PinHeader_2x03_P2.54mm_Horizontal
- J3: footprint Connector_PinHeader_2.54mm:PinHeader_2x04_P2.54mm_Vertical -> Connector_PinHeader_2.54mm:PinHeader_2x04_P2.54mm_Horizontal
- J8: footprint Connector_PinHeader_2.54mm:PinHeader_2x05_P2.54mm_Vertical -> Connector_PinHeader_2.54mm:PinHeader_2x05_P2.54mm_Horizontal
- J9: value I2C1_Headers -> LPUART1_Headers; footprint Connector_PinHeader_2.54mm:PinHeader_1x04_P2.54mm_Vertical -> Connector_PinHeader_2.54mm:PinHeader_2x03_P2.54mm_Horizontal
- R12, R13, R16: value 100R -> 33R; moved to B.Cu
- moved C69 26.7 mm to (175.7, 79.5)
- moved J2 24.3 mm to (157.6, 97.8), turned to -90 degrees
- moved C55 22.5 mm to (175.7, 81.8), turned to 0 degrees
- moved R6 20.0 mm to (165.9, 81.5), turned to 90 degrees
- moved R20 19.0 mm to (175.7, 84.1), turned to 180 degrees
- moved C54 18.1 mm to (170.5, 81.5)
- moved C52 17.2 mm to (168.2, 81.5), turned to -90 degrees
- moved R16 17.1 mm to (168.5, 93.0)
- moved J9 14.1 mm to (188.5, 97.8)
- moved C15 10.8 mm to (136.5, 82.5), turned to -90 degrees
- moved J8 4.81 mm to (144.1, 97.8)
- moved FB1 4.71 mm to (136.5, 78.8), turned to -90 degrees
- moved C19 4.68 mm to (135.8, 67.3), turned to 180 degrees
- moved ESD1 4.52 mm to (108.4, 69.3), turned to -90 degrees
- moved R5 4.44 mm to (165.6, 76.1), turned to 90 degrees
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Connections:
- ESD1 pad 3: unconnected-(ESD1-I/O2-Pad3) -> /EXT_5V
- ESD1 pad 4: /EXT_5V -> /EXT_3V
- J1 pad 1: /EXT_3V -> /LD_OUT_3V3
- J1 pad 3: /LD_OUT_3V3 -> /EXT_3V
- J2 pad 3: Net-(J2-Pin_3) -> /PB7_I2C1_SDA
- J2 pad 4: Net-(J2-Pin_4) -> GND
- J3 pad 2: /PA13_SWDIO -> /PA14_SWCLK
- J3 pad 4: /PA14_SWCLK -> /PB3_SWO
- J3 pad 6: /PB3_SWO -> /NRST
- J3 pad 8: /NRST -> /PA13_SWDIO
- J5 pad 2: /PB4 -> /PB12_USR_BTN
- J8 pad 1: /PA0 -> GND
- J8 pad 2: /PA5 -> /PA0
- J8 pad 3: /PA7 -> GND
- J8 pad 5: /PA9 -> GND
- J8 pad 7: /PB4 -> GND
- J8 pad 8: /PB12 -> /PB12_USR_BTN
- J8 pad 9: /PC15-OSC32_OUT -> GND
- J9 pad 1: +3.3V -> GND
- J9 pad 2: GND -> Net-(J9-Pin_2)
- J9 pad 3: Net-(J9-Pin_3) -> GND
- R12 pad 2: Net-(J2-Pin_3) -> Net-(J9-Pin_4)
- R13 pad 2: Net-(J2-Pin_4) -> Net-(J9-Pin_2)
- R20 pad 1: /PB4_CTRL1 -> /PA7_HPLP_CTRL
- R6 pad 1: /PB2_CTRL2 -> /PA5_INOUTRF
- SW1 pad 6: /PB4_CTRL1 -> /PA7_HPLP_CTRL
- SW2 pad 6: /PB4_CTRL1 -> /PB2_RFVCTRL
- U1 pad 13: /PA5 -> /PA5_INOUTRF
- U1 pad 14: /PA6_SPI1_MISO -> unconnected-(U1-PA6-Pad14)
- U1 pad 15: /PA7 -> /PA7_HPLP_CTRL
- U1 pad 17: /PA9 -> unconnected-(U1-PA9-Pad17)
- U1 pad 2: /PB4_CTRL1 -> /PB4_SPI1_MISO
- U1 pad 31: /PB2_CTRL2 -> /PB2_RFVCTRL
- U1 pad 32: /PB12 -> /PB12_USR_BTN
Routing:
- net +3.3V: track 60.5 -> 209.5 mm, vias 4 -> 14
- net /NRST: track 0.00 -> 88.9 mm, vias 0 -> 2
- net /PA13_SWDIO: track 10.9 -> 81.1 mm, vias 1 -> 2
- net /PB3_SWO: track 0.00 -> 68.1 mm, vias 0 -> 1
- net /PA14_SWCLK: track 14.9 -> 82.3 mm, vias 0 -> 1
- net /BOOT0: track 0.00 -> 49.1 mm, vias 0 -> 2
- net /PA7_HPLP_CTRL: track 0.00 -> 39.6 mm, vias 0 -> 2
- net /PB12_USR_BTN: track 0.00 -> 34.2 mm, vias 0 -> 2
- net /EXT_3V: track 0.00 -> 31.9 mm, vias 0 -> 1
- net /PA8_MCO: track 0.00 -> 27.7 mm, vias 0 -> 1
- net /RF1: track 0.00 -> 25.9 mm
- net /LD_OUT_3V3: track 1.95 -> 24.1 mm, vias 0 -> 1
- net /PA5_INOUTRF: track 0.00 -> 21.0 mm, vias 0 -> 2
- net /VBAT: track 13.6 -> 33.4 mm, vias 0 -> 2
- net /RFI_P: track 0.00 -> 16.0 mm
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Other:
- board size 100 x 50 mm -> 100 x 51 mm
- board text added: "BAT/3V3"
- board text added: "BT/PB12"
- board text added: "GN/BT/3V3"
- board text added: "LD/EX3"
- board text added: "USRBT"
- board text removed: "3V3/VBAT/BAT"
- board text removed: "EX3V3/LDO"
- board text removed: "PC5V"
- board text removed: "USR BTN"
