File: LoRa_Board.kicad_pcb (KiCad board)
At the start: 4 copper layers, 100 x 51 mm, 117 parts, among them IC1 RF_Switch_PE42440MLBB-Z, J1 3V_Selection_Header, J11 SPI1_Headers, J16 USB_B_Micro, J17 BOOT0_Jumper, J19 SMA PCB END LAUNCH JACK ROUND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, J2 I2C1_Headers, J3 Debug_Pins, J4 Coin Battery Jumper, J5 User Button Jumper, J6 Power Pins, J7 5V_Selection_Header, J8 Conn_02x05_Odd_Even, J9 LPUART1_Headers, SW1 Switch_NX3L1T3157GM,115, SW2 Switch_NX3L1T3157GM,115, U1 STM32WL55CCU6, U3 USBLC6-2SC6, U7 FT230XS

Commit message: Update
Parts:
- removed ESD1: ESDALC6V1W5, Personal_Project:SOT323-5L_STM-L
- removed J11: SPI1_Headers, Connector_PinHeader_2.54mm:PinHeader_2x05_P2.54mm_Horizontal
- removed J7: 5V_Selection_Header, Connector_PinHeader_2.54mm:PinHeader_1x03_P2.54mm_Vertical
- removed J8: Conn_02x05_Odd_Even, Connector_PinHeader_2.54mm:PinHeader_2x05_P2.54mm_Horizontal
- removed R16, R4, R9: 33R, Resistor_SMD:R_0805_2012Metric
- added ESD2: ESDALC6V1W5, Personal_Project:SOT323-5L_STM-L, F.Cu at (108.4, 69.4)
- added J10: 3V_Selection_Header, Connector_PinHeader_2.54mm:PinHeader_1x03_P2.54mm_Vertical, F.Cu at (113.0, 90.7)
- added J12: 5V_Selection_Header, Connector_PinHeader_2.54mm:PinHeader_1x03_P2.54mm_Vertical, F.Cu at (111.9, 62.2)
- added R14: 33R, Resistor_SMD:R_0805_2012Metric, B.Cu at (180.6, 99.0)
- added R15: 33R, Resistor_SMD:R_0805_2012Metric, B.Cu at (163.8, 98.5)
- added S1: Switch_WS-SLSU SMT Mini Slide, Personal_Project:Switch_WS-SLSU SMT Mini Slide, F.Cu at (115.5, 102.0)
- C1: moved to B.Cu
- J1: value 3V_Selection_Header -> SPI1_Headers; footprint Connector_PinHeader_2.54mm:PinHeader_1x03_P2.54mm_Vertical -> Connector_PinHeader_2.54mm:PinHeader_2x04_P2.54mm_Horizontal
- J5: value User Button Jumper -> General_Pin_Header; footprint Connector_PinHeader_2.54mm:PinHeader_1x02_P2.54mm_Vertical -> Connector_PinHeader_2.54mm:PinHeader_2x03_P2.54mm_Horizontal
- moved J1 62.2 mm to (174.8, 97.9), turned to -90 degrees
- moved J5 45.6 mm to (142.2, 97.9), turned to -90 degrees
- moved R12 20.6 mm to (168.6, 103.2), turned to 180 degrees
- moved U2 12.3 mm to (124.2, 102.8)
- moved C8 12.2 mm to (131.1, 101.2)
- moved R13 7.72 mm to (181.6, 95.2), turned to 0 degrees
- moved R3 5.84 mm to (165.5, 95.0), turned to 0 degrees
- moved C1 2.02 mm to (116.2, 92.2), turned to 90 degrees
- moved C10 0.60 mm to (146.2, 84.2)
- moved J2 0.37 mm to (157.2, 97.9)
- moved J9 0.21 mm to (188.7, 97.8)
Connections:
- C3 pad 2: Net-(J5-Pin_1) -> /PB12_USR_BTN
- J1 pad 1: /LD_OUT_3V3 -> +3.3V
- J1 pad 2: +3.3V -> GND
- J1 pad 3: /EXT_3V -> GND
- J2 pad 3: /PB7_I2C1_SDA -> GND
- J2 pad 4: GND -> /PB7_I2C1_SDA
- J5 pad 1: Net-(J5-Pin_1) -> GND
- J5 pad 2: /PB12_USR_BTN -> /PA8_MCO
- J9 pad 1: GND -> +3.3V
- J9 pad 2: Net-(J9-Pin_2) -> GND
- J9 pad 5: GND -> Net-(J9-Pin_5)
- J9 pad 6: +3.3V -> GND
- R12 pad 1: /PA2_LPUART1_TX -> Net-(J1-Pin_4)
- R12 pad 2: Net-(J9-Pin_4) -> /PB4_SPI1_MISO
- R13 pad 2: Net-(J9-Pin_2) -> Net-(J9-Pin_5)
- R3 pad 1: /PA4_SPI1_NSS -> /PB5_SPI1_MOSI
- R3 pad 2: Net-(J11-Pin_5) -> Net-(J1-Pin_5)
- U1 pad 38: /PC13 -> unconnected-(U1-PC13-Pad38)
- U1 pad 43: /PA15 -> unconnected-(U1-PA15-Pad43)
- U6 pad 1: Net-(J5-Pin_1) -> /PB12_USR_BTN
- U6 pad 2: Net-(J5-Pin_1) -> /PB12_USR_BTN
Routing:
- net +3.3V: track 209.5 -> 337.1 mm, vias 14 -> 15
- net /PB4_SPI1_MISO: track 7.40 -> 47.1 mm
- net /PA2_LPUART1_TX: track 10.2 -> 48.7 mm
- net /PA3_LPUART1_RX: track 10.3 -> 45.6 mm
- net /PB7_I2C1_SDA: track 12.9 -> 40.5 mm
- net /PB5_SPI1_MOSI: track 5.85 -> 33.2 mm
- net /PA1_SPI1_SCK: track 9.53 -> 33.4 mm
- net /PA0: track 10.1 -> 27.5 mm
- net /PB8_I2C1_SCL: track 11.4 -> 28.1 mm
- net /PC13: track 14.3 -> 0.00 mm
- net /PB12_USR_BTN: track 34.2 -> 44.5 mm
- net /PA4_SPI1_NSS: track 13.5 -> 23.7 mm
- net Net-(J9-Pin_4): track 0.00 -> 8.99 mm
- net /PA15: track 8.77 -> 0.00 mm
- net Net-(J10-Pin_2): track 0.00 -> 8.54 mm
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Other:
- board text added: "CK/MO/MI/3V3"
- board text added: "I2C1"
- board text added: "LPUART1"
- board text added: "NR/SO/CL/SD"
- board text added: "ON/OFF"
- board text added: "PA0"
- board text added: "PA8MCO"
- board text added: "RX/TX/3V3"
- board text added: "SCL/SDA/3V3"
- board text added: "SPI1"
- board text added: "SPINSS"
- board text removed: "BT/PB12"
- board text removed: "NR/SWO/CL/SWD"

Commit message: update
Parts:
- removed C1: 4u7, Capacitor_SMD:C_0805_2012Metric
- removed ESD2: ESDALC6V1W5, Personal_Project:SOT323-5L_STM-L
- added C23: 4u7, Capacitor_SMD:C_0603_1608Metric_Pad1.08x0.95mm_HandSolder, B.Cu at (116.6, 91.5)
- added D1: BZX84C4V3LT1G, Package_TO_SOT_SMD:SOT-23, B.Cu at (113.6, 63.8)
- added D2: BZX84C6V2LT1G, Package_TO_SOT_SMD:SOT-23, B.Cu at (113.7, 71.0)
- added Q2: MOSFET_SI2333DDS-T1-BE3, Personal_Project:MOSFET_ SI2333DDS_SOT_DS-T1-BE3_VIS, B.Cu at (109.7, 63.8)
- added R4: 100k, Resistor_SMD:R_0603_1608Metric_Pad0.98x0.95mm_HandSolder, B.Cu at (110.5, 59.6)
- added Z2: Diode_BZX84C6V2-7-F, Personal_Project:Diode_BZX84C6V2_SOT96P240X110-3N, B.Cu at (113.5, 59.5)
- J10: value 3V_Selection_Header -> Power_Selector_Jumper; footprint Connector_PinHeader_2.54mm:PinHeader_1x03_P2.54mm_Vertical -> Connector_PinHeader_2.54mm:PinHeader_2x03_P2.54mm_Vertical
- J12: value 5V_Selection_Header -> 3V_Selection_Header
- J6: value Power Pins -> JST_XH_2.54_Plug; footprint Connector_PinHeader_2.54mm:PinHeader_1x04_P2.54mm_Vertical -> Personal_Project:Connector_Power2pin_SHDRRA2W80P0X250_1X2_740X1150X610P
- moved J12 33.6 mm to (113.8, 95.7), turned to 180 degrees
- moved J10 28.9 mm to (117.3, 62.1)
- moved C15 14.7 mm to (150.7, 78.5), turned to 0 degrees
- moved FB1 11.8 mm to (147.8, 75.5), turned to 90 degrees
- moved J4 9.63 mm to (119.7, 57.6), turned to 90 degrees
- moved J6 7.84 mm to (109.7, 70.3), turned to 90 degrees
- moved C12 6.63 mm to (143.1, 75.5)
- moved C13 6.63 mm to (145.5, 75.5)
- moved C14 0.95 mm to (117.8, 70.5)
- moved C16 0.95 mm to (117.8, 73.0)
- moved LDO1 0.95 mm to (113.9, 71.7)
- moved C3 0.94 mm to (116.5, 57.8), turned to -90 degrees
- moved U6 0.94 mm to (109.6, 59.4)
- moved L15 0.87 mm to (153.6, 71.3)
- moved C17 0.75 mm to (155.9, 67.6)
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Connections:
- C14 pad 1: +5V -> /LDO_IN
- J10 pad 1: /LD_OUT_3V3 -> /EXT_POWER+_PP
- J10 pad 2: Net-(J10-Pin_2) -> /EXT_POWER+_NOLDO
- J10 pad 3: /EXT_3V -> /EXT_POWER+_PP
- J12 pad 1: /EXT_5V -> /EXT_POWER+_NOLDO
- J12 pad 2: +5V -> /POWER_3V3
- J12 pad 3: /VBUS_5V -> /LD_OUT_3V3
- J6 pad 1: /EXT_5V -> GND
- J6 pad 2: GND -> /EXT_POWER+
- LDO1 pad 1: +5V -> /LDO_IN
- LDO1 pad 3: +5V -> /LDO_IN
- S1 pad 1: Net-(J10-Pin_2) -> /POWER_3V3
Routing:
- net /EXT_POWER+_NOLDO: track 0.00 -> 41.9 mm
- net /EXT_3V: track 31.1 -> 0.00 mm, vias 1 -> 0
- net /LDO_IN: track 0.00 -> 20.0 mm, vias 0 -> 1
- net /EXT_5V: track 17.8 -> 0.00 mm
- net /POWER_3V3: track 0.00 -> 14.7 mm, vias 0 -> 1
- net +5V: track 13.3 -> 0.00 mm
- net +3.3V: track 337.1 -> 323.8 mm, vias 15 -> 14
- net Net-(J10-Pin_2): track 8.54 -> 0.00 mm
- net /VBAT: track 33.5 -> 36.9 mm, vias 2 -> 1
- net /VBUS_5V: track 28.1 -> 31.1 mm
- net /PA5_INOUTRF: track 21.0 -> 22.8 mm
- net /VDDPA: track 15.0 -> 16.8 mm
- net /PB6_USART1_TX: track 39.9 -> 41.7 mm
- net /PA10_USART1_RX: track 33.9 -> 35.5 mm
- net /PB12_USR_BTN: track 44.5 -> 45.9 mm
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- added copper zone on B.Cu, net /EXT_POWER+
- added copper zone on B.Cu, net /EXT_POWER+_PP
- added copper zone on B.Cu, net /MOSFET_GATE
Other:
- board text added: "V+"
- board text removed: "5V/GN/3V3/GN"
- board text removed: "EX5V/VBS"
