File: LoRa_Board.kicad_pcb (KiCad board)
At the start: 4 copper layers, 100 x 51 mm, 120 parts, among them IC1 RF_Switch_PE42440MLBB-Z, J1 SPI1_Headers, J10 Power_Selector_Jumper, J12 3V_Selection_Header, J16 USB_B_Micro, J17 BOOT0_Jumper, J19 SMA PCB END LAUNCH JACK ROUND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, J2 I2C1_Headers, J3 Debug_Pins, J4 Coin Battery Jumper, J5 General_Pin_Header, J6 JST_XH_2.54_Plug, J9 LPUART1_Headers, Q2 MOSFET_SI2333DDS-T1-BE3, SW1 Switch_NX3L1T3157GM,115, SW2 Switch_NX3L1T3157GM,115, U1 STM32WL55CCU6, U3 USBLC6-2SC6, U7 FT230XS

Commit message: Update
Parts:
- removed C23: 4u7, Capacitor_SMD:C_0603_1608Metric_Pad1.08x0.95mm_HandSolder
- removed D1: BZX84C4V3LT1G, Package_TO_SOT_SMD:SOT-23
- removed D2: BZX84C6V2LT1G, Package_TO_SOT_SMD:SOT-23
- removed J10: Power_Selector_Jumper, Connector_PinHeader_2.54mm:PinHeader_2x03_P2.54mm_Vertical
- removed J12: 3V_Selection_Header, Connector_PinHeader_2.54mm:PinHeader_1x03_P2.54mm_Vertical
- removed J16: USB_B_Micro, Connector_USB:USB_Micro-B_Molex-105017-0001
- removed J18: ~, Personal_Project:SMA Clip Mount Adapter (bottom)
- removed J6: JST_XH_2.54_Plug, Personal_Project:Connector_Power2pin_SHDRRA2W80P0X250_1X2_740X1150X610P
- removed Q2: MOSFET_SI2333DDS-T1-BE3, Personal_Project:MOSFET_ SI2333DDS_SOT_DS-T1-BE3_VIS
- removed R12, R13, R14, R15: 33R, Resistor_SMD:R_0805_2012Metric
- removed R4: 100k, Resistor_SMD:R_0603_1608Metric_Pad0.98x0.95mm_HandSolder
- removed S1: Switch_WS-SLSU SMT Mini Slide, Personal_Project:Switch_WS-SLSU SMT Mini Slide
- removed Z2: Diode_BZX84C6V2-7-F, Personal_Project:Diode_BZX84C6V2_SOT96P240X110-3N
- added C1: 4u7, Capacitor_SMD:C_0805_2012Metric, B.Cu at (116.7, 91.7)
- added D3: ESD_TSD05DYFR, Personal_Project:ESD_TSD05DYFR_SOD2613X100N, B.Cu at (114.1, 63.9)
- added D4: ESD_TSD03DYFR, Personal_Project:ESD_TSD05DYFR_SOD2613X100N, F.Cu at (124.5, 64.7)
- added J11: I2C1_Headers, Connector_PinHeader_2.54mm:PinHeader_2x03_P2.54mm_Horizontal, F.Cu at (159.3, 97.9)
- added J13: SPI1_Headers, Connector_PinHeader_2.54mm:PinHeader_2x03_P2.54mm_Horizontal, F.Cu at (174.0, 97.9)
- added J7: LPUART1_Headers, Connector_PinHeader_2.54mm:PinHeader_2x03_P2.54mm_Horizontal, F.Cu at (188.7, 97.9)
- added J8: USB_B_Micro, Connector_USB:USB_Micro-B_XKB_U254-051T-4BH83-F1S, F.Cu at (103.2, 78.7)
- added Q1: MOSFET_SI2333DDS-T1-BE3, Personal_Project:MOSFET_ SI2333DDS_SOT_DS-T1-BE3_VIS, B.Cu at (109.7, 63.8)
- added R16: 33R, Resistor_SMD:R_0805_2012Metric, B.Cu at (180.6, 94.4)
- added R17: 33R, Resistor_SMD:R_0805_2012Metric, B.Cu at (177.1, 100.6)
- added R18: 33R, Resistor_SMD:R_0805_2012Metric, B.Cu at (165.1, 97.9)
- added R25: 33R, Resistor_SMD:R_0805_2012Metric, B.Cu at (168.4, 95.0)
- added R9: 33R, Resistor_SMD:R_0805_2012Metric, B.Cu at (178.4, 94.4)
- added S2: Switch_WS-SLSU SMT Mini Slide, Personal_Project:Switch_WS-SLSU SMT Mini Slide, F.Cu at (115.4, 102.0)
- added Z1: Diode_BZX84C6V2-7-F, Personal_Project:Diode_BZX84C6V2_SOT96P240X110-3N, B.Cu at (113.4, 59.8)
- C11: moved to B.Cu
- IC1: footprint Personal_Project:PE42440_QFN50P300X300X80-17N -> Personal_Project:RF_SWITCH_PE42440_QFN50P300X300X80-17N
- J1: value SPI1_Headers -> JST_XH_2.54_Plug; footprint Connector_PinHeader_2.54mm:PinHeader_2x04_P2.54mm_Horizontal -> Personal_Project:Connector_Power2pin_SHDRRA2W80P0X250_1X2_740X1150X610P
- J2: value I2C1_Headers -> Power_Selector_Jumper; footprint Connector_PinHeader_2.54mm:PinHeader_2x03_P2.54mm_Horizontal -> Connector_PinHeader_2.54mm:PinHeader_2x03_P2.54mm_Vertical
- J9: value LPUART1_Headers -> 3V_Selection_Header; footprint Connector_PinHeader_2.54mm:PinHeader_2x03_P2.54mm_Horizontal -> Connector_PinHeader_2.54mm:PinHeader_1x03_P2.54mm_Vertical
- R3: value 33R -> 100k
- moved J9 75.0 mm to (113.8, 95.8), turned to 180 degrees
- moved J1 70.7 mm to (109.7, 70.3), turned to 90 degrees
- moved R3 65.5 mm to (110.3, 59.8), turned to 90 degrees
- moved J2 53.6 mm to (117.3, 62.1), turned to 0 degrees
- moved C11 3.31 mm to (138.7, 75.4), turned to 90 degrees
- moved J5 2.20 mm to (144.4, 97.9)
- moved C12 0.56 mm to (143.7, 75.5)
- moved C13 0.56 mm to (146.0, 75.5)
- moved FB1 0.56 mm to (148.4, 75.5)
Connections:
- net /VBUS_5V_FB renamed /+5V_VBUS_FB
- J1 pad 1: +3.3V -> GND
- J1 pad 2: GND -> /EXT_POWER+
- J2 pad 1: +3.3V -> /EXT_POWER+_PP
- J2 pad 2: GND -> /EXT_POWER+_NOLDO
- J2 pad 3: GND -> /EXT_POWER+_PP
- J2 pad 4: /PB7_I2C1_SDA -> /LDO_IN
- J2 pad 5: /PB8_I2C1_SCL -> /VBUS_5V
- J2 pad 6: GND -> /LDO_IN
- J9 pad 1: +3.3V -> /EXT_POWER+_NOLDO
- J9 pad 2: GND -> /POWER_3V3
- J9 pad 3: GND -> /LD_OUT_3V3
- R3 pad 1: /PB5_SPI1_MOSI -> /MOSFET_GATE
- R3 pad 2: Net-(J1-Pin_5) -> GND
Routing:
- net Net-(J7-Pin_1): track 0.00 -> 26.1 mm
- net GND: track 20.2 -> 45.8 mm, vias 220 -> 223
- net +3.3V: track 323.8 -> 298.5 mm, vias 14 -> 16
- net /PB7_I2C1_SDA: track 40.5 -> 57.5 mm
- net /PB4_SPI1_MISO: track 47.1 -> 58.4 mm
- net Net-(J9-Pin_4): track 8.99 -> 0.00 mm
- net Net-(J13-Pin_4): track 0.00 -> 8.72 mm
- net Net-(J1-Pin_5): track 5.55 -> 0.00 mm
- net /EXT_POWER+_NOLDO: track 41.9 -> 47.2 mm, vias 0 -> 1
- net Net-(J7-Pin_5): track 0.00 -> 4.99 mm
- net Net-(J1-Pin_4): track 4.92 -> 0.00 mm
- net Net-(J13-Pin_1): track 0.00 -> 4.45 mm
- net Net-(J1-Pin_8): track 4.11 -> 0.00 mm
- net Net-(J9-Pin_5): track 3.52 -> 0.00 mm
- net /PA2_LPUART1_TX: track 48.9 -> 45.7 mm
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Other:
- board text added: "MCU: STM32WL55CCU6 VIN:"

Commit message: Update
Parts:
- added G***: LOGO, Personal_Project:PCB_Logo, B.Cu at (192.0, 89.0)
- moved D4 1.49 mm to (125.4, 65.8), turned to -90 degrees
Other:
- board text added: "CK/MO/MI"
- board text added: "MCU: STM32WL55CCU6 VIN: 1.45V to 5.5V WLDO POWER: EXT, VBUS"
- board text added: "NOLDO"
- board text added: "RX"
- board text added: "SCL"
- board text added: "SDA"
- board text added: "TX"
- board text added: "VBUS"
- board text added: "WLD"
- board text removed: "CK/MO/MI/3V3"
- board text removed: "MCU: STM32WL55CCU6 VIN:"
- board text removed: "RX/TX/3V3"
- board text removed: "SCL/SDA/3V3"

Commit message: Update
Routing:
- net /RFI_P: track 16.0 -> 17.1 mm
- net /RFI_N: track 14.7 -> 15.6 mm
- net GND: vias 223 -> 231
Other:
- board text added: "LORA TRANCEIVER BOARD MCU: STM32WL55CCU6 VIN: 1.45V to 5.5V WLDO POWER: EXT, VBUS"
- board text removed: "MCU: STM32WL55CCU6 VIN: 1.45V to 5.5V WLDO POWER: EXT, VBUS"
Changed lines of the file:
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@@
 		(tags "capacitor")
 		(property "Reference" "C35"
-			(at -1.1 -2.8 180)
+			(at -0.9 -5.8 180)
 			(layer "F.SilkS")
 			(effects
@@
 		(tags "capacitor")
 		(property "Reference" "C13"
-			(at -3.94 0.035 90)
+			(at -3.34 0.0725 -90)
 			(layer "B.SilkS")
 			(effects
@@
 		(layer "Edge.Cuts")
 	)
-	(gr_text "MCU: STM32WL55CCU6\nVIN: 1.45V to 5.5V WLDO\nPOWER: EXT, VBUS"
+	(gr_text "LORA TRANCEIVER BOARD\nMCU: STM32WL55CCU6\nVIN: 1.45V to 5.5V WLDO\nPOWER: EXT, VBUS"
 		(at 190.8 62.6 0)
 		(layer "B.SilkS")
@@
 	)
 	(via
-		(at 154.2 86)
+		(at 154.2 87.8)
 		(size 0.7)
 		(drill 0.3)
@@
 	)
 	(via
+		(at 145.9 77.55)
+		(size 0.7)
+		(drill 0.3)
+		(layers "F.Cu" "B.Cu")
+		(net 2)
+	)
+	(via
 		(at 124.6 79.05)
 		(size 0.7)
@@
 	)
 	(via
+		(at 147.8 79.5)
+		(size 0.7)
+		(drill 0.3)
+		(layers "F.Cu" "B.Cu")
+		(net 2)
+	)
+	(via
 		(at 158.5 70)
 		(size 0.7)
@@
 	)
 	(via
-		(at 153.2 85.1)
+		(at 153.2 87)
 		(size 0.7)
 		(drill 0.3)
@@
 	)
 	(via
+		(at 145.9 77.55)
+		(size 0.7)
+		(drill 0.3)
+		(layers "F.Cu" "B.Cu")
+		(net 2)
+	)
+	(via
 		(at 162.5 67.5)
 		(size 0.7)
@@
 	)
 	(via
+		(at 146 79.5)
+		(size 0.7)
+		(drill 0.3)
+		(layers "F.Cu" "B.Cu")
+		(net 2)
+	)
+	(via
 		(at 175 67)
 		(size 0.7)
@@
 	)
 	(via
+		(at 145.9 77.55)
+		(size 0.7)
+		(drill 0.3)
+		(layers "F.Cu" "B.Cu")
+		(net 2)
+	)
+	(via
 		(at 182.6 73.4)
 		(size 0.7)
@@
 	)
 	(via
+		(at 145.9 77.55)
+		(size 0.7)
+		(drill 0.3)
+		(layers "F.Cu" "B.Cu")
+		(net 2)
+	)
+	(via
 		(at 176.1875 76.3875)
 		(size 0.7)
@@
 	)
 	(via
-		(at 177 67)
+		(at 145.9 77.55)
 		(size 0.7)
 		(drill 0.3)
 		(layers "F.Cu" "B.Cu")
-		(remove_unused_layers yes)
-		(keep_end_layers yes)
-		(free yes)
-		(zone_layer_connections "In1.Cu" "In2.Cu")
-		(teardrops
-			(best_length_ratio 0.5)
-			(max_length 1)
-			(best_width_ratio 1)
-			(max_width 2)
-			(curve_points 0)
-			(filter_ratio 0.9)
-			(enabled yes)
-			(allow_two_segments yes)
-			(prefer_zone_connections yes)
-		)
 		(net 2)
 	)
 	(via
-		(at 145.4 87.2)
+		(at 177 67)
 		(size 0.7)
 		(drill 0.3)
@@
 	)
 	(via
-		(at 158.75 77.75)
+		(at 145.4 87.2)
 		(size 0.7)
 		(drill 0.3)
@@
 	)
 	(via
-		(at 155.3 87)
+		(at 158.75 77.75)
 		(size 0.7)
 		(drill 0.3)
@@
 	)
 	(via
-		(at 153.2 87.2)
+		(at 153.2 88.6)
 		(size 0.7)
 		(drill 0.3)
@@
 	)
 	(via
+		(at 145.9 77.55)
+		(size 0.7)
+		(drill 0.3)
+		(layers "F.Cu" "B.Cu")
+		(net 2)
+	)
+	(via
 		(at 173 73.5)
 		(size 0.7)
@@
 	)
 	(via
+		(at 145.9 77.55)
+		(size 0.7)
+		(drill 0.3)
+		(layers "F.Cu" "B.Cu")
+		(net 2)
+	)
+	(via
 		(at 178.78825 84.11)
 		(size 0.7)
@@
 	)
 	(segment
+		(start 152.65 84.75)
+		(end 154.825 86.925)
+		(width 0.1765)
+		(layer "F.Cu")
+		(net 21)
+	)
+	(segment
 		(start 157.475 86.925)
 		(end 158 87.45)
@@
 	)
 	(segment
-		(start 152.65 82.825)
-		(end 156.75 86.925)
+		(start 150.35 76.8)
+		(end 152.65 79.1)
 		(width 0.1765)
 		(layer "F.Cu")
@@
 	)
 	(segment
-		(start 150.35 76.8)
-		(end 152.65 79.1)
+		(start 154.825 86.925)
+		(end 156.75 86.925)
 		(width 0.1765)
 		(layer "F.Cu")
@@
 	(segment
 		(start 152.65 79.1)
-		(end 152.65 82.825)
+		(end 152.65 84.75)
 		(width 0.1765)
 		(layer "F.Cu")
@@
 	)
 	(segment
-		(start 150.7 76.3)
-		(end 153.35 78.95)
+		(start 149.3375 76.3)
+		(end 150.7 76.3)
 		(width 0.1765)
 		(layer "F.Cu")
@@
 	)
 	(segment
-		(start 149.3375 76.3)
-		(end 150.7 76.3)
+		(start 155.275 85.175)
+		(end 156.75 85.175)
 		(width 0.1765)
 		(layer "F.Cu")
@@
 	)
 	(segment
-		(start 153.35 81.775)
-		(end 156.75 85.175)
+		(start 156.9 85.15)
+		(end 158.7 85.15)
 		(width 0.1765)
 		(layer "F.Cu")
@@
 	)
 	(segment
-		(start 156.9 85.15)
-		(end 158.7 85.15)
+		(start 150.7 76.3)
+		(end 153.35 78.95)
+		(width 0.1765)
+		(layer "F.Cu")
+		(net 23)
+	)
+	(segment
+		(start 153.35 83.25)
+		(end 155.275 85.175)
 		(width 0.1765)
 		(layer "F.Cu")
@@
 	(segment
 		(start 153.35 78.95)
-		(end 153.35 81.775)
+		(end 153.35 83.25)
 		(width 0.1765)
 		(layer "F.Cu")

Commit message: Update
Parts:
- added DI1: Diode_PESD5V0U2BT-Q, Package_TO_SOT_SMD:SOT-23, F.Cu at (96.3, 72.0)

Commit message: Update
Parts:
- removed BH1: Battery_Holder_1060TR, Personal_Project:Battery_Holder_1060TR
- removed C34: 68p_Murata_GCM1555C1H680JA16, Capacitor_SMD:C_0805_2012Metric
- removed C35: 18p_GJM1555C1H180FB01, Capacitor_SMD:C_0805_2012Metric
- removed C36: 20p_GJM1555C1H200GB01, Capacitor_SMD:C_0805_2012Metric
- removed C46: 2p2_GJM1555C1H200GB01, Capacitor_SMD:C_0805_2012Metric
- removed C47, C50: 1p2_GJM1555C1H180FB01, Capacitor_SMD:C_0805_2012Metric
- removed C48: 5p6_GJM1555C1H300FB01, Capacitor_SMD:C_0805_2012Metric
- removed C49: 33p_CC0402GRNPO9BN330, Capacitor_SMD:C_0805_2012Metric
- removed C52, C55, C68: 10p, Capacitor_SMD:C_0805_2012Metric
- removed C54, C69: 1n, Capacitor_SMD:C_0805_2012Metric
- removed C58: 33p_GRM1555C2A221GE01, Capacitor_SMD:C_0805_2012Metric
- removed C59, C60: 3p3_GJM1555C1H220FB01, Capacitor_SMD:C_0805_2012Metric
- removed C61: 3p6_GJM1555C1H150FB01, Capacitor_SMD:C_0805_2012Metric
- removed C62: 2p7_GJM1555C1H120FB01, Capacitor_SMD:C_0805_2012Metric
- removed C63, C64: 47p, Capacitor_SMD:C_0805_2012Metric
- removed C65, C66: 100n, Capacitor_SMD:C_0805_2012Metric
- removed C67: 4u7, Capacitor_SMD:C_0805_2012Metric
- removed D3: ESD_TSD05DYFR, Personal_Project:ESD_TSD05DYFR_SOD2613X100N
- removed D4: ESD_TSD03DYFR, Personal_Project:ESD_TSD05DYFR_SOD2613X100N
- removed FB1: BLM21PG601SN1D_0805, Capacitor_SMD:C_0805_2012Metric
- removed G***: LOGO, Personal_Project:PCB_Logo
- removed H1, H2, H3, H4: MountingHole_Pad, MountingHole:MountingHole_3.2mm_M3_Pad
- removed IC1: RF_Switch_PE42440MLBB-Z, Personal_Project:RF_SWITCH_PE42440_QFN50P300X300X80-17N
- removed J1: JST_XH_2.54_Plug, Personal_Project:Connector_Power2pin_SHDRRA2W80P0X250_1X2_740X1150X610P
- removed J13: SPI1_Headers, Connector_PinHeader_2.54mm:PinHeader_2x03_P2.54mm_Horizontal
- removed J17: BOOT0_Jumper, Connector_PinHeader_2.54mm:PinHeader_1x03_P2.54mm_Vertical
- removed J19: SMA PCB END LAUNCH JACK ROUND PO, Personal_Project:SMA Clip Mount Adapter (top)
- removed L10: 11n_LQW18ANR12G00, Inductor_SMD:L_0603_1608Metric_Pad1.05x0.95mm_HandSolder
- removed L14, L5: 6n8_LQW18AN6N8C00, Inductor_SMD:L_0603_1608Metric_Pad1.05x0.95mm_HandSolder
- removed L15: 160n_LQW18ANR16G00, Inductor_SMD:L_0603_1608Metric_Pad1.05x0.95mm_HandSolder
- removed L16: 12n_LQW18AN12NG0Z, Inductor_SMD:L_0603_1608Metric_Pad1.05x0.95mm_HandSolder
- removed L17: 51n_LQW18AN51NG0Z, Inductor_SMD:L_0603_1608Metric_Pad1.05x0.95mm_HandSolder
- removed L18: 47n_LQW15AN47NJ00, Inductor_SMD:L_0603_1608Metric_Pad1.05x0.95mm_HandSolder
- removed L2: 8n7_LQW18AN51NG0Z, Inductor_SMD:L_0603_1608Metric_Pad1.05x0.95mm_HandSolder
- removed L6: 33n_LQW15AN33NG00, Inductor_SMD:L_0603_1608Metric_Pad1.05x0.95mm_HandSolder
- removed L7: 3n6_LQW18AN12NG0Z, Inductor_SMD:L_0603_1608Metric_Pad1.05x0.95mm_HandSolder
- removed L9: 8n7_LQW18AN47NG0Z, Inductor_SMD:L_0603_1608Metric_Pad1.05x0.95mm_HandSolder
- removed LDO1: LDO_TLV75733PDBVR, Personal_Project:LDO_SOT95P280X145-5N
- removed OS1: Oscillator_ECS-327MVATX-3-CN-TR, Personal_Project:Oscillator_ECS327MVATX3CNTR
- removed OS2: Oscillator_ECS-TXO-32CSMV-320-AN-TR, Personal_Project:Oscillator_ECSTXO32CSMV320ANTR
- removed Q1: MOSFET_SI2333DDS-T1-BE3, Personal_Project:MOSFET_ SI2333DDS_SOT_DS-T1-BE3_VIS
- removed R10, R11: 27, Resistor_SMD:R_0805_2012Metric
- removed R17, R25: 33R, Resistor_SMD:R_0805_2012Metric
- removed R3: 100k, Resistor_SMD:R_0805_2012Metric
- removed S2: Switch_WS-SLSU SMT Mini Slide, Personal_Project:Switch_WS-SLSU SMT Mini Slide
- removed SW1: Switch_NX3L1T3157GM,115, Personal_Project:Switch_NX3L1T3157GM115
- removed U7: FT230XS, Package_SO:SSOP-16_3.9x4.9mm_P0.635mm
- removed Z1: Diode_BZX84C6V2-7-F, Personal_Project:Diode_BZX84C6V2_SOT96P240X110-3N
- added BH2: Battery_Holder_1060TR, Personal_Project:Battery_Holder_1060TR, F.Cu at (0.47, 53.6)
- added C23: 4u7, Capacitor_SMD:C_0805_2012Metric, F.Cu at (47.5, -24.8)
- added C24: 100n, Capacitor_SMD:C_0805_2012Metric, F.Cu at (47.5, 6.21)
- added C25: 100n_CL21B104KCFNNNE, Capacitor_SMD:C_0805_2012Metric, F.Cu at (47.5, -21.8)
- added C26: 100n, Capacitor_SMD:C_0805_2012Metric, F.Cu at (-21.7, 54.6)
- added C27: 100n, Capacitor_SMD:C_0805_2012Metric, F.Cu at (47.5, -18.8)
- added C28: 47p_KGQ21HCG2D470JT, Capacitor_SMD:C_0805_2012Metric, F.Cu at (47.5, -15.7)
- added C29: 10n, Capacitor_SMD:C_0805_2012Metric, F.Cu at (47.5, -12.7)
- added C30: 100n, Capacitor_SMD:C_0805_2012Metric, F.Cu at (51.9, -27.8)
- added C31: 10p, Capacitor_SMD:C_0805_2012Metric, F.Cu at (51.9, -24.8)
- added C32: 470n, Capacitor_SMD:C_0805_2012Metric, F.Cu at (51.9, -21.8)
- added C57: 33p_NMC0603NPO330J50TRPF, Capacitor_SMD:C_0603_1608Metric, F.Cu at (56.1, -23.0)
- added C7: 100n, Capacitor_SMD:C_0805_2012Metric, F.Cu at (47.5, -27.8)
- added C70: 3p3_GRM1885C1H3R3CA01D, Capacitor_SMD:C_0603_1608Metric, F.Cu at (56.1, -20.5)
- added C71: 10n, Capacitor_SMD:C_0805_2012Metric, F.Cu at (51.9, -18.8)
- added C74: 10p, Capacitor_SMD:C_0805_2012Metric, F.Cu at (31.1, 57.6)
- added C75: 1n, Capacitor_SMD:C_0805_2012Metric, F.Cu at (31.1, 60.6)
- added C76: 10p, Capacitor_SMD:C_0805_2012Metric, F.Cu at (31.1, 63.6)
- added C77: 1n, Capacitor_SMD:C_0805_2012Metric, F.Cu at (35.5, 45.6)
- added C78: 1p2_GJM1555C1H180FB01, Capacitor_SMD:C_0805_2012Metric, F.Cu at (35.5, 48.6)
- added C79: 18p_GJM1555C1H180FB01, Capacitor_SMD:C_0805_2012Metric, F.Cu at (35.5, 51.6)
- added C80: 10p, Capacitor_SMD:C_0805_2012Metric, F.Cu at (35.5, 54.6)
- added C81: 1n, Capacitor_SMD:C_0805_2012Metric, F.Cu at (35.5, 57.6)
- added D1: SMAJ6.0A, Personal_Project:DO-214AC-2, F.Cu at (-3.42, 75.0)
- added DI2: Diode_PESD5V0U2BT-Q, Package_TO_SOT_SMD:SOT-23, F.Cu at (25.6, 23.6)
- added FB5: Murata_BLM21AG102SZ1D, Capacitor_SMD:C_0805_2012Metric, F.Cu at (51.9, -15.7)
- added FPC1: FPC_0545481072, Personal_Project:FPC_0545481072, F.Cu at (29.4, 13.4)
- added H5: MountingHole_Pad, MountingHole:MountingHole_3.2mm_M3_Pad, F.Cu at (105.0, 58.0)
- added H6: MountingHole_Pad, MountingHole:MountingHole_3.2mm_M3_Pad, F.Cu at (-19.9, 22.2)
- added H7: MountingHole_Pad, MountingHole:MountingHole_3.2mm_M3_Pad, F.Cu at (-19.9, 30.1)
- added H8: MountingHole_Pad, MountingHole:MountingHole_3.2mm_M3_Pad, F.Cu at (-19.9, 38.1)
- added IC2: RF_Switch_PE42440MLBB-Z, Personal_Project:RF_SWITCH_PE42440_QFN50P300X300X80-17N, F.Cu at (22.6, 67.8)
- added J10: SMA PCB END LAUNCH JACK ROUND PO, Personal_Project:SMA Clip Mount Adapter (top), F.Cu at (44.8, 63.2)
- added J6: BOOT0_Jumper, Connector_PinHeader_2.54mm:PinHeader_1x03_P2.54mm_Vertical, F.Cu at (60.5, -27.0)
- added JST1: JST_S3B-XH-2.54, Personal_Project:JST_S3B-XH-SHDRRA3W64P0X250_1X3_990X1150X610P, F.Cu at (-11.2, 71.5)
- added L11: 160n_LQW18ANR16G00, Inductor_SMD:L_0603_1608Metric_Pad1.05x0.95mm_HandSolder, F.Cu at (40.0, 52.9)
- added L12: 33n_LQW15AN33NG00, Inductor_SMD:L_0603_1608Metric_Pad1.05x0.95mm_HandSolder, F.Cu at (40.0, 55.4)
- added L13: 47n_LQW15AN47NJ00, Inductor_SMD:L_0603_1608Metric_Pad1.05x0.95mm_HandSolder, F.Cu at (40.0, 57.9)
- added L19: 8n7_LQW18AN47NG0Z, Inductor_SMD:L_0603_1608Metric_Pad1.05x0.95mm_HandSolder, F.Cu at (44.3, 45.3)
- added L20: 3n6_LQW18AN12NG0Z, Inductor_SMD:L_0603_1608Metric_Pad1.05x0.95mm_HandSolder, F.Cu at (44.3, 47.8)
- added L21: 12n_LQW18AN12NG0Z, Inductor_SMD:L_0603_1608Metric_Pad1.05x0.95mm_HandSolder, F.Cu at (44.3, 50.3)
- added L22: 8n7_LQW18AN51NG0Z, Inductor_SMD:L_0603_1608Metric_Pad1.05x0.95mm_HandSolder, F.Cu at (44.3, 52.9)
- added L23: 51n_LQW18AN51NG0Z, Inductor_SMD:L_0603_1608Metric_Pad1.05x0.95mm_HandSolder, F.Cu at (44.3, 55.4)
- added L3: 15u_MLZ2012M150W_TDK, Inductor_SMD:L_0805_2012Metric_Pad1.15x1.40mm_HandSolder, F.Cu at (65.2, -22.9)
- added L4: 6n8_LQW18AN6N8C00, Inductor_SMD:L_0603_1608Metric_Pad1.05x0.95mm_HandSolder, F.Cu at (40.0, 47.8)
- added L8: 6n8_LQW18AN6N8C00, Inductor_SMD:L_0603_1608Metric_Pad1.05x0.95mm_HandSolder, F.Cu at (40.0, 50.3)
- added LDO2: LDO_LDLN050PU33R, Package_DFN_QFN:DFN-8-1EP_3x3mm_P0.65mm_EP1.7x2.05mm, F.Cu at (14.2, 65.5)
- added OS3: Oscillator_ECS-327MVATX-3-CN-TR, Personal_Project:Oscillator_ECS327MVATX3CNTR, F.Cu at (48.2, -8.78)
- added OS4: Oscillator_ECS-TXO-32CSMV-320-AN-TR, Personal_Project:Oscillator_ECSTXO32CSMV320ANTR, F.Cu at (65.6, -26.8)
- added Q2: MOSFET_SI2333DDS-T1-BE3, Personal_Project:MOSFET_ SI2333DDS_SOT_DS-T1-BE3_VIS, F.Cu at (3.63, 65.7)
- added R12: 1k, Resistor_SMD:R_0805_2012Metric, F.Cu at (65.6, -14.8)
- added R13: 220R, Resistor_SMD:R_0805_2012Metric, F.Cu at (65.6, -11.9)
- added R14: 33R, Resistor_SMD:R_0805_2012Metric, F.Cu at (9.38, 24.0)
- added R21: 10k, Resistor_SMD:R_0805_2012Metric, F.Cu at (9.38, 32.8)
- added R22: 10k, Resistor_SMD:R_0805_2012Metric, F.Cu at (9.38, 35.8)
- added R4: 10R, Resistor_SMD:R_0805_2012Metric, F.Cu at (65.6, -17.8)
- added SW3: Switch_NX3L1T3157GM,115, Personal_Project:Switch_NX3L1T3157GM115, F.Cu at (64.9, -9.14)
- added U4: STM32WL55CCU6, Package_DFN_QFN:QFN-48-1EP_7x7mm_P0.5mm_EP5.6x5.6mm, F.Cu at (58.8, -14.6)
- added VS1: VS_STM1818TWX7F, Personal_Project:SOT-23-3_SOT103P237X112-3N, F.Cu at (8.45, 70.1)
- added Z3: Diode_BZX84C6V2-7-F, Personal_Project:Diode_BZX84C6V2_SOT96P240X110-3N, F.Cu at (8.35, 74.7)
- C1: value 4u7 -> 1uF; moved to F.Cu
- C10: value 100n -> 1p2_GJM1555C1H1R2WB01D; moved to F.Cu
- C11, C12: value 100n -> 33p_CC0402GRNPO9BN330; moved to F.Cu
- C13: value 4u7 -> 3p3_GJM1555C1H220FB01; moved to F.Cu
- C14: value 1u -> 100n
- C15: value 1u -> 1p2_GJM1555C1H180FB01; moved to F.Cu
- C16: value 1u -> 33p_NMC0603NPO330J50TRPF; footprint Capacitor_SMD:C_0805_2012Metric -> Capacitor_SMD:C_0603_1608Metric
- C17: value 1p2_GJM1555C1H1R2WB01D -> 10n; moved to F.Cu
- C18: value 10n -> 18p_GJM1555C1H180FB01
- C2: value 68p_GRM1555C2A221GE01 -> 1u
- C20: value 33p_NMC0603NPO330J50TRPF -> 3p3_GJM1555C1H220FB01; footprint Capacitor_SMD:C_0603_1608Metric -> Capacitor_SMD:C_0805_2012Metric; moved to F.Cu
- C21: value 33p_NMC0603NPO330J50TRPF -> 2p2_GJM1555C1H200GB01; footprint Capacitor_SMD:C_0603_1608Metric -> Capacitor_SMD:C_0805_2012Metric
- C22: value 3p3_GRM1885C1H3R3CA01D -> 20p_GJM1555C1H200GB01; footprint Capacitor_SMD:C_0603_1608Metric -> Capacitor_SMD:C_0805_2012Metric; moved to F.Cu
- C3: value 1uF -> 4u7
- C33: value 47n_Murata_GCM155R71E473KA55 -> 2u2; moved to F.Cu
- C37: value 30p_GJM1555C1H300FB01 -> 33p_NMC0603NPO330J50TRPF; footprint Capacitor_SMD:C_0805_2012Metric -> Capacitor_SMD:C_0603_1608Metric
- C38: value 220p_GRM1555C2A221GE01 -> 47p
- C39: value 18p_GJM1555C1H180FB01 -> 100n
- C4: value 10n -> 47n_Murata_GCM155R71E473KA55
- C40: value 470n -> 33p_GRM1555C2A221GE01
- C41: value 4u7 -> 5p6_GJM1555C1H300FB01; moved to F.Cu
- C42: value 100n -> 30p_GJM1555C1H300FB01; moved to F.Cu
- C43: value 100n_CL21B104KCFNNNE -> 68p_GRM1555C2A221GE01; moved to F.Cu
- C44: value 33p_CC0402GRNPO9BN330 -> 47p
- C45: value 1n -> 4u7; moved to F.Cu
- C5: value 33p_NMC0603NPO330J50TRPF -> 2p7_GJM1555C1H120FB01; footprint Capacitor_SMD:C_0603_1608Metric -> Capacitor_SMD:C_0805_2012Metric; moved to F.Cu
- C51: value 47p_KGQ21HCG2D470JT -> 220p_GRM1555C2A221GE01; moved to F.Cu
- C6: value 10p -> 68p_Murata_GCM1555C1H680JA16
- C8: value 1uF -> 3p6_GJM1555C1H150FB01
- C9: value 10p -> 100n
- FB2: value Murata_BLM21AG102SZ1D -> BLM21AG121BH1D
- FB3: moved to F.Cu
- J11: value I2C1_Headers -> Coin Battery Jumper; footprint Connector_PinHeader_2.54mm:PinHeader_2x03_P2.54mm_Horizontal -> Connector_PinHeader_2.54mm:PinHeader_1x03_P2.54mm_Vertical
- J2: value Power_Selector_Jumper -> UART1_HDR; footprint Connector_PinHeader_2.54mm:PinHeader_2x03_P2.54mm_Vertical -> Connector_PinHeader_2.54mm:PinHeader_2x03_P2.54mm_Horizontal
- J3: value Debug_Pins -> SWDB
- J4: value Coin Battery Jumper -> USB_C_Receptacle_USB2.0_16P; footprint Connector_PinHeader_2.54mm:PinHeader_1x03_P2.54mm_Vertical -> Connector_USB:USB_C_Receptacle_HRO_TYPE-C-31-M-12
- J5: value General_Pin_Header -> I/O_HDR; footprint Connector_PinHeader_2.54mm:PinHeader_2x03_P2.54mm_Horizontal -> Connector_PinHeader_2.54mm:PinHeader_2x06_P2.54mm_Vertical
- J7: value LPUART1_Headers -> I2C2_Headers
- J8: value USB_B_Micro -> PWR_SRC_JMP; footprint Connector_USB:USB_Micro-B_XKB_U254-051T-4BH83-F1S -> Connector_PinHeader_2.54mm:PinHeader_1x03_P2.54mm_Vertical
- J9: value 3V_Selection_Header -> I2C1_Headers; footprint Connector_PinHeader_2.54mm:PinHeader_1x03_P2.54mm_Vertical -> Connector_PinHeader_2.54mm:PinHeader_2x03_P2.54mm_Horizontal
- L1: value 15u_MLZ2012M150W_TDK -> 11n_LQW18ANR12G00; footprint Inductor_SMD:L_0805_2012Metric_Pad1.15x1.40mm_HandSolder -> Inductor_SMD:L_0603_1608Metric_Pad1.05x0.95mm_HandSolder
- R1: value 220R -> 100R
- R16, R9: value 33R -> 27; moved to F.Cu
- R18: value 33R -> 10k; moved to F.Cu
- R2: value 10R -> 100R
- R20: value 100R -> 10k; moved to F.Cu
- R5, R6: value 100R -> 5k1; moved to F.Cu
- R8: value 1k -> 100R
- U1: value STM32WL55CCU6 -> USBLC6-2SC6; footprint Package_DFN_QFN:QFN-48-1EP_7x7mm_P0.5mm_EP5.6x5.6mm -> Package_TO_SOT_SMD:SOT-23-6
- U3: value USBLC6-2SC6 -> SN74LVC1G07DBVR; footprint Package_TO_SOT_SMD:SOT-23-6 -> Package_TO_SOT_SMD:SOT-23-5
- U6: value ~ -> FT230XS; footprint Personal_Project:Button_KMR231GLFS -> Package_SO:SSOP-16_3.9x4.9mm_P0.635mm
- moved J7 216.0 mm to (-13.7, 22.3), turned to 0 degrees
- moved C39 198.9 mm to (-21.7, 60.6), turned to 0 degrees
- moved C2 193.0 mm to (-21.7, 45.6)
- moved C45 192.4 mm to (-21.7, 63.6), turned to 0 degrees
- moved FB2 180.0 mm to (-21.7, 66.6), turned to 0 degrees
- moved C17 178.3 mm to (-21.7, 51.6), turned to 0 degrees
- moved R20 174.9 mm to (9.38, 29.9), turned to 0 degrees
- moved C33 173.3 mm to (-21.7, 57.6), turned to 0 degrees
- moved SHLD1 172.5 mm to (-1.90, -17.3)
- moved R18 171.1 mm to (9.38, 26.9)
- moved J5 165.8 mm to (2.30, 12.6), turned to 0 degrees
- moved J11 163.6 mm to (-1.05, 65.5), turned to 0 degrees
- moved C37 154.0 mm to (56.1, -25.5), turned to 0 degrees
- moved R16 150.5 mm to (51.9, 16.5), turned to 0 degrees
- moved R9 150.2 mm to (51.9, 13.5), turned to 0 degrees
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Connections:
- C1 pad 1: /POWER_3V3 -> GND
- C1 pad 2: GND -> /Interfaces/USR_BTN
- C10 pad 1: +3.3V -> /RF_ANT/VR_PA
- C11 pad 1: +3.3V -> GND
- C11 pad 2: GND -> /RF_ANT/Y0
- C12 pad 1: +3.3VA -> GND
- C12 pad 2: GND -> /RF_ANT/Y1
- C13 pad 1: +3.3VA -> GND
- C13 pad 2: GND -> /RF_ANT/RFIN_2
- C14 pad 1: /LDO_IN -> USB_VBUS+
- C15 pad 1: +3.3V -> GND
- C15 pad 2: GND -> /RF_ANT/RF1_4
- C16 pad 1: /LD_OUT_3V3 -> GND
- C16 pad 2: GND -> /STM32WL55CCU6/VFBSMPS
- C17 pad 1: /VR_PA -> Net-(LDO2-FB)
- C18 pad 2: +3.3V -> /RF_ANT/RF2_4
- C19 pad 1: /VBAT -> Net-(U6-3V3OUT)
- C2 pad 1: /RF1_3 -> /Power_Management/PWR+_PS
- C2 pad 2: /RF1_2 -> GND
- C20 pad 1: /VDDPA -> GND
- C20 pad 2: GND -> /RF_ANT/RFIN_1
- C21 pad 1: /VFBSMPS -> /RF_ANT/RF1_4
- C21 pad 2: GND -> /RF_ANT/RF1_3
- C22 pad 1: +3.3V -> /RF_ANT/RF2_4
- C22 pad 2: GND -> /RF_ANT/RF2_3
- C3 pad 1: GND -> USB_VBUS+
- C3 pad 2: /PB12_USR_BTN -> GND
- C33 pad 1: /VR_PA -> +3.3V
- C37 pad 2: /RF2_3 -> /STM32WL55CCU6/VDDPA
- C38 pad 1: /RF2_3 -> /USB/USB_D2+_DI
- C38 pad 2: /RF2_2 -> GND
- C39 pad 1: GND -> +3.3VA
- C39 pad 2: /RF2_1 -> GND
- C4 pad 1: GND -> /RF_ANT/VR_PA
- C4 pad 2: Net-(OS2-VDD) -> GND
- C40 pad 1: /VFBSMPS -> /RF_ANT/RFIN_1
- C40 pad 2: GND -> /RF_ANT/RFIN
- C41 pad 1: +3.3V -> GND
- C41 pad 2: GND -> /RF_ANT/RF1_3
- C42 pad 1: +3.3V -> GND
- C42 pad 2: GND -> /RF_ANT/RF2_3
- C43 pad 1: /PB0_VDD_TCXO -> /RF_ANT/RF1_3
- C43 pad 2: GND -> /RF_ANT/RF1_2
- C44 pad 1: GND -> /USB/USB_D2-_DI
- C44 pad 2: /Y0 -> GND
- C45 pad 1: /VDD -> +3.3VA
- C5 pad 1: +3.3V -> GND
- C5 pad 2: GND -> /RF_ANT/RFI_N
- C51 pad 1: /PB0_VDD_TCXO -> /RF_ANT/RF2_3
- C51 pad 2: GND -> /RF_ANT/RF2_2
- C6 pad 1: Net-(C6-Pad1) -> /RF_ANT/VR_PA
- C6 pad 2: /PH0-OSC_IN -> GND
- C8 pad 1: GND -> /RF_ANT/RFI_P
- C8 pad 2: /NRST -> /RF_ANT/RF1
- C9 pad 1: /VBUS_5V -> VBAT+
- DI1 pad 1: /PB7_I2C1_SDA -> /Interfaces/I2C2_SDA_HDR
- DI1 pad 2: /PB8_I2C1_SCL -> /Interfaces/I2C2_SCL_HDR
- FB2 pad 1: /PB0_VDD_TCXO -> +3.3VA
- FB2 pad 2: Net-(OS2-VDD) -> +3.3V
- FB3 pad 1: /VBUS_5V -> USB_VBUS+
- FB3 pad 2: /+5V_VBUS_FB -> USB_VBUS+
- J11 pad 1: /PB7_I2C1_SDA -> +3.3V
- J11 pad 2: GND -> VBAT+
- J11 pad 3: GND -> Net-(BH2-+)
- J2 pad 1: /EXT_POWER+_PP -> GND
- J2 pad 2: /EXT_POWER+_NOLDO -> GND
- J2 pad 3: /EXT_POWER+_PP -> Net-(J2-Pin_3)
- J2 pad 4: /LDO_IN -> GND
- J2 pad 5: /VBUS_5V -> GND
- J2 pad 6: /LDO_IN -> GND
- J3 pad 2: /PA14_SWCLK -> /Interfaces/SWCLK
- J3 pad 4: /PB3_SWO -> /Interfaces/SWO
- J3 pad 6: /NRST -> /Interfaces/NRST
- J3 pad 8: /PA13_SWDIO -> /Interfaces/SWDIO
- J5 pad 2: /PA8_MCO -> /Interfaces/I/O_HDR0
- J5 pad 3: /PA4_SPI1_NSS -> GND
- J5 pad 4: GND -> /Interfaces/I/O_HDR1
- J5 pad 6: /PA0 -> /Interfaces/I/O_HDR2
- J7 pad 1: Net-(J7-Pin_1) -> /Interfaces/I2C2_SDA_HDR
- J7 pad 5: Net-(J7-Pin_5) -> /Interfaces/I2C2_SCL_HDR
- J8 pad 1: /VBUS_5V -> /Power_Management/PWR+_PS
- J8 pad 2: /USB_D2- -> /Power_Management/PWR+_PP
- J8 pad 3: /USB_D2+ -> USB_VBUS+
- J9 pad 1: /EXT_POWER+_NOLDO -> /Interfaces/I2C1_SDA_HDR
- J9 pad 2: /POWER_3V3 -> GND
- J9 pad 3: /LD_OUT_3V3 -> GND
- L1 pad 1: /VFBSMPS -> /RF_ANT/RFI_N
- L1 pad 2: /VLXSMPS -> /RF_ANT/RFI_P
- R1 pad 1: Net-(OS2-OUTPUT) -> +3.3V
- R1 pad 2: Net-(C6-Pad1) -> /RF_ANT/VDD
- R16 pad 1: /PA3_LPUART1_RX -> /USB/USB_D2+_DI
- R16 pad 2: Net-(J7-Pin_5) -> /USB/USBDP
- R18 pad 1: /PA1_SPI1_SCK -> +3.3V
- R18 pad 2: Net-(J13-Pin_5) -> /Interfaces/I2C2_SDA_HDR
- R2 pad 1: Net-(OS1-OUTPUT) -> /RF_ANT/PA5_INOUTRF
- R2 pad 2: /PC14-OSC32_IN -> /RF_ANT/V2
- R20 pad 1: /PA7_HPLP_CTRL -> +3.3V
- R20 pad 2: /V1 -> /Interfaces/I2C2_SCL_HDR
- R5 pad 1: +3.3V -> Net-(J4-CC1)
- R5 pad 2: /VDD -> GND
- R6 pad 1: /PA5_INOUTRF -> Net-(J4-CC2)
- R6 pad 2: /V2 -> GND
- R7 pad 1: GND -> /Power_Management/PWR+_GATE
- R7 pad 2: Net-(J8-ID) -> GND
- R8 pad 1: /BOOT0J -> /RF_ANT/PA7_HPLP_CTRL
- R8 pad 2: /BOOT0 -> /RF_ANT/V1
- R9 pad 1: Net-(J7-Pin_1) -> /USB/USB_D2-_DI
- R9 pad 2: /PA2_LPUART1_TX -> /USB/USBDM
- SW2 pad 1: /VFBSMPS -> /RF_ANT/Y1
- SW2 pad 3: +3.3V -> /RF_ANT/Y0
- SW2 pad 4: /VDDPA -> Net-(SW2-Z)
- SW2 pad 6: /PB2_RFVCTRL -> /RF_ANT/PA7_HPLP_CTRL
- U1 pad 1: /PB3_SWO -> /USB/USB_D2-_DI
- U1 pad 2: /PB4_SPI1_MISO -> GND
- U1 pad 3: /PB5_SPI1_MOSI -> /USB/USB_D2+_DI
- U1 pad 4: /PB6_USART1_TX -> /USB/USB_D2+
- U1 pad 5: /PB7_I2C1_SDA -> USB_VBUS+
- U1 pad 6: /PB8_I2C1_SCL -> /USB/USB_D2-
- U2 pad 1: /NRST -> /Interfaces/USR_BTN
- U2 pad 2: /NRST -> /Interfaces/USR_BTN
- U3 pad 1: /USB_D2- -> unconnected-(U3-NC-Pad1)
- U3 pad 2: GND -> /Power_Management/RST_PWR
- U3 pad 3: /USB_D2+ -> GND
- U3 pad 4: /USB_D+ -> /Interfaces/NRST
- U3 pad 5: /VBUS_5V -> +3.3V
- U6 pad 1: /PB12_USR_BTN -> /STM32WL55CCU6/PA2_LPUART1_TX
- U6 pad 2: /PB12_USR_BTN -> /STM32WL55CCU6/PB12_LPUART1_RTS
- U6 pad 3: GND -> Net-(U6-3V3OUT)
- U6 pad 4: GND -> /STM32WL55CCU6/PA3_LPUART1_RX
Routing:
- net +3.3V: track 298.5 -> 0.00 mm, vias 16 -> 0
- net /NRST: track 95.9 -> 0.00 mm, vias 3 -> 0
- net /PA13_SWDIO: track 82.4 -> 0.00 mm, vias 2 -> 0
- net /PA14_SWCLK: track 75.9 -> 0.00 mm, vias 1 -> 0
- net /PB3_SWO: track 64.0 -> 0.00 mm, vias 1 -> 0
- net /VFBSMPS: track 62.9 -> 0.00 mm
- net /PB4_SPI1_MISO: track 58.4 -> 0.00 mm, vias 1 -> 0
- net /PB7_I2C1_SDA: track 57.5 -> 0.00 mm, vias 1 -> 0
- net /BOOT0: track 49.1 -> 0.00 mm, vias 2 -> 0
- net /EXT_POWER+_NOLDO: track 46.8 -> 0.00 mm, vias 1 -> 0
- net /PA3_LPUART1_RX: track 46.1 -> 0.00 mm, vias 1 -> 0
- net /PB12_USR_BTN: track 45.9 -> 0.00 mm, vias 2 -> 0
- net GND: track 45.8 -> 0.00 mm, vias 231 -> 0
- net /PA2_LPUART1_TX: track 45.7 -> 0.00 mm, vias 1 -> 0
- net /PB6_USART1_TX: track 41.7 -> 0.00 mm, vias 2 -> 0
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- removed copper zone on B.Cu, net /EXT_POWER+
- removed copper zone on B.Cu, net /EXT_POWER+_PP
- removed copper zone on B.Cu, net /MOSFET_GATE
- removed copper zone on B.Cu, net GND
- removed copper zone on F.Cu, net GND
- removed copper zone on In1.Cu, net GND
- removed copper zone on In2.Cu, net GND
Other:
- board text removed: "BAT/3V3"
- board text removed: "CK/MO/MI"
- board text removed: "GN/BT/3V3"
- board text removed: "I2C1"
- board text removed: "LD/EX3"
- board text removed: "LORA TRANCEIVER BOARD MCU: STM32WL55CCU6 VIN: 1.45V to 5.5V WLDO POWER: EXT, VBUS"
- board text removed: "LPUART1"
- board text removed: "NOLDO"
- board text removed: "NR/SO/CL/SD"
- board text removed: "NRST"
- board text removed: "ON/OFF"
- board text removed: "PA0"
- board text removed: "PA8MCO"
- board text removed: "RX"
- board text removed: "SCL"
- board text removed: "SDA"
- board text removed: "SPI1"
- board text removed: "SPINSS"
- board text removed: "TX"
- board text removed: "USRBT"
- board text removed: "V+"
- board text removed: "VBUS"
- board text removed: "WLD"

Commit message: Update
Parts:
- added C34: 100n, Capacitor_SMD:C_0805_2012Metric, B.Cu at (131.7, 92.8)
- BH2, C17, C2, C26, C33, C39, C45, FB2, LDO2, U3, VS1: moved to B.Cu
- J5: footprint Connector_PinHeader_2.54mm:PinHeader_2x06_P2.54mm_Vertical -> Connector_PinHeader_2.54mm:PinHeader_2x06_P2.54mm_Horizontal
- moved H7 228.2 mm to (197.0, 101.0)
- moved H6 219.9 mm to (197.0, 58.0)
- moved J7 217.2 mm to (189.0, 100.5), turned to -90 degrees
- moved J9 202.1 mm to (176.5, 100.3), turned to -90 degrees
- moved R18 200.4 mm to (188.9, 116.0)
- moved R20 200.4 mm to (188.9, 119.0)
- moved J2 198.2 mm to (164.0, 100.5), turned to -90 degrees
- moved DI1 187.2 mm to (185.3, 116.8)
- moved R21 185.9 mm to (175.1, 117.0)
- moved R22 185.9 mm to (175.1, 120.0)
- moved BH2 174.0 mm to (174.0, 66.6)
- moved DI2 173.6 mm to (171.3, 118.0)
- moved SHLD1 172.4 mm to (147.8, 68.2)
- moved C13 170.8 mm to (194.3, 78.2), turned to 90 degrees
- moved R14 168.5 mm to (160.8, 98.0)
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Connections:
- net /RF_ANT/PA5_INOUTRF renamed /Antenna/PA5_INOUTRF
- net /RF_ANT/PA7_HPLP_CTRL renamed /Antenna/PA7_HPLP_CTRL
- net /RF_ANT/RF1 renamed /Antenna/RF1
- net /RF_ANT/RF1_1 renamed /Antenna/RF1_1
- net /RF_ANT/RF1_2 renamed /Antenna/RF1_2
- net /RF_ANT/RF1_3 renamed /Antenna/RF1_3
- net /RF_ANT/RF1_4 renamed /Antenna/RF1_4
- net /RF_ANT/RF2_1 renamed /Antenna/RF2_1
- net /RF_ANT/RF2_2 renamed /Antenna/RF2_2
- net /RF_ANT/RF2_3 renamed /Antenna/RF2_3
- net /RF_ANT/RF2_4 renamed /Antenna/RF2_4
- net /RF_ANT/RFIN renamed /Antenna/RFIN
- net /RF_ANT/RFIN_1 renamed /Antenna/RFIN_1
- net /RF_ANT/RFIN_2 renamed /Antenna/RFIN_2
- net /RF_ANT/RFI_N renamed /Antenna/RFI_N
- net /RF_ANT/RFI_P renamed /Antenna/RFI_P
- net /RF_ANT/RFO_HP renamed /Antenna/RFO_HP
- net /RF_ANT/RFO_LP renamed /Antenna/RFO_LP
- net /RF_ANT/V1 renamed /Antenna/V1
- net /RF_ANT/V2 renamed /Antenna/V2
- net /RF_ANT/VDD renamed /Antenna/VDD
- net /RF_ANT/VR_PA renamed /Antenna/VR_PA
- net /RF_ANT/Y0 renamed /Antenna/Y0
- net /RF_ANT/Y1 renamed /Antenna/Y1
- net Net-(J4-CC1) renamed /USB/CC1
- net Net-(J4-CC2) renamed /USB/CC2
- C24 pad 1: USB_VBUS+ -> /USB/VBUS
- FB3 pad 1: USB_VBUS+ -> /USB/VBUS
- J4 pad A4: USB_VBUS+ -> /USB/VBUS
- J4 pad A9: USB_VBUS+ -> /USB/VBUS
- J4 pad B4: USB_VBUS+ -> /USB/VBUS
- J4 pad B9: USB_VBUS+ -> /USB/VBUS
- J8 pad 1: /Power_Management/PWR+_PS -> /Power_Management/PWR+_PP
- J8 pad 2: /Power_Management/PWR+_PP -> /Power_Management/PWR+_PS
- U1 pad 5: USB_VBUS+ -> /USB/VBUS
Routing:
- net +3.3V: track 0.00 -> 24.9 mm
- net /USB/VBUS: track 0.00 -> 18.0 mm, vias 0 -> 3
- net /STM32WL55CCU6/VFBSMPS: track 0.00 -> 13.5 mm, vias 0 -> 2
- net +3.3VA: track 0.00 -> 12.1 mm, vias 0 -> 1
- net GND: track 0.00 -> 10.5 mm, vias 0 -> 2
- net /Interfaces/SWCLK: track 0.00 -> 6.01 mm
- net /Interfaces/I2C1_SDA_HDR: track 0.00 -> 5.95 mm
- net Net-(OS4-VDD): track 0.00 -> 4.87 mm
- net /STM32WL55CCU6/PH0-OSC_IN: track 0.00 -> 4.78 mm
- net /USB/CC1: track 0.00 -> 4.72 mm
- net PB0_VDD_TCXO+: track 0.00 -> 4.51 mm
- net /USB/CC2: track 0.00 -> 4.50 mm
- net /STM32WL55CCU6/VLXSMPS: track 0.00 -> 4.41 mm
- net /USB/USB_D2+_DI: track 0.00 -> 4.07 mm
- net /USB/USB_D2-_DI: track 0.00 -> 4.07 mm
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- added copper zone on B.Cu, net +3.3V
- added copper zone on B.Cu, net +3.3VA
- added copper zone on F.Cu, net /Power_Management/PWR+
- added copper zone on F.Cu, net /Power_Management/PWR+_GATE
- added copper zone on F.Cu, net /Power_Management/PWR+_PP
- added copper zone on B.Cu, net /Power_Management/PWR+_PS
- added copper zone on F.Cu, net /Power_Management/PWR+_PS
- added copper zone on B.Cu, net /USB/VBUS
- added copper zone on B.Cu, net GND
- added copper zone on F.Cu, net GND
- added copper zone on In1.Cu, net GND
- added copper zone on In2.Cu, net GND
- added copper zone on F.Cu, net USB_VBUS+
Other:
- board size 100 x 51 mm -> 100 x 54 mm

Commit message: Update
Parts:
- C10, C4, C6: footprint Capacitor_SMD:C_0805_2012Metric -> Capacitor_SMD:C_0603_1608Metric_Pad1.08x0.95mm_HandSolder; moved to B.Cu
- C11, C12, C13, C15, C18, C20, C21, C22, C40, C41, C42, C43, C5, C51, C78, C79, C8: footprint Capacitor_SMD:C_0805_2012Metric -> Capacitor_SMD:C_0603_1608Metric_Pad1.08x0.95mm_HandSolder
- L11, R1, R2, R8, SW2: moved to B.Cu
- moved L21 10.0 mm to (162.7, 83.4)
- moved R8 9.17 mm to (158.4, 79.9), turned to 180 degrees
- moved R1 9.15 mm to (158.4, 75.3)
- moved R2 9.15 mm to (158.4, 77.6)
- moved C18 8.41 mm to (160.0, 84.3), turned to 90 degrees
- moved L23 8.40 mm to (171.9, 83.4)
- moved C51 8.33 mm to (168.2, 83.4)
- moved C42 7.90 mm to (165.5, 84.3), turned to 90 degrees
- moved C78 7.42 mm to (174.6, 70.7)
- moved C43 7.28 mm to (168.2, 71.6)
- moved L22 7.21 mm to (171.9, 71.6)
- moved C41 6.85 mm to (165.5, 70.7)
- moved C22 6.65 mm to (162.7, 85.2)
- moved L20 6.56 mm to (162.8, 71.6)
- moved C21 6.48 mm to (162.8, 69.8)
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Connections:
- C11 pad 2: /Antenna/Y0 -> /Antenna/Y1
- C12 pad 2: /Antenna/Y1 -> /Antenna/Y0
- L12 pad 1: /Antenna/Y0 -> /Antenna/Y1
- L13 pad 2: /Antenna/Y1 -> /Antenna/Y0
Routing:
- net /STM32WL55CCU6/PA3_LPUART1_RX: track 0.00 -> 30.7 mm, vias 0 -> 2
- net /STM32WL55CCU6/PA2_LPUART1_TX: track 0.00 -> 28.2 mm, vias 0 -> 2
- net /Antenna/RF1: track 0.00 -> 27.7 mm
- net /Interfaces/SPI_MISO: track 0.00 -> 25.6 mm, vias 0 -> 2
- net /Interfaces/SPI_CLK: track 0.00 -> 23.9 mm, vias 0 -> 2
- net /Interfaces/SPI_MOSI: track 0.00 -> 23.9 mm, vias 0 -> 2
- net /Antenna/RFI_P: track 0.00 -> 21.3 mm
- net /Antenna/RFI_N: track 0.00 -> 20.5 mm
- net /Antenna/RFO_LP: track 0.00 -> 13.6 mm
- net Net-(U6-3V3OUT): track 0.00 -> 11.9 mm
- net /Antenna/RFIN_2: track 0.00 -> 11.7 mm
- net /Antenna/V2: track 0.00 -> 9.30 mm
- net /Antenna/RF1_1: track 0.00 -> 8.76 mm
- net /Antenna/RF2_1: track 0.00 -> 8.42 mm
- net GND: track 10.5 -> 18.8 mm
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