File: LoRa_Board.kicad_pcb (KiCad board)
At the start: 4 copper layers, 100 x 54 mm, 120 parts, among them IC2 RF_Switch_PE42440MLBB-Z, J1 I/O_HDR, J10 SMA PCB END LAUNCH JACK ROUND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, J2 UART1_HDR, J3 SWDB, J4 USB_C_Receptacle_USB2.0_16P, J6 BOOT0_Jumper, J7 I2C2_Headers, J8 PWR_SRC_JMP, J9 I2C1_Headers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

Commit message: Update
Parts:
- added C9: 4u7, Capacitor_SMD:C_0805_2012Metric, F.Cu at (107.0, 89.9)
- moved R18 26.4 mm to (144.0, 108.6)
- moved C14 26.3 mm to (116.8, 114.1), turned to -90 degrees
- moved C3 23.4 mm to (114.6, 114.1), turned to -90 degrees
- moved R20 20.5 mm to (146.1, 108.6)
- moved FB3 18.8 mm to (111.6, 113.4), turned to 0 degrees
- moved C24 13.6 mm to (109.7, 111.2)
- moved D1 0.75 mm to (112.9, 94.4)
- moved C76 0.60 mm to (165.8, 92.7)
- moved C77 0.50 mm to (168.0, 92.7)
- turned DI2 to 90 degrees
Connections:
- C14 pad 1: USB_VBUS+ -> /USB/USB_VBUS+
- C24 pad 1: /USB/VBUS -> VBUS+
- C3 pad 1: USB_VBUS+ -> /USB/USB_VBUS+
- FB3 pad 1: /USB/VBUS -> VBUS+
- FB3 pad 2: USB_VBUS+ -> /USB/USB_VBUS+
- J4 pad A4: /USB/VBUS -> VBUS+
- J4 pad A9: /USB/VBUS -> VBUS+
- J4 pad B4: /USB/VBUS -> VBUS+
- J4 pad B9: /USB/VBUS -> VBUS+
- J8 pad 3: USB_VBUS+ -> VBUS+
- U1 pad 5: /USB/VBUS -> VBUS+
- U6 pad 12: USB_VBUS+ -> /USB/USB_VBUS+
Routing:
- net GND: track 28.8 -> 166.5 mm, vias 171 -> 307
- net VBUS+: track 0.00 -> 23.1 mm, vias 0 -> 3
- net USB_VBUS+: track 19.9 -> 0.00 mm, vias 1 -> 0
- net +3.3V: track 180.1 -> 198.6 mm
- net /USB/USB_VBUS+: track 0.00 -> 18.4 mm, vias 0 -> 2
- net /USB/VBUS: track 18.0 -> 0.00 mm, vias 3 -> 0
- net /Interfaces/NRST: track 117.8 -> 121.3 mm
- net /Interfaces/I2C2_SDA_HDR: track 66.8 -> 69.0 mm
- net /Interfaces/I2C2_SCL_HDR: track 53.7 -> 55.9 mm
- net /Antenna/PA5_INOUTRF: track 18.8 -> 20.5 mm
- net /Interfaces/USR_BTN: track 61.5 -> 60.3 mm
- net /Interfaces/I2C1_SCL_HDR: track 112.3 -> 111.3 mm
- net /Interfaces/SPI_MISO: track 58.3 -> 59.2 mm
- net /STM32WL55CCU6/BOOT0: track 63.3 -> 63.9 mm
- net /Interfaces/SPI_MOSI: track 54.8 -> 55.3 mm
- added copper zone on F.Cu, net VBUS+
- removed copper zone on B.Cu, net /USB/VBUS
- removed copper zone on F.Cu, net USB_VBUS+
Other:
- board text added: "BT0"
- board text added: "HIGH"

Commit message: Update
Routing:
- net GND: track 166.5 -> 166.9 mm, vias 307 -> 446

Commit message: Update
Parts:
- FPC1: value FPC_0545481072 -> FPC_10051922-1010ELF; footprint Personal_Project:FPC_0545481072 -> Personal_Project:FPC_10051922_1010
- turned FPC1 to 180 degrees
Routing:
- net GND: track 166.9 -> 171.9 mm
Other:
- board text added: "CLK"
- board text added: "CS"
- board text added: "MISO"
- board text added: "MOSI"
- board text added: "PWR+"
- board text added: "RST"
- board text added: "SPI1"
- board text added: "SW"
- board text added: "UART1"
- board text added: "USB-C"
- board text added: "VIN: 4.0 V to 6.5 V"
- board text removed: "SPI"
- board text removed: "UART"

Commit message: Update
Parts:
- removed L11: 160n_LQW18ANR16G00, Inductor_SMD:L_0603_1608Metric_Pad1.05x0.95mm_HandSolder
- removed L4: 6n8_LQW18AN6N8C00, Inductor_SMD:L_0603_1608Metric_Pad1.05x0.95mm_HandSolder
- added L2: 0H, Inductor_SMD:L_0603_1608Metric_Pad1.05x0.95mm_HandSolder, F.Cu at (155.5, 85.6)
- C13: value 3p3_GJM1555C1H220FB01 -> 2p6_CC0402BRNPO9BN3R3
- C15: value 1p2_GJM1555C1H180FB01 -> 4p4_GJM1555C1H180FB01
- C18: value 18p_GJM1555C1H180FB01 -> 5p6_CC0402BRNPO9BN5R6
- C20: value 3p3_GJM1555C1H220FB01 -> 3p6_CC0402BRNPO9BN3R3
- C21: value 2p2_GJM1555C1H200GB01 -> 1p9_CC0402BRNPO9BN2R2
- C22: value 20p_GJM1555C1H200GB01 -> 2p7_CC0402BRNPO9BN2R7
- C31: value 10p -> 1n
- C40: value 33p_GRM1555C2A221GE01 -> 40p_CC0402GRNPO9BN330
- C41: value 5p6_GJM1555C1H300FB01 -> 5p6_CC0402BRNPO9BN5R6
- C42: value 30p_GJM1555C1H300FB01 -> 3p3_CC0402BRNPO9BN3R3
- C5: value 2p7_GJM1555C1H120FB01 -> 2p7_CC0402BRNPO9BN2R7
- C51: value 220p_GRM1555C2A221GE01 -> 33p_CC0402GRNPO9BN330
- C78: value 1p2_GJM1555C1H180FB01 -> 1p3_GJM1555C1H1R2WB01D
- C79: value 18p_GJM1555C1H180FB01 -> 1p3_CC0402BRNPO9BN1R3
- C8: value 3p6_GJM1555C1H150FB01 -> 3p6_CC0402BRNPO9BN3R6
- FB5: value Murata_BLM21AG102SZ1D -> Murata_BLM21AG102SZ1D_1400R@1GHz
- L1: value 11n_LQW18ANR12G00 -> 11n_LQW15AN11NG00
- L19: value 8n7_LQW18AN47NG0Z -> 6n1_LQW15AN8N7H00
- L20: value 3n6_LQW18AN12NG0Z -> 4n7_LQW15AN3N6C10
- L21: value 12n_LQW18AN12NG0Z -> 3n_LQW15AN3N0B00
- L22: value 8n7_LQW18AN51NG0Z -> 8n8_LQW15AN8N7H00
- L23: value 51n_LQW18AN51NG0Z -> 8n7_LQW15AN8N7H00
- L8: value 6n8_LQW18AN6N8C00 -> 3n3_LQW15AN3N3C80
- OS4: value Oscillator_ECS-TXO-32CSMV-320-AN-TR -> Oscillator_HCI 8132S-32.000MN33DTL
- SW2, SW3: value Switch_NX3L1T3157GM,115 -> Switch_NX3L1T3157GMZ
Connections:
- OS3 pad 1: unconnected-(OS3-TRI-STATE-Pad1) -> +3.3V
- SW2 pad 4: Net-(SW2-Z) -> /Antenna/VR_PA
Routing:
- net /Antenna/VR_PA: track 12.1 -> 16.4 mm, vias 1 -> 2
- net Net-(SW2-Z): track 4.31 -> 0.00 mm, vias 1 -> 0
- net +3.3V: track 198.6 -> 200.5 mm
