File: STM32WL55CCU6.kicad_sch (KiCad schematic)
At the start: 31 parts, among them J6 BOOT0_Jumper, SW3 Switch_NX3L1T3157GM,115, U4 STM32WL55CCU6

Commit message: Update
Parts:
- removed C56: 1uF, Capacitor_SMD:C_0805_2012Metric, symbol Device:C
- removed C72, C73: 33p_NMC0603NPO330J50TRPF, Capacitor_SMD:C_0603_1608Metric, symbol Device:C
- removed SHLD2: RFShield_OnePiece, Personal_Project:RF_Shield_MS631-10F, symbol Device:RFShield_OnePiece
- removed U5: ~, Personal_Project:Button_KMR231GLFS, symbol Personal_Projects:Button_KMR231GLFS
- added C16, C37: 33p_NMC0603NPO330J50TRPF, Capacitor_SMD:C_0603_1608Metric, symbol Device:C
Connections:
- net GND: now also C16.1, C37.1
- net PC14-OSC32_IN: now also R4.1; no longer R4.2
- net VDDPA: now also C37.2
- net VFBSMPS: now also C16.2
- net at OS3.3 (OUTPUT): now also R4.2; no longer R4.1
- net PA6_LPUART1_CTS: now reaches U4.14 (PA6)
- net PA9_USR_BTN: now reaches U4.17 (PA9)
- net PA15_I2C2_SDA: now reaches U4.43 (PA15)
- net PA0 renamed PA0_DEBUG_PWR-REGLP1S
- net PA10_USART1_RX renamed PA10_DEBUG_RF-HSE32RDY
- net PA11_USART1_CTS renamed PA11_DEBUG_RF-NRESET
- net PA12_USART1_RTS renamed PA12_I2C2_SCL
- net PB0_VDD_TCXO renamed PB0_VDD_TCXO+
- net PB12_USR_BTN renamed PB12_LPUART1_RTS
- net VBAT renamed VBAT+
- no-connect marks 7 -> 3
Other:
- note removed: "100 nF for each VDD or VDDIO2 (Ceramic capacitors)"
- note removed: "10uF could be 4u7"
- note removed: "Clock Output"
- note removed: "PWR_FLG tells KiCad that this is power source"
- note removed: "Place 33p Capacitors near the MCU"
- note removed: "This 3.3V is from digital power rail"
- note removed: "VDDA feeds ADC and DAC pins, and it needs more filtering"
- title: (none) -> LORA_STM32WL55CCU6_Board
- moved on the sheet: C23, C24, C25, C26, C27, C28, C29, C30, C31, C32, C53, C57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

Commit message: Update
Parts:
- removed C24: 100n, Capacitor_SMD:C_0805_2012Metric, symbol Device:C
- removed C26: 4u7, Capacitor_SMD:C_0805_2012Metric, symbol Device:C
- removed C53: 1u, Capacitor_SMD:C_0805_2012Metric, symbol Device:C
- removed FB4: BLM21PG601SN1D_0805, Capacitor_SMD:C_0805_2012Metric, symbol Device:FerriteBead
Other:
- note added: "VFBSMPS = 1.55 V"
- note removed: "70R@100MHz"
- note removed: "FCM1608KF-601T03TAI-TECH"
- moved on the sheet: C16, C25, C27, C28, C29, C30, C31, C32, C37, C57, C70, C71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

Commit message: Update
Changed lines of the file:
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@@
 		)
 		(property "Value" "10n"
-			(at 160.782 152.4 90)
+			(at 167.64 149.86 90)
 			(effects
 				(font

Commit message: Update
Parts:
- added C35: 100n, Capacitor_SMD:C_0805_2012Metric, symbol Device:C
- C25: value 100n_CL21B104KCFNNNE -> 100n_CC0402KRX7R7BB104
- C28: value 47p_KGQ21HCG2D470JT -> 47p_CC0402JRNPO9BN470
- C71: value 10n -> 220n
Connections:
- net VBAT+ is gone; now on net +3.3V: U4.37 (VBAT)
- net +3.3V: now also C35.1
- net GND: now also C35.2

Commit message: Update
Parts:
- C31: value 10p -> 1n
- OS4: value Oscillator_ECS-TXO-32CSMV-320-AN-TR -> Oscillator_ATX-11-F-32.000MHZ-F05-T
- SW3: value Switch_NX3L1T3157GM,115 -> Switch_NX3L1T3157GMZ
Changed lines of the file:
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@@
 			)
 		)
-		(property "Value" "10p"
+		(property "Value" "1n"
 			(at 173.736 107.188 90)
 			(effects
@@
 			)
 		)
-		(property "Value" "Oscillator_ECS-TXO-32CSMV-320-AN-TR"
+		(property "Value" "Oscillator_ATX-11-F-32.000MHZ-F05-T"
 			(at 220.98 100.33 0)
 			(effects
@@
 			)
 		)
-		(property "Value" "Switch_NX3L1T3157GM,115"
+		(property "Value" "Switch_NX3L1T3157GMZ"
 			(at 58.42 168.91 0)
 			(effects

Commit message: Update Readme file
Other:
- note removed: "4u7 capacitor added near poower output"
- note removed: "BOOT0 Switch HIGH enables UART or I2C too allow programminng of the MCU"
- note removed: "Regulated PA supply output"
- note removed: "These capacitors must be placed as close as possible to (or below) the appropriate pins on the underside of the PCB"
- company: (none) -> Peter Hancak
- title: LORA_STM32WL55CCU6_Board -> LoRa Board
Changed lines of the file:
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@@
 	(paper "USLetter")
 	(title_block
-		(title "LORA_STM32WL55CCU6_Board")
-		(date "2025-10-14")
+		(title "LoRa Board")
+		(date "2026-03-17")
 		(rev "B")
+		(company "Peter Hancak")
 	)
 	(junction
@@
 			)
 			(justify left top)
-		)
-	)
-	(text "BOOT0 Switch HIGH enables \nUART or I2C too allow\nprogramminng of the MCU"
-		(exclude_from_sim no)
-		(at 213.868 142.494 0)
-		(effects
-			(font
-				(size 1 1)
-			)
-			(justify left bottom)
 		)
 	)
@@
 		)
 	)
-	(text "These capacitors must be placed as close\nas possible to (or below) the appropriate \npins on the underside of the PCB"
-		(exclude_from_sim no)
-		(at 34.798 57.15 0)
-		(effects
-			(font
-				(size 1 1)
-			)
-		)
-	)
 	(text "Clipped Sine Wave Oscillator\n- Series C eliminates DC component\n- MCU acciepots clock above zero so the \n  clock signal gets biased (increased)\n  inside the MCU."
 		(exclude_from_sim no)
@@
 		(effects
 			(font
-				(size 1 1)
-			)
-		)
-	)
-	(text "Regulated PA supply output"
-		(exclude_from_sim no)
-		(at 147.828 83.058 0)
-		(effects
-			(font
-				(size 1 1)
-			)
-		)
-	)
-	(text "4u7 capacitor added\nnear poower output"
-		(exclude_from_sim no)
-		(at 174.244 60.198 0)
-		(effects
-			(font

Commit message: Update
Parts:
- FB5: value Murata_BLM21AG102SZ1D -> Murata_BLM21AG102SZ1D_1400R@1GHz
Changed lines of the file:
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@@
 			)
 		)
-		(property "Value" "Murata_BLM21AG102SZ1D"
+		(property "Value" "Murata_BLM21AG102SZ1D_1400R@1GHz"
 			(at 250.444 114.046 90)
 			(effects

Commit message: Update
Parts:
- OS4: value Oscillator_ATX-11-F-32.000MHZ-F05-T -> Oscillator_HCI 8132S-32.000MN33DTL
Connections:
- net +3.3V: now also OS3.1 (TRI-STATE)
- no-connect marks 3 -> 2
Changed lines of the file:
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@@
 	)
 	(junction
+		(at 200.66 144.78)
+		(diameter 0)
+		(color 0 0 0 0)
+	)
+	(junction
 		(at 245.11 74.93)
 		(diameter 0)
@@
 		(at 133.35 116.84)
 	)
-	(no_connect
-		(at 196.85 144.78)
-	)
 	(wire
 		(pts
@@
 	(wire
 		(pts
-			(xy 200.66 142.24) (xy 200.66 151.13)
+			(xy 200.66 142.24) (xy 200.66 144.78)
 		)
 		(stroke
@@
 	(wire
 		(pts
+			(xy 200.66 144.78) (xy 200.66 151.13)
+		)
+		(stroke
+			(width 0)
+			(type default)
+		)
+	)
+	(wire
+		(pts
 			(xy 102.87 58.42) (xy 102.87 68.58)
 		)
@@
 	(wire
 		(pts
+			(xy 196.85 144.78) (xy 200.66 144.78)
+		)
+		(stroke
+			(width 0)
+			(type default)
+		)
+	)
+	(wire
+		(pts
 			(xy 220.98 88.9) (xy 220.98 87.63)
 		)
@@
 			)
 		)
-		(property "Value" "Oscillator_ATX-11-F-32.000MHZ-F05-T"
+		(property "Value" "Oscillator_HCI 8132S-32.000MN33DTL"
 			(at 220.98 100.33 0)
 			(effects
