File: RF_ANT.kicad_sch (KiCad schematic)
At the start: 43 parts, among them IC2 RF_Switch_PE42440MLBB-Z, J10 SMA PCB END LAUNCH JACK ROUND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, SW2 Switch_NX3L1T3157GM,115

Commit message: Update
Changed lines of the file:
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@@
 	(wire
 		(pts
-			(xy 138.43 106.68) (xy 109.22 106.68)
+			(xy 101.6 153.67) (xy 92.71 153.67)
 		)
 		(stroke
@@
 	(wire
 		(pts
-			(xy 101.6 153.67) (xy 92.71 153.67)
+			(xy 186.69 40.64) (xy 196.85 40.64)
 		)
 		(stroke
@@
 	(wire
 		(pts
-			(xy 186.69 40.64) (xy 196.85 40.64)
+			(xy 34.29 57.15) (xy 48.26 57.15)
 		)
 		(stroke
@@
 	(wire
 		(pts
-			(xy 34.29 57.15) (xy 48.26 57.15)
+			(xy 198.12 83.82) (xy 218.44 83.82)
 		)
 		(stroke
@@
 	(wire
 		(pts
-			(xy 198.12 83.82) (xy 218.44 83.82)
+			(xy 43.18 137.16) (xy 43.18 140.97)
 		)
 		(stroke
@@
 	(wire
 		(pts
-			(xy 43.18 137.16) (xy 43.18 140.97)
+			(xy 114.3 102.87) (xy 114.3 106.68)
 		)
 		(stroke
@@
 	(wire
 		(pts
+			(xy 114.3 106.68) (xy 138.43 106.68)
+		)
+		(stroke
+			(width 0)
+			(type default)
+		)
+	)
+	(wire
+		(pts
 			(xy 34.29 54.61) (xy 34.29 57.15)
 		)
@@
 		)
 	)
+	(hierarchical_label "RFO_HP"
+		(shape input)
+		(at 25.4 29.21 180)
+		(fields_autoplaced yes)
+		(effects
+			(font
+				(size 1.27 1.27)
+			)
+			(justify right)
+		)
+	)
+	(hierarchical_label "RFO_LP"
+		(shape input)
+		(at 25.4 93.98 180)
+		(fields_autoplaced yes)
+		(effects
+			(font
+				(size 1.27 1.27)
+			)
+			(justify right)
+		)
+	)
+	(hierarchical_label "RFI_N"
+		(shape output)
+		(at 25.4 127 180)
+		(fields_autoplaced yes)
+		(effects
+			(font
+				(size 1.27 1.27)
+			)
+			(justify right)
+		)
+	)
+	(hierarchical_label "PA5_INOUTRF"
+		(shape bidirectional)
+		(at 115.57 109.22 180)
+		(fields_autoplaced yes)
+		(effects
+			(font
+				(size 1.27 1.27)
+			)
+			(justify right)
+		)
+	)
+	(hierarchical_label "PA7_HPLP_CTRL"
+		(shape input)
+		(at 49.53 68.58 180)
+		(fields_autoplaced yes)
+		(effects
+			(font
+				(size 1.27 1.27)
+			)
+			(justify right)
+		)
+	)
+	(hierarchical_label "VR_PA"
+		(shape bidirectional)
+		(at 25.4 43.18 180)
+		(fields_autoplaced yes)
+		(effects
+			(font
+				(size 1.27 1.27)
+			)
+			(justify right)
+		)
+	)
+	(hierarchical_label "RFI_P"
+		(shape output)
+		(at 25.4 114.3 180)
+		(fields_autoplaced yes)
+		(effects
+			(font
+				(size 1.27 1.27)
+			)
+			(justify right)
+		)
+	)
 	(symbol
 		(lib_id "Device:L")
@@
 	(symbol
 		(lib_id "power:+3.3V")
-		(at 109.22 106.68 90)
-		(mirror x)
+		(at 114.3 102.87 0)
+		(mirror y)
 		(unit 1)
 		(exclude_from_sim no)
@@
 		(dnp no)
 		(property "Reference" "#PWR016"
-			(at 113.03 106.68 0)
+			(at 114.3 106.68 0)
 			(effects
 				(font
@@
 		)
 		(property "Value" "+3.3V"
-			(at 106.426 108.966 90)
+			(at 117.094 100.076 90)
 			(effects
 				(font
@@
 		)
 		(property "Footprint" ""
-			(at 109.22 106.68 0)
+			(at 114.3 102.87 0)
 			(effects
 				(font
@@
 		)
 		(property "Datasheet" ""
-			(at 109.22 106.68 0)
+			(at 114.3 102.87 0)
 			(effects
 				(font
@@
 		)
 		(property "Description" "Power symbol creates a global label with name \"+3.3V\""
-			(at 109.22 106.68 0)
+			(at 114.3 102.87 0)
 			(effects
 				(font

Commit message: Update
Other:
- moved on the sheet: C74, C75, C76, C81

Commit message: Update
Parts:
- C10, C11, C12, C13, C15, C18, C20, C21, C22, C4, C40, C41, C42, C43, C5, C51, C6, C78, C79, C8: footprint Capacitor_SMD:C_0805_2012Metric -> Capacitor_SMD:C_0603_1608Metric_Pad1.08x0.95mm_HandSolder
Connections:
- net Y0: now also C12.2, L13.2; no longer C11.2, L12.1
- net Y1: now also C11.2, L12.1; no longer C12.2, L13.2
Other:
- note added: "CHECK!"
Changed lines of the file:
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@@
 	(wire
 		(pts
+			(xy 96.52 68.58) (xy 96.52 72.39)
+		)
+		(stroke
+			(width 0)
+			(type default)
+		)
+	)
+	(wire
+		(pts
 			(xy 252.73 111.76) (xy 256.54 111.76)
 		)
@@
 	(wire
 		(pts
+			(xy 93.98 63.5) (xy 93.98 53.34)
+		)
+		(stroke
+			(width 0)
+			(type default)
+		)
+	)
+	(wire
+		(pts
 			(xy 67.31 66.04) (xy 59.69 66.04)
 		)
@@
 	(wire
 		(pts
+			(xy 96.52 68.58) (xy 87.63 68.58)
+		)
+		(stroke
+			(width 0)
+			(type default)
+		)
+	)
+	(wire
+		(pts
 			(xy 96.52 72.39) (xy 96.52 73.66)
 		)
@@
 	(wire
 		(pts
-			(xy 87.63 68.58) (xy 93.98 68.58)
-		)
-		(stroke
-			(width 0)
-			(type default)
-		)
-	)
-	(wire
-		(pts
 			(xy 146.05 106.68) (xy 156.21 106.68)
 		)
@@
 	(wire
 		(pts
-			(xy 87.63 63.5) (xy 96.52 63.5)
-		)
-		(stroke
-			(width 0)
-			(type default)
-		)
-	)
-	(wire
-		(pts
 			(xy 109.22 40.64) (xy 109.22 46.99)
 		)
@@
 	(wire
 		(pts
-			(xy 93.98 68.58) (xy 93.98 53.34)
-		)
-		(stroke
-			(width 0)
-			(type default)
-		)
-	)
-	(wire
-		(pts
 			(xy 123.19 29.21) (xy 109.22 29.21)
 		)
@@
 	(wire
 		(pts
+			(xy 93.98 63.5) (xy 87.63 63.5)
+		)
+		(stroke
+			(width 0)
+			(type default)
+		)
+	)
+	(wire
+		(pts
 			(xy 115.57 111.76) (xy 138.43 111.76)
 		)
@@
 	(wire
 		(pts
-			(xy 96.52 63.5) (xy 96.52 72.39)
-		)
-		(stroke
-			(width 0)
-			(type default)
-		)
-	)
-	(wire
-		(pts
 			(xy 92.71 153.67) (xy 92.71 156.21)
 		)
@@
 		)
 	)
+	(text "CHECK!"
+		(exclude_from_sim no)
+		(at 92.71 64.008 0)
+		(effects
+			(font
+				(size 1.27 1.27)
+				(thickness 0.254)
+				(bold yes)
+			)
+		)
+	)
 	(label "PA5_INOUTRF"
 		(at 115.57 109.22 0)
@@
 		)
 	)
+	(label "Y1"
+		(at 87.63 63.5 0)
+		(fields_autoplaced yes)
+		(effects
+			(font
+				(size 1.27 1.27)
+			)
+			(justify left bottom)
+		)
+	)
 	(label "PA7_HPLP_CTRL"
 		(at 115.57 111.76 0)
@@
 		)
 	)
+	(label "Y0"
+		(at 87.63 68.58 0)
+		(fields_autoplaced yes)
+		(effects
+			(font
+				(size 1.27 1.27)
+			)
+			(justify left bottom)
+		)
+	)
 	(label "RF1_4"
 		(at 102.87 40.64 0)
@@
 		)
 	)
-	(label "Y0"
-		(at 87.63 68.58 0)
-		(fields_autoplaced yes)
-		(effects
-			(font
-				(size 1.27 1.27)
-			)
-			(justify left bottom)
-		)
-	)
 	(label "RFI_N"
 		(at 25.4 127 0)
@@
 		)
 	)
-	(label "Y1"
-		(at 87.63 63.5 0)
-		(fields_autoplaced yes)
-		(effects
-			(font
-				(size 1.27 1.27)
-			)
-			(justify left bottom)
-		)
-	)
 	(hierarchical_label "RFO_HP"
 		(shape input)
@@
 			)
 		)
-		(property "Footprint" "Capacitor_SMD:C_0805_2012Metric"
+		(property "Footprint" "Capacitor_SMD:C_0603_1608Metric_Pad1.08x0.95mm_HandSolder"
 			(at 33.3248 54.61 0)
 			(effects
@@
 			)
 		)
-		(property "Footprint" "Capacitor_SMD:C_0805_2012Metric"
+		(property "Footprint" "Capacitor_SMD:C_0603_1608Metric_Pad1.08x0.95mm_HandSolder"
 			(at 108.2548 46.99 0)
 			(effects
@@
 			)
 		)
-		(property "Footprint" "Capacitor_SMD:C_0805_2012Metric"
+		(property "Footprint" "Capacitor_SMD:C_0603_1608Metric_Pad1.08x0.95mm_HandSolder"
 			(at 91.7448 156.21 0)
 			(effects
@@
 			)
 		)
-		(property "Footprint" "Capacitor_SMD:C_0805_2012Metric"
+		(property "Footprint" "Capacitor_SMD:C_0603_1608Metric_Pad1.08x0.95mm_HandSolder"
 			(at 42.2148 129.54 0)
 			(effects
@@
 			)
 		)
-		(property "Footprint" "Capacitor_SMD:C_0805_2012Metric"
+		(property "Footprint" "Capacitor_SMD:C_0603_1608Metric_Pad1.08x0.95mm_HandSolder"
 			(at 139.7 152.7048 0)
 			(effects
@@
 			)
 		)
-		(property "Footprint" "Capacitor_SMD:C_0805_2012Metric"
+		(property "Footprint" "Capacitor_SMD:C_0603_1608Metric_Pad1.08x0.95mm_HandSolder"
 			(at 118.4148 156.21 0)
 			(effects
@@
 			)
 		)
-		(property "Footprint" "Capacitor_SMD:C_0805_2012Metric"
+		(property "Footprint" "Capacitor_SMD:C_0603_1608Metric_Pad1.08x0.95mm_HandSolder"
 			(at 132.08 71.4248 0)
 			(effects
@@
 			)
 		)
-		(property "Footprint" "Capacitor_SMD:C_0805_2012Metric"
+		(property "Footprint" "Capacitor_SMD:C_0603_1608Metric_Pad1.08x0.95mm_HandSolder"
 			(at 47.2948 54.61 0)
 			(effects
@@
 			)
 		)
-		(property "Footprint" "Capacitor_SMD:C_0805_2012Metric"
+		(property "Footprint" "Capacitor_SMD:C_0603_1608Metric_Pad1.08x0.95mm_HandSolder"
 			(at 165.1 82.8548 0)
 			(effects
@@
 			)
 		)
-		(property "Footprint" "Capacitor_SMD:C_0805_2012Metric"
+		(property "Footprint" "Capacitor_SMD:C_0603_1608Metric_Pad1.08x0.95mm_HandSolder"
 			(at 195.8848 44.45 0)
 			(effects
@@
 			)
 		)
-		(property "Footprint" "Capacitor_SMD:C_0805_2012Metric"
+		(property "Footprint" "Capacitor_SMD:C_0603_1608Metric_Pad1.08x0.95mm_HandSolder"
 			(at 86.0552 74.93 0)
 			(effects
@@
 			)
 		)
-		(property "Footprint" "Capacitor_SMD:C_0805_2012Metric"
+		(property "Footprint" "Capacitor_SMD:C_0603_1608Metric_Pad1.08x0.95mm_HandSolder"
 			(at 130.81 28.2448 0)
 			(effects
@@
 			)
 		)
-		(property "Footprint" "Capacitor_SMD:C_0805_2012Metric"
+		(property "Footprint" "Capacitor_SMD:C_0603_1608Metric_Pad1.08x0.95mm_HandSolder"
 			(at 197.1548 81.28 0)
 			(effects
@@
 			)
 		)
-		(property "Footprint" "Capacitor_SMD:C_0805_2012Metric"
+		(property "Footprint" "Capacitor_SMD:C_0603_1608Metric_Pad1.08x0.95mm_HandSolder"
 			(at 62.23 113.3348 0)
 			(effects
@@
 			)
 		)
-		(property "Footprint" "Capacitor_SMD:C_0805_2012Metric"
+		(property "Footprint" "Capacitor_SMD:C_0603_1608Metric_Pad1.08x0.95mm_HandSolder"
 			(at 70.1548 53.34 0)
 			(effects
@@
 			)
 		)
-		(property "Footprint" "Capacitor_SMD:C_0805_2012Metric"
+		(property "Footprint" "Capacitor_SMD:C_0603_1608Metric_Pad1.08x0.95mm_HandSolder"
 			(at 88.9 54.3052 0)
 			(effects
@@
 			)
 		)
-		(property "Footprint" "Capacitor_SMD:C_0805_2012Metric"
+		(property "Footprint" "Capacitor_SMD:C_0603_1608Metric_Pad1.08x0.95mm_HandSolder"
 			(at 143.8148 46.99 0)
 			(effects
@@
 			)
 		)
-		(property "Footprint" "Capacitor_SMD:C_0805_2012Metric"
+		(property "Footprint" "Capacitor_SMD:C_0603_1608Metric_Pad1.08x0.95mm_HandSolder"
 			(at 109.5248 90.17 0)
 			(effects
@@
 			)
 		)
-		(property "Footprint" "Capacitor_SMD:C_0805_2012Metric"
+		(property "Footprint" "Capacitor_SMD:C_0603_1608Metric_Pad1.08x0.95mm_HandSolder"
 			(at 163.83 39.6748 0)
 			(effects
@@
 			)
 		)
-		(property "Footprint" "Capacitor_SMD:C_0805_2012Metric"
+		(property "Footprint" "Capacitor_SMD:C_0603_1608Metric_Pad1.08x0.95mm_HandSolder"
 			(at 145.0848 90.17 0)
 			(effects

Commit message: Update
Connections:
- net Y0: now also C11.2, L12.1; no longer C12.2, L13.2
- net Y1: now also C12.2, L13.2; no longer C11.2, L12.1
Other:
- note added: "NX3L1T3157GM,115 Ouputs S OUT CCT HIGH Y1 LP(Y0) LOW Y0 HP(Y1)"
- note added: "RF_Switch_PE42440MLBB-Z V1 (PA7_HPLP_CTRL) V2 (PA5_INOUTRF) OUTPUT CCT 0 0 RFC - RF1 (PIN13) HP 1 0 RFC - RF2 (PIN15) NC 0 1 RFC - RF3 (PIN8) RFIN 1 1 RFC - RF4 (PIN6) LP"
- note removed: "CHECK!"
Changed lines of the file:
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@@
 	)
 	(junction
-		(at 59.69 66.04)
-		(diameter 0)
-		(color 0 0 0 0)
-	)
-	(junction
 		(at 43.18 114.3)
 		(diameter 0)
@@
 	(wire
 		(pts
-			(xy 242.57 127) (xy 242.57 142.24)
+			(xy 242.57 127) (xy 242.57 146.05)
 		)
 		(stroke
@@
 	(wire
 		(pts
-			(xy 96.52 68.58) (xy 96.52 72.39)
+			(xy 96.52 63.5) (xy 96.52 72.39)
 		)
 		(stroke
@@
 	(wire
 		(pts
+			(xy 93.98 53.34) (xy 93.98 68.58)
+		)
+		(stroke
+			(width 0)
+			(type default)
+		)
+	)
+	(wire
+		(pts
 			(xy 109.22 54.61) (xy 109.22 58.42)
 		)
@@
 	(wire
 		(pts
-			(xy 93.98 63.5) (xy 93.98 53.34)
-		)
-		(stroke
-			(width 0)
-			(type default)
-		)
-	)
-	(wire
-		(pts
-			(xy 67.31 66.04) (xy 59.69 66.04)
+			(xy 55.88 66.04) (xy 67.31 66.04)
 		)
 		(stroke
@@
 	(wire
 		(pts
-			(xy 96.52 68.58) (xy 87.63 68.58)
+			(xy 96.52 72.39) (xy 96.52 73.66)
 		)
 		(stroke
@@
 	(wire
 		(pts
-			(xy 96.52 72.39) (xy 96.52 73.66)
+			(xy 93.98 68.58) (xy 87.63 68.58)
 		)
 		(stroke
@@
 	(wire
 		(pts
+			(xy 96.52 63.5) (xy 87.63 63.5)
+		)
+		(stroke
+			(width 0)
+			(type default)
+		)
+	)
+	(wire
+		(pts
 			(xy 198.12 83.82) (xy 218.44 83.82)
 		)
@@
 	(wire
 		(pts
-			(xy 92.71 114.3) (xy 92.71 142.24)
+			(xy 92.71 114.3) (xy 92.71 146.05)
 		)
 		(stroke
@@
 	(wire
 		(pts
-			(xy 93.98 63.5) (xy 87.63 63.5)
-		)
-		(stroke
-			(width 0)
-			(type default)
-		)
-	)
-	(wire
-		(pts
 			(xy 115.57 111.76) (xy 138.43 111.76)
 		)
@@
 	(wire
 		(pts
-			(xy 59.69 66.04) (xy 55.88 66.04)
-		)
-		(stroke
-			(width 0)
-			(type default)
-		)
-	)
-	(wire
-		(pts
 			(xy 43.18 124.46) (xy 43.18 127)
 		)
@@
 	(wire
 		(pts
-			(xy 92.71 142.24) (xy 242.57 142.24)
+			(xy 92.71 146.05) (xy 242.57 146.05)
 		)
 		(stroke
@@
 		)
 	)
-	(text "CHECK!"
+	(text "RF_Switch_PE42440MLBB-Z\nV1 (PA7_HPLP_CTRL)   V2 (PA5_INOUTRF)   OUTPUT                 CCT\n0                    0                  RFC - RF1 (PIN13)      HP\n1                    0                  RFC - RF2 (PIN15)      NC\n0                    1                  RFC - RF3 (PIN8)       RFIN\n1                    1                  RFC - RF4 (PIN6)       LP"
 		(exclude_from_sim no)
-		(at 92.71 64.008 0)
+		(at 204.216 162.814 0)
 		(effects
 			(font
-				(size 1.27 1.27)
-				(thickness 0.254)
-				(bold yes)
+				(size 1 1)
+			)
+			(justify left)
+		)
+	)
+	(text "NX3L1T3157GM,115 Ouputs\nS      OUT    CCT\nHIGH   Y1     LP(Y0)\nLOW    Y0     HP(Y1)"
+		(exclude_from_sim no)
+		(at 46.99 74.93 0)
+		(effects
+			(font
+				(size 1 1)
 			)
+			(justify left)
 		)
 	)
@@
 					(unit 1)
 				)
-			)
-		)
-	)
-	(symbol
-		(lib_id "power:PWR_FLAG")
-		(at 59.69 66.04 0)
-		(unit 1)
-		(exclude_from_sim no)
-		(in_bom yes)
-		(on_board yes)
-		(dnp no)
-		(fields_autoplaced yes)
-		(property "Reference" "#FLG07"
-			(at 59.69 64.135 0)
-			(effects
-				(font
-					(size 1.27 1.27)
-				)
-				(hide yes)
-			)
-		)
-		(property "Value" "PWR_FLAG"
-			(at 59.6901 62.23 90)
-			(effects
-				(font
-					(size 1.27 1.27)
-				)
-				(justify left)
-				(hide yes)
-			)
-		)
-		(property "Footprint" ""
-			(at 59.69 66.04 0)
-			(effects
-				(font
-					(size 1.27 1.27)
-				)
-				(hide yes)
-			)
-		)
-		(property "Datasheet" "~"
-			(at 59.69 66.04 0)
-			(effects
-				(font
-					(size 1.27 1.27)
-				)
-				(hide yes)
-			)
-		)
-		(property "Description" "Special symbol for telling ERC where power comes from"
-			(at 59.69 66.04 0)
-			(effects
-				(font
-					(size 1.27 1.27)
-				)
-				(hide yes)
-			)
-		)
-		(pin "1"
-		)
-		(instances
-			(project "LoRa_Board"
-				(path "/34ccaf76-212c-4f8e-9afa-bb7eea5015e3/3303ad38-3ac3-4e68-96af-2b05d17ec8a5"
-					(reference "#FLG07")
-					(unit 1)
-				)

Commit message: Update
Parts:
- SW2: value Switch_NX3L1T3157GM,115 -> Switch_NX3L1T3157GMZ
Changed lines of the file:
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@@
 			)
 		)
-		(property "Value" "Switch_NX3L1T3157GM,115"
+		(property "Value" "Switch_NX3L1T3157GMZ"
 			(at 77.47 58.42 0)
 			(effects

Commit message: Update Readme file
Other:
- company: (none) -> Peter Hancak
- title: (none) -> LoRa Board
Changed lines of the file:
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@@
 	(generator_version "8.0")
 	(paper "USLetter")
+	(title_block
+		(title "LoRa Board")
+		(date "2026-03-17")
+		(rev "B")
+		(company "Peter Hancak")
+	)
 	(junction
 		(at 196.85 40.64)

Commit message: Update
Parts:
- removed L11: 160n_LQW18ANR16G00, Inductor_SMD:L_0603_1608Metric_Pad1.05x0.95mm_HandSolder, symbol Device:L
- removed L4: 6n8_LQW18AN6N8C00, Inductor_SMD:L_0603_1608Metric_Pad1.05x0.95mm_HandSolder, symbol Device:L
- added L2: 0H, Inductor_SMD:L_0603_1608Metric_Pad1.05x0.95mm_HandSolder, symbol Device:L
- C13: value 3p3_GJM1555C1H220FB01 -> 2p6_CC0402BRNPO9BN3R3
- C15: value 1p2_GJM1555C1H180FB01 -> 4p4_GJM1555C1H180FB01
- C18: value 18p_GJM1555C1H180FB01 -> 5p6_CC0402BRNPO9BN5R6
- C20: value 3p3_GJM1555C1H220FB01 -> 3p6_CC0402BRNPO9BN3R3
- C21: value 2p2_GJM1555C1H200GB01 -> 1p9_CC0402BRNPO9BN2R2
- C22: value 20p_GJM1555C1H200GB01 -> 2p7_CC0402BRNPO9BN2R7
- C40: value 33p_GRM1555C2A221GE01 -> 40p_CC0402GRNPO9BN330
- C41: value 5p6_GJM1555C1H300FB01 -> 5p6_CC0402BRNPO9BN5R6
- C42: value 30p_GJM1555C1H300FB01 -> 3p3_CC0402BRNPO9BN3R3
- C5: value 2p7_GJM1555C1H120FB01 -> 2p7_CC0402BRNPO9BN2R7
- C51: value 220p_GRM1555C2A221GE01 -> 33p_CC0402GRNPO9BN330
- C78: value 1p2_GJM1555C1H180FB01 -> 1p3_GJM1555C1H1R2WB01D
- C79: value 18p_GJM1555C1H180FB01 -> 1p3_CC0402BRNPO9BN1R3
- C8: value 3p6_GJM1555C1H150FB01 -> 3p6_CC0402BRNPO9BN3R6
- L1: value 11n_LQW18ANR12G00 -> 11n_LQW15AN11NG00
- L19: value 8n7_LQW18AN47NG0Z -> 6n1_LQW15AN8N7H00
- L20: value 3n6_LQW18AN12NG0Z -> 4n7_LQW15AN3N6C10
- L21: value 12n_LQW18AN12NG0Z -> 3n_LQW15AN3N0B00
- L22: value 8n7_LQW18AN51NG0Z -> 8n8_LQW15AN8N7H00
- L23: value 51n_LQW18AN51NG0Z -> 8n7_LQW15AN8N7H00
- L8: value 6n8_LQW18AN6N8C00 -> 3n3_LQW15AN3N3C80
Connections:
- net RF1_4: now also L2.2
- net RFO_HP: now also L2.1
- net VR_PA: now also SW2.4 (Z)
Other:
- note added: "RFI Differential Input Impedance 60+j125 Ω"
- note added: "RFO_HP Impedance Matching 10.71 - j1.85 Ohm"
- note added: "RFO_LP Impedance Matching 14.18 - j1.20 Ohm"
- moved on the sheet: C79
