File: RF_ANT.kicad_sch (KiCad schematic)
At the start: 42 parts, among them IC2 RF_Switch_PE42440MLBB-Z, J10 SMA PCB END LAUNCH JACK ROUND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, SW2 Switch_NX3L1T3157GMZ

Commit message: Schematics Update
Parts:
- removed C10: 1p2_GJM1555C1H1R2WB01D, Capacitor_SMD:C_0603_1608Metric_Pad1.08x0.95mm_HandSolder, symbol Device:C
- removed C11, C12, C51: 33p_CC0402GRNPO9BN330, Capacitor_SMD:C_0603_1608Metric_Pad1.08x0.95mm_HandSolder, symbol Device:C
- removed C13: 2p6_CC0402BRNPO9BN3R3, Capacitor_SMD:C_0603_1608Metric_Pad1.08x0.95mm_HandSolder, symbol Device:C
- removed C15: 4p4_GJM1555C1H180FB01, Capacitor_SMD:C_0603_1608Metric_Pad1.08x0.95mm_HandSolder, symbol Device:C
- removed C18, C41: 5p6_CC0402BRNPO9BN5R6, Capacitor_SMD:C_0603_1608Metric_Pad1.08x0.95mm_HandSolder, symbol Device:C
- removed C20: 3p6_CC0402BRNPO9BN3R3, Capacitor_SMD:C_0603_1608Metric_Pad1.08x0.95mm_HandSolder, symbol Device:C
- removed C21: 1p9_CC0402BRNPO9BN2R2, Capacitor_SMD:C_0603_1608Metric_Pad1.08x0.95mm_HandSolder, symbol Device:C
- removed C22, C5: 2p7_CC0402BRNPO9BN2R7, Capacitor_SMD:C_0603_1608Metric_Pad1.08x0.95mm_HandSolder, symbol Device:C
- removed C4: 47n_Murata_GCM155R71E473KA55, Capacitor_SMD:C_0603_1608Metric_Pad1.08x0.95mm_HandSolder, symbol Device:C
- removed C40: 40p_CC0402GRNPO9BN330, Capacitor_SMD:C_0603_1608Metric_Pad1.08x0.95mm_HandSolder, symbol Device:C
- removed C42: 3p3_CC0402BRNPO9BN3R3, Capacitor_SMD:C_0603_1608Metric_Pad1.08x0.95mm_HandSolder, symbol Device:C
- removed C43: 68p_GRM1555C2A221GE01, Capacitor_SMD:C_0603_1608Metric_Pad1.08x0.95mm_HandSolder, symbol Device:C
- removed C6: 68p_Murata_GCM1555C1H680JA16, Capacitor_SMD:C_0603_1608Metric_Pad1.08x0.95mm_HandSolder, symbol Device:C
- removed C74, C76, C80: 10p, Capacitor_SMD:C_0805_2012Metric, symbol Device:C
- removed C75, C77, C81: 1n, Capacitor_SMD:C_0805_2012Metric, symbol Device:C
- removed C78: 1p3_GJM1555C1H1R2WB01D, Capacitor_SMD:C_0603_1608Metric_Pad1.08x0.95mm_HandSolder, symbol Device:C
- removed C79: 1p3_CC0402BRNPO9BN1R3, Capacitor_SMD:C_0603_1608Metric_Pad1.08x0.95mm_HandSolder, symbol Device:C
- removed C8: 3p6_CC0402BRNPO9BN3R6, Capacitor_SMD:C_0603_1608Metric_Pad1.08x0.95mm_HandSolder, symbol Device:C
- removed IC2: RF_Switch_PE42440MLBB-Z, Personal_Project:RF_SWITCH_PE42440_QFN50P300X300X80-17N, symbol Personal_Projects:RF_Switch_PE42440MLBB-Z
- removed J10: SMA PCB END LAUNCH JACK ROUND PO, Personal_Project:SMA Clip Mount Adapter (top), symbol Personal_Projects:SMA PCB END LAUNCH JACK ROUND PO
- removed L1: 11n_LQW15AN11NG00, Inductor_SMD:L_0603_1608Metric_Pad1.05x0.95mm_HandSolder, symbol Device:L
- removed L12: 33n_LQW15AN33NG00, Inductor_SMD:L_0603_1608Metric_Pad1.05x0.95mm_HandSolder, symbol Device:L
- removed L13: 47n_LQW15AN47NJ00, Inductor_SMD:L_0603_1608Metric_Pad1.05x0.95mm_HandSolder, symbol Device:L
- removed L19: 6n1_LQW15AN8N7H00, Inductor_SMD:L_0603_1608Metric_Pad1.05x0.95mm_HandSolder, symbol Device:L
- removed L2: 0H, Inductor_SMD:L_0603_1608Metric_Pad1.05x0.95mm_HandSolder, symbol Device:L
- removed L20: 4n7_LQW15AN3N6C10, Inductor_SMD:L_0603_1608Metric_Pad1.05x0.95mm_HandSolder, symbol Device:L
- removed L21: 3n_LQW15AN3N0B00, Inductor_SMD:L_0603_1608Metric_Pad1.05x0.95mm_HandSolder, symbol Device:L
- removed L22: 8n8_LQW15AN8N7H00, Inductor_SMD:L_0603_1608Metric_Pad1.05x0.95mm_HandSolder, symbol Device:L
- removed L23: 8n7_LQW15AN8N7H00, Inductor_SMD:L_0603_1608Metric_Pad1.05x0.95mm_HandSolder, symbol Device:L
- removed L8: 3n3_LQW15AN3N3C80, Inductor_SMD:L_0603_1608Metric_Pad1.05x0.95mm_HandSolder, symbol Device:L
- removed R1, R2, R8: 100R, Resistor_SMD:R_0805_2012Metric, symbol Device:R
- removed SW2: Switch_NX3L1T3157GMZ, Personal_Project:Switch_NX3L1T3157GM115, symbol Personal_Projects:Switch_NX3L1T3157GM,115
Connections:
- no-connect marks 1 -> 0
Other:
- note removed: "Band pass filter for around 900 MHz"
- note removed: "NX3L1T3157GM,115 Ouputs S OUT CCT HIGH Y1 LP(Y0) LOW Y0 HP(Y1)"
- note removed: "RFI Differential Input Impedance 60+j125 Ω"
- note removed: "RFO_HP Impedance Matching 10.71 - j1.85 Ohm"
- note removed: "RFO_LP Impedance Matching 14.18 - j1.20 Ohm"
- note removed: "RF_Switch_PE42440MLBB-Z V1 (PA7_HPLP_CTRL) V2 (PA5_INOUTRF) OUTPUT CCT 0 0 RFC - RF1 (PIN13) HP 1 0 RFC - RF2 (PIN15) NC 0 1 RFC - RF3 (PIN8) RFIN 1 1 RFC - RF4 (PIN6) LP"
