File: USB.kicad_sch (KiCad schematic)
At the start: 13 parts, among them J2 USB_B_Micro, U6 FT230XS, U7 USBLC6-2SC6

Commit message: Update
Parts:
- removed J2: USB_B_Micro, Connector_USB:USB_Micro-B_XKB_U254-051T-4BH83-F1S, symbol Connector:USB_B_Micro
- removed R17: 100k, Resistor_SMD:R_0805_2012Metric, symbol Device:R
- removed U7: USBLC6-2SC6, Package_TO_SOT_SMD:SOT-23-6, symbol Power_Protection:USBLC6-2SC6
- added J4: USB_C_Receptacle_USB2.0_16P, Connector_USB:USB_C_Receptacle_HRO_TYPE-C-31-M-12, symbol Connector:USB_C_Receptacle_USB2.0_16P
- added R5, R6: 5k1, Resistor_SMD:R_0805_2012Metric, symbol Device:R
- added U1: USBLC6-2SC6, Package_TO_SOT_SMD:SOT-23-6, symbol Power_Protection:USBLC6-2SC6
Connections:
- net GND: now also J4.A1 (GND), J4.A12 (GND), J4.B1 (GND), J4.B12 (GND), J4.S1 (SHIELD), R5.2, R6.2, U1.2 (GND)
- net USB_D2+: now also J4.A6 (D+), J4.B6 (D+), U1.4 (I/O2)
- net USB_D2-: now also J4.A7 (D-), J4.B7 (D-), U1.6 (I/O1)
- net +5V_VBUS_FB renamed USB_VBUS+
- net PA10_USART1_RX renamed UART_RX
- net PA11_USART1_CTS renamed UART_CTS
- net PA12_USART1_RTS renamed UART_RTS
- net PB6_USART1_TX renamed UART_TX
- net USB_D+ renamed USB_D2-_DI
- net USB_D2-_DI: now also U1.1 (I/O1)
- net USB_D- renamed USB_D2+_DI
- net USB_D2+_DI: now also U1.3 (I/O2)
- net VBUS_5V renamed USB_VBUS
- net USB_VBUS: now also J4.A4 (VBUS), J4.A9 (VBUS), J4.B4 (VBUS), J4.B9 (VBUS), U1.5 (VBUS)
- new net: J4.B5 (CC2), R6.1
- new net: J4.A5 (CC1), R5.1
- no-connect marks 4 -> 6
Other:
- moved on the sheet: C14, C19, C3, C38, C44, C48, FB3, R16, R9, U6

Commit message: Update
Parts:
- removed C48: 10p, Capacitor_SMD:C_0805_2012Metric, symbol Device:C
- added C24: 100n, Capacitor_SMD:C_0805_2012Metric, symbol Device:C
Connections:
- net USB_VBUS is gone; now on net USB_VBUS+: FB3.1, J4.A4 (VBUS), J4.A9 (VBUS), J4.B4 (VBUS), J4.B9 (VBUS), U1.5 (VBUS)
- net GND: now also C24.2
- net USB_VBUS+: now also C24.1
Other:
- note added: "600 Ohms @ 100 MHz"
- moved on the sheet: C14, C3, FB3

Commit message: Update
Connections:
- net USB_VBUS+: no longer C24.1, FB3.1, J4.A4 (VBUS), J4.A9 (VBUS), J4.B4 (VBUS), J4.B9 (VBUS), U1.5 (VBUS)
- net CC2: now reaches J4.B5 (CC2), R6.1
- net CC1: now reaches J4.A5 (CC1), R5.1
- new net VBUS: C24.1, FB3.1, J4.A4 (VBUS), J4.A9 (VBUS), J4.B4 (VBUS), J4.B9 (VBUS), U1.5 (VBUS)
Changed lines of the file:
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@@
-	)
-	(junction
-		(at 210.82 97.79)
-		(diameter 0)
-		(color 0 0 0 0)
 	)
 	(junction
@@
 	)
 	(junction
-		(at 210.82 100.33)
-		(diameter 0)
-		(color 0 0 0 0)
-	)
-	(junction
-		(at 210.82 92.71)
-		(diameter 0)
-		(color 0 0 0 0)
-	)
-	(junction
 		(at 224.79 130.81)
 		(diameter 0)
@@
 	)
 	(junction
+		(at 219.71 130.81)
+		(diameter 0)
+		(color 0 0 0 0)
+	)
+	(junction
 		(at 205.74 74.93)
 		(diameter 0)
@@
 	(junction
 		(at 135.89 114.3)
-		(diameter 0)
-		(color 0 0 0 0)
-	)
-	(junction
-		(at 219.71 130.81)
-		(diameter 0)
-		(color 0 0 0 0)
-	)
-	(junction
-		(at 210.82 95.25)
 		(diameter 0)
 		(color 0 0 0 0)
@@
 	(wire
 		(pts
-			(xy 210.82 83.82) (xy 180.34 83.82)
+			(xy 180.34 83.82) (xy 210.82 83.82)
 		)
 		(stroke
@@
 	(wire
 		(pts
-			(xy 219.71 130.81) (xy 187.96 130.81)
+			(xy 187.96 130.81) (xy 219.71 130.81)
 		)
 		(stroke
@@
 	(wire
 		(pts
+			(xy 227.33 130.81) (xy 233.68 130.81)
+		)
+		(stroke
+			(width 0)
+			(type default)
+		)
+	)
+	(wire
+		(pts
 			(xy 77.47 115.57) (xy 77.47 119.38)
 		)
@@
 	(wire
 		(pts
-			(xy 227.33 130.81) (xy 224.79 130.81)
-		)
-		(stroke
-			(width 0)
-			(type default)
-		)
-	)
-	(wire
-		(pts
 			(xy 210.82 86.36) (xy 187.96 86.36)
 		)
@@
 	(wire
 		(pts
-			(xy 212.09 100.33) (xy 210.82 100.33)
-		)
-		(stroke
-			(width 0)
-			(type default)
-		)
-	)
-	(wire
-		(pts
-			(xy 210.82 97.79) (xy 212.09 97.79)
-		)
-		(stroke
-			(width 0)
-			(type default)
-		)
-	)
-	(wire
-		(pts
 			(xy 125.73 97.79) (xy 120.65 97.79)
 		)
@@
 	(wire
 		(pts
-			(xy 210.82 92.71) (xy 205.74 92.71)
+			(xy 205.74 92.71) (xy 210.82 92.71)
 		)
 		(stroke
@@
 	(wire
 		(pts
+			(xy 219.71 130.81) (xy 222.25 130.81)
+		)
+		(stroke
+			(width 0)
+			(type default)
+		)
+	)
+	(wire
+		(pts
 			(xy 82.55 80.01) (xy 82.55 58.42)
 		)
@@
 	(wire
 		(pts
+			(xy 224.79 130.81) (xy 227.33 130.81)
+		)
+		(stroke
+			(width 0)
+			(type default)
+		)
+	)
+	(wire
+		(pts
 			(xy 172.72 95.25) (xy 205.74 95.25)
 		)
@@
 	(wire
 		(pts
-			(xy 212.09 92.71) (xy 210.82 92.71)
-		)
-		(stroke
-			(width 0)
-			(type default)
-		)
-	)
-	(wire
-		(pts
 			(xy 125.73 114.3) (xy 135.89 114.3)
 		)
@@
 	(wire
 		(pts
+			(xy 205.74 69.85) (xy 210.82 69.85)
+		)
+		(stroke
+			(width 0)
+			(type default)
+		)
+	)
+	(wire
+		(pts
 			(xy 167.64 69.85) (xy 167.64 90.17)
 		)
@@
 	(wire
 		(pts
-			(xy 233.68 130.81) (xy 227.33 130.81)
-		)
-		(stroke
-			(width 0)
-			(type default)
-		)
-	)
-	(wire
-		(pts
 			(xy 125.73 97.79) (xy 125.73 102.87)
 		)
@@
 	(wire
 		(pts
-			(xy 222.25 130.81) (xy 219.71 130.81)
-		)
-		(stroke
-			(width 0)
-			(type default)
-		)
-	)
-	(wire
-		(pts
-			(xy 210.82 100.33) (xy 205.74 100.33)
+			(xy 205.74 100.33) (xy 210.82 100.33)
 		)
 		(stroke
@@
 	(wire
 		(pts
-			(xy 210.82 95.25) (xy 212.09 95.25)
-		)
-		(stroke
-			(width 0)
-			(type default)
-		)
-	)
-	(wire
-		(pts
 			(xy 105.41 119.38) (xy 105.41 120.65)
 		)
@@
 	(wire
 		(pts
-			(xy 205.74 69.85) (xy 210.82 69.85)
-		)
-		(stroke
-			(width 0)
-			(type default)
-		)
-	)
-	(wire
-		(pts
 			(xy 205.74 95.25) (xy 210.82 95.25)
 		)
@@
 	(wire
 		(pts
+			(xy 224.79 130.81) (xy 222.25 130.81)
+		)
+		(stroke
+			(width 0)
+			(type default)
+		)
+	)
+	(wire
+		(pts
+			(xy 210.82 72.39) (xy 205.74 72.39)
+		)
+		(stroke
+			(width 0)
+			(type default)
+		)
+	)
+	(wire
+		(pts
+			(xy 205.74 77.47) (xy 205.74 74.93)
+		)
+		(stroke
+			(width 0)
+			(type default)
+		)
+	)
+	(wire
+		(pts
 			(xy 200.66 69.85) (xy 205.74 69.85)
-		)
-		(stroke
-			(width 0)
-			(type default)
-		)
-	)
-	(wire
-		(pts
-			(xy 210.82 72.39) (xy 205.74 72.39)
-		)
-		(stroke
-			(width 0)
-			(type default)
-		)
-	)
-	(wire
-		(pts
-			(xy 205.74 77.47) (xy 205.74 74.93)
-		)
-		(stroke
-			(width 0)
-			(type default)
-		)
-	)
-	(wire
-		(pts
-			(xy 224.79 130.81) (xy 222.25 130.81)
 		)
 		(stroke
@@
 		)
 	)
-	(label "USB_VBUS+"
-		(at 185.42 69.85 0)
-		(fields_autoplaced yes)
-		(effects
-			(font
-				(size 1.27 1.27)
-			)
-			(justify left bottom)
-		)
-	)
 	(label "UART_RX"
 		(at 44.45 90.17 0)
@@
 		)
 	)
+	(label "VBUS"
+		(at 190.5 69.85 180)
+		(effects
+			(font
+				(size 1.27 1.27)
+			)
+			(justify right bottom)
+		)
+	)
 	(label "UART_TX"
 		(at 44.45 87.63 0)
@@
 		)
 	)
+	(label "CC1"
+		(at 210.82 83.82 180)
+		(fields_autoplaced yes)
+		(effects
+			(font
+				(size 1.27 1.27)
+			)
+			(justify right bottom)
+		)
+	)
 	(label "UART_RTS"
 		(at 44.45 92.71 0)
@@
 		)
 	)
+	(label "CC2"
+		(at 210.82 86.36 180)
+		(fields_autoplaced yes)
+		(effects
+			(font
+				(size 1.27 1.27)
+			)
+			(justify right bottom)
+		)
+	)

Commit message: Update
Changed lines of the file:
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@@
+	)
+	(junction
+		(at 110.49 58.42)
+		(diameter 0)
+		(color 0 0 0 0)
 	)
 	(junction
@@
 	(wire
 		(pts
-			(xy 82.55 58.42) (xy 116.84 58.42)
+			(xy 82.55 58.42) (xy 110.49 58.42)
 		)
 		(stroke
@@
 	(wire
 		(pts
+			(xy 110.49 58.42) (xy 116.84 58.42)
+		)
+		(stroke
+			(width 0)
+			(type default)
+		)
+	)
+	(wire
+		(pts
 			(xy 167.64 69.85) (xy 167.64 90.17)
 		)
@@
 			(width 0)
 			(type default)
-		)
-	)
-	(text_box "Place near the USB connector"
-		(exclude_from_sim no)
-		(at 107.95 45.085 0)
-		(size 62.865 34.29)
-		(stroke
-			(width 0)
-			(type dash)
-		)
-		(fill
-			(type none)
-		)
-		(effects
-			(font
-				(size 1.27 1.27)
-			)
-			(justify left top)
 		)
 	)
@@
 					(unit 1)
 				)
+			)
+		)
+	)
+	(symbol
+		(lib_id "power:PWR_FLAG")
+		(at 110.49 58.42 0)
+		(unit 1)
+		(exclude_from_sim no)
+		(in_bom yes)
+		(on_board yes)
+		(dnp no)
+		(fields_autoplaced yes)
+		(property "Reference" "#FLG04"
+			(at 110.49 56.515 0)
+			(effects
+				(font
+					(size 1.27 1.27)
+				)
+				(hide yes)
+			)
+		)
+		(property "Value" "PWR_FLAG"
+			(at 110.4901 54.61 90)
+			(effects
+				(font
+					(size 1.27 1.27)
+				)
+				(justify left)
+				(hide yes)
+			)
+		)
+		(property "Footprint" ""
+			(at 110.49 58.42 0)
+			(effects
+				(font
+					(size 1.27 1.27)
+				)
+				(hide yes)
+			)
+		)
+		(property "Datasheet" "~"
+			(at 110.49 58.42 0)
+			(effects
+				(font
+					(size 1.27 1.27)
+				)
+				(hide yes)
+			)
+		)
+		(property "Description" "Special symbol for telling ERC where power comes from"
+			(at 110.49 58.42 0)
+			(effects
+				(font
+					(size 1.27 1.27)
+				)
+				(hide yes)
+			)
+		)
+		(pin "1"
+		)
+		(instances
+			(project "LoRa_Board"
+				(path "/34ccaf76-212c-4f8e-9afa-bb7eea5015e3/e6eb96f4-8769-4ab2-bb8c-30c74f2fe241"
+					(reference "#FLG04")
+					(unit 1)
+				)

Commit message: Update
Parts:
- added C9: 4u7, Capacitor_SMD:C_0805_2012Metric, symbol Device:C
Connections:
- net GND: now also C9.2
- net VBUS renamed VBUS+
- net VBUS+: now also C9.1
Changed lines of the file:
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@@
+	)
+	(junction
+		(at 167.64 58.42)
+		(diameter 0)
+		(color 0 0 0 0)
 	)
 	(junction
@@
 	)
 	(junction
-		(at 82.55 58.42)
-		(diameter 0)
-		(color 0 0 0 0)
-	)
-	(junction
 		(at 205.74 95.25)
 		(diameter 0)
@@
 	)
 	(junction
+		(at 193.04 49.53)
+		(diameter 0)
+		(color 0 0 0 0)
+	)
+	(junction
 		(at 135.89 114.3)
 		(diameter 0)
@@
 	(wire
 		(pts
+			(xy 167.64 49.53) (xy 167.64 58.42)
+		)
+		(stroke
+			(width 0)
+			(type default)
+		)
+	)
+	(wire
+		(pts
 			(xy 205.74 74.93) (xy 205.74 72.39)
 		)
@@
 	(wire
 		(pts
+			(xy 193.04 49.53) (xy 193.04 52.07)
+		)
+		(stroke
+			(width 0)
+			(type default)
+		)
+	)
+	(wire
+		(pts
 			(xy 135.89 95.25) (xy 162.56 95.25)
 		)
@@
 	(wire
 		(pts
-			(xy 82.55 55.88) (xy 82.55 58.42)
-		)
-		(stroke
-			(width 0)
-			(type default)
-		)
-	)
-	(wire
-		(pts
 			(xy 167.64 58.42) (xy 167.64 69.85)
 		)
@@
 	(wire
 		(pts
+			(xy 193.04 59.69) (xy 193.04 60.96)
+		)
+		(stroke
+			(width 0)
+			(type default)
+		)
+	)
+	(wire
+		(pts
 			(xy 224.79 124.46) (xy 224.79 130.81)
 		)
@@
 	(wire
 		(pts
+			(xy 199.39 49.53) (xy 193.04 49.53)
+		)
+		(stroke
+			(width 0)
+			(type default)
+		)
+	)
+	(wire
+		(pts
 			(xy 125.73 97.79) (xy 125.73 102.87)
 		)
@@
 		(pts
 			(xy 205.74 100.33) (xy 210.82 100.33)
+		)
+		(stroke
+			(width 0)
+			(type default)
+		)
+	)
+	(wire
+		(pts
+			(xy 199.39 46.99) (xy 199.39 49.53)
+		)
+		(stroke
+			(width 0)
+			(type default)
+		)
+	)
+	(wire
+		(pts
+			(xy 193.04 49.53) (xy 167.64 49.53)
 		)
 		(stroke
@@
 		)
 	)
-	(label "VBUS"
+	(label "VBUS+"
 		(at 190.5 69.85 180)
 		(fields_autoplaced yes)
@@
 			)
 			(justify right)
+		)
+	)
+	(symbol
+		(lib_id "power:+3.3V")
+		(at 199.39 46.99 0)
+		(unit 1)
+		(exclude_from_sim no)
+		(in_bom yes)
+		(on_board yes)
+		(dnp no)
+		(property "Reference" "#PWR043"
+			(at 199.39 50.8 0)
+			(effects
+				(font
+					(size 1.27 1.27)
+				)
+				(hide yes)
+			)
+		)
+		(property "Value" "VBUS+"
+			(at 204.47 46.228 0)
+			(effects
+				(font
+					(size 1.27 1.27)
+				)
+			)
+		)
+		(property "Footprint" ""
+			(at 199.39 46.99 0)
+			(effects
+				(font
+					(size 1.27 1.27)
+				)
+				(hide yes)
+			)
+		)
+		(property "Datasheet" ""
+			(at 199.39 46.99 0)
+			(effects
+				(font
+					(size 1.27 1.27)
+				)
+				(hide yes)
+			)
+		)
+		(property "Description" "Power symbol creates a global label with name \"+3.3V\""
+			(at 199.39 46.99 0)
+			(effects
+				(font
+					(size 1.27 1.27)
+				)
+				(hide yes)
+			)
+		)
+		(pin "1"
+		)
+		(instances
+			(project "LoRa_Board"
+				(path "/34ccaf76-212c-4f8e-9afa-bb7eea5015e3/e6eb96f4-8769-4ab2-bb8c-30c74f2fe241"
+					(reference "#PWR043")
+					(unit 1)
+				)
+			)
 		)
 	)
@@
 				(path "/34ccaf76-212c-4f8e-9afa-bb7eea5015e3/e6eb96f4-8769-4ab2-bb8c-30c74f2fe241"
 					(reference "R16")
+					(unit 1)
+				)
+			)
+		)
+	)
+	(symbol
+		(lib_id "Device:C")
+		(at 193.04 55.88 0)
+		(mirror y)
+		(unit 1)
+		(exclude_from_sim no)
+		(in_bom yes)
+		(on_board yes)
+		(dnp no)
+		(property "Reference" "C9"
+			(at 192.024 53.594 0)
+			(effects
+				(font
+					(size 1.27 1.27)
+				)
+				(justify left)
+			)
+		)
+		(property "Value" "4u7"
+			(at 192.278 58.42 0)
+			(effects
+				(font
+					(size 1.27 1.27)
+				)
+				(justify left)
+			)
+		)
+		(property "Footprint" "Capacitor_SMD:C_0805_2012Metric"
+			(at 192.0748 59.69 0)
+			(effects
+				(font
+					(size 1.27 1.27)
+				)
+				(hide yes)
+			)
+		)
+		(property "Datasheet" "~"
+			(at 193.04 55.88 0)
+			(effects
+				(font
+					(size 1.27 1.27)
+				)
+				(hide yes)
+			)
+		)
+		(property "Description" "Unpolarized capacitor"
+			(at 193.04 55.88 0)
+			(effects
+				(font
+					(size 1.27 1.27)
+				)
+				(hide yes)
+			)
+		)
+		(pin "1"
+		)
+		(pin "2"
+		)
+		(instances
+			(project "LoRa_Board"
+				(path "/34ccaf76-212c-4f8e-9afa-bb7eea5015e3/e6eb96f4-8769-4ab2-bb8c-30c74f2fe241"
+					(reference "C9")
 					(unit 1)
 				)
@@
 	)
 	(symbol
-		(lib_id "power:+3.3V")
-		(at 82.55 55.88 0)
-		(unit 1)
-		(exclude_from_sim no)
-		(in_bom yes)
-		(on_board yes)
-		(dnp no)
-		(property "Reference" "#PWR051"
-			(at 82.55 59.69 0)
-			(effects
-				(font
-					(size 1.27 1.27)
-				)
-				(hide yes)
-			)
-		)
-		(property "Value" "USB_VBUS+"
-			(at 89.916 55.118 0)
-			(effects
-				(font
-					(size 1.27 1.27)
-				)
-			)
-		)
-		(property "Footprint" ""
-			(at 82.55 55.88 0)
-			(effects
-				(font
-					(size 1.27 1.27)
-				)
-				(hide yes)
-			)
-		)
-		(property "Datasheet" ""
-			(at 82.55 55.88 0)
-			(effects
-				(font
-					(size 1.27 1.27)
-				)
-				(hide yes)
-			)
-		)
-		(property "Description" "Power symbol creates a global label with name \"+3.3V\""
-			(at 82.55 55.88 0)
-			(effects
-				(font
-					(size 1.27 1.27)
-				)
-				(hide yes)
-			)
-		)
-		(pin "1"
-		)
-		(instances
-			(project "LoRa_Board"
-				(path "/34ccaf76-212c-4f8e-9afa-bb7eea5015e3/e6eb96f4-8769-4ab2-bb8c-30c74f2fe241"
-					(reference "#PWR051")
-					(unit 1)
-				)
-			)
-		)
-	)
-	(symbol
 		(lib_id "Interface_USB:FT230XS")
 		(at 80.01 97.79 0)
@@
 					(unit 1)
 				)
+			)
+		)
+	)
+	(symbol
+		(lib_id "power:GND")
+		(at 193.04 60.96 0)
+		(mirror y)
+		(unit 1)
+		(exclude_from_sim no)
+		(in_bom yes)
+		(on_board yes)
+		(dnp no)
+		(property "Reference" "#PWR051"
+			(at 193.04 67.31 0)
+			(effects
+				(font
+					(size 1.27 1.27)
+				)
+				(hide yes)
+			)
+		)
+		(property "Value" "GND"
+			(at 195.58 60.96 90)
+			(effects
+				(font
+					(size 1.27 1.27)
+				)
+				(justify left)
+				(hide yes)
+			)
+		)
+		(property "Footprint" ""
+			(at 193.04 60.96 0)
+			(effects
+				(font
+					(size 1.27 1.27)
+				)
+				(hide yes)
+			)
+		)
+		(property "Datasheet" ""
+			(at 193.04 60.96 0)
+			(effects
+				(font
+					(size 1.27 1.27)
+				)
+				(hide yes)
+			)
+		)
+		(property "Description" "Power symbol creates a global label with name \"GND\" , ground"
+			(at 193.04 60.96 0)
+			(effects
+				(font
+					(size 1.27 1.27)
+				)
+				(hide yes)
+			)
+		)
+		(pin "1"
+		)
+		(instances
+			(project "LoRa_Board"
+				(path "/34ccaf76-212c-4f8e-9afa-bb7eea5015e3/e6eb96f4-8769-4ab2-bb8c-30c74f2fe241"
+					(reference "#PWR051")
+					(unit 1)
+				)

Commit message: Update Readme file
Other:
- note removed: "FT230XS as close as possible to USB port"
- note removed: "VBUS is the voltage from the USB connector (5V)"
- company: (none) -> Peter Hancak
- title: (none) -> LoRa Board
Changed lines of the file:
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@@
 	(generator_version "8.0")
 	(paper "USLetter")
+	(title_block
+		(title "LoRa Board")
+		(date "2026-03-17")
+		(rev "B")
+		(company "Peter Hancak")
+	)
 	(junction
 		(at 205.74 97.79)
@@
 			(width 0)
 			(type default)
-		)
-	)
-	(text "FT230XS as close as possible\nto USB port"
-		(exclude_from_sim no)
-		(at 132.334 123.444 0)
-		(effects
-			(font
-				(size 1.27 1.27)
-			)
 		)
 	)
@@
 		)
 	)
-	(text "VBUS is the voltage from\nthe USB connector (5V)"
-		(exclude_from_sim no)
-		(at 80.01 67.818 0)
-		(effects
-			(font
-				(size 1.27 1.27)
-			)
-			(justify right bottom)
-		)
-	)
