File: USB.kicad_sch (KiCad schematic)
At the start: 21 parts, among them J4 USB_C_Receptacle_USB2.0_16P, J6 VREGIN_HDR, J8 CP2102N_HDR, U1 USBLC6-2SC6, U5 CP2102N-A02-GQFN24R

Commit message: PCB Layout
Parts:
- added C69: 100n, Capacitor_SMD:C_0805_2012Metric, symbol Device:C
- added J3: CP2102N_NRST, symbol Connector_Generic:Conn_01x02
- J6: footprint (none) -> Connector_PinHeader_2.54mm:PinHeader_1x03_P2.54mm_Vertical
- J8: footprint (none) -> Connector_PinHeader_2.54mm:PinHeader_2x06_P2.54mm_Horizontal
- R11, R16, R5, R6, R9: footprint Resistor_SMD:R_0805_2012Metric -> Resistor_SMD:R_0603_1608Metric
Connections:
- net DCD: now also J8.8 (Pin_8); no longer J8.2 (Pin_2)
- net DSR: now also J8.12 (Pin_12); no longer J8.6 (Pin_6)
- net DTR: now also J8.10 (Pin_10); no longer J8.4 (Pin_4)
- net GND: now also J4.SH (SHIELD), J8.5 (Pin_5), C69.2; no longer J4.S1 (SHIELD)
- net GPIO.2/RS485: now also J8.4 (Pin_4); no longer J8.10 (Pin_10)
- net RI/CLK: now also J8.6 (Pin_6); no longer J8.12 (Pin_12)
- net SUSPEND: now also J8.2 (Pin_2); no longer J8.8 (Pin_8)
- net SUSPENDb: now also J8.1 (Pin_1)
- net CP2102N_VBUS: now reaches R17.2, R19.1, U5.8 (VBUS)
- net CP2102N_D-: now reaches R9.2, U5.4 (D-)
- net CP2102N_D+: now reaches R16.2, U5.3 (D+)
- net CP2102N_VREGIN: now reaches C63.1, C64.1, J6.2 (Pin_2), U5.7 (VREGIN)
- net GPIO.0_/_TXT renamed GPIO.0_TXT
- net GPIO.0_TXT: now also J3.1 (Pin_1); no longer J8.5 (Pin_5)
- net GPIO.1_/_RXT renamed GPIO.1_RXT
- net GPIO.1_RXT: no longer J8.1 (Pin_1)
- net RSTb: no longer names the net of R11.2, U5.9 (RSTb)
- net RSTb: now also C69.1
- new net CP2102N_NRST: J3.2 (Pin_2)

Commit message: Power domain update
Parts:
- C63, C64, C69: footprint Capacitor_SMD:C_0805_2012Metric -> Capacitor_SMD:C_0603_1608Metric
- J3: footprint (none) -> Connector_PinHeader_2.54mm:PinHeader_1x02_P2.54mm_Vertical
Connections:
- net SUSPEND: now also J8.1 (Pin_1); no longer J8.2 (Pin_2)
- net SUSPENDb: now also J8.2 (Pin_2); no longer J8.1 (Pin_1)
- net RSTb: now reaches C69.1, R11.2, U5.9 (RSTb)
- net +3.3VIO renamed +3.3V
