File: Power_Management.kicad_sch (KiCad schematic)
At the start: 21 parts, among them J1 JST_XH_2.54_Plug_5V+, J11 Coin Battery Jumper, Q1 MOSFET_SI2333DDS-T1-BE3

Commit message: Update
Parts:
- removed C1: 1u, Capacitor_SMD:C_0805_2012Metric, symbol Device:C
- removed C16: 10n, Capacitor_SMD:C_0805_2012Metric, symbol Device:C
- removed C37: 2u2, Capacitor_SMD:C_0805_2012Metric, symbol Device:C
- removed C39: 1uF, Capacitor_SMD:C_0805_2012Metric, symbol Device:C
- removed C45, C49: 47u, Capacitor_SMD:C_0805_2012Metric, symbol Device:C_Polarized
- removed C46, C47: 10n_X7R, Capacitor_SMD:C_0805_2012Metric, symbol Device:C
- removed D3: SMAJ6.0A, Personal_Project:DO-214AC-2, symbol Personal_Projects:DIODE_SMAJ6.0A
- removed FB2: BLM21PG601SN1D_0805, Capacitor_SMD:C_0805_2012Metric, symbol Device:FerriteBead
- removed J1: JST_XH_2.54_Plug_5V+, Personal_Project:Connector_Power2pin_SHDRRA2W80P0X250_1X2_740X1150X610P, symbol Personal_Projects:Connector_Power2pin_JST_XH_2.54_Plug
- removed LDO1: LDO_LDLN050PU33R, Package_DFN_QFN:DFN-8-1EP_3x3mm_P0.65mm_EP1.7x2.05mm, symbol Personal_Projects:LDO_LDLN050PUR
- removed Q1: MOSFET_SI2333DDS-T1-BE3, Personal_Project:MOSFET_ SI2333DDS_SOT_DS-T1-BE3_VIS, symbol Personal_Projects:MOSFET_SI2333DDS-T1-BE3
- removed R3: 100k, Resistor_SMD:R_0805_2012Metric, symbol Device:R
- removed S2: Switch_WS-SLSU SMT Mini Slide, Personal_Project:Switch_WS-SLSU SMT Mini Slide, symbol Personal_Projects:Switch_WS-SLSU SMT Mini Slide
- removed U3: ~, Personal_Project:Button_KMR231GLFS, symbol Personal_Projects:Button_KMR231GLFS
- removed VS2: VS_STM1818TWX7F, Personal_Project:SOT-23-3_SOT103P237X112-3N, symbol Personal_Projects:VS_STM1813LWX7F
- removed Z1: Diode_BZX84C6V2-7-F, Personal_Project:Diode_BZX84C6V2_SOT96P240X110-3N, symbol Personal_Projects:Diode_BZX84C6V2-7-F
- added C17: 10n, Capacitor_SMD:C_0805_2012Metric, symbol Device:C
- added C2: 1u, Capacitor_SMD:C_0805_2012Metric, symbol Device:C
- added C33: 2u2, Capacitor_SMD:C_0805_2012Metric, symbol Device:C
- added C34, C50: 47u, Capacitor_SMD:C_0805_2012Metric, symbol Device:C_Polarized
- added C35, C36: 10n_X7R, Capacitor_SMD:C_0805_2012Metric, symbol Device:C
- added D1: SMAJ6.0A, Personal_Project:DO-214AC-2, symbol Personal_Projects:DIODE_SMAJ6.0A
- added FB1: BLM21PG601SN1D_0805, Capacitor_SMD:C_0805_2012Metric, symbol Device:FerriteBead
- added J8: PWR_SRC_JMP, Connector_PinHeader_2.54mm:PinHeader_1x03_P2.54mm_Vertical, symbol Connector_Generic:Conn_01x03
- added JST1: JST_S3B-XH-2.54, Personal_Project:JST_S3B-XH-SHDRRA3W64P0X250_1X3_990X1150X610P, symbol Personal_Projects:JST_S3B-XH-A-1_LF_SN
- added LDO2: LDO_LDLN050PU33R, Package_DFN_QFN:DFN-8-1EP_3x3mm_P0.65mm_EP1.7x2.05mm, symbol Personal_Projects:LDO_LDLN050PUR
- added Q2: MOSFET_SI2333DDS-T1-BE3, Personal_Project:MOSFET_ SI2333DDS_SOT_DS-T1-BE3_VIS, symbol Personal_Projects:MOSFET_SI2333DDS-T1-BE3
- added R7: 100k, Resistor_SMD:R_0805_2012Metric, symbol Device:R
- added U3: SN74LVC1G07DBVR, Package_TO_SOT_SMD:SOT-23-5, symbol 74xGxx:74LVC1G07
- added VS1: VS_STM1818TWX7F, Personal_Project:SOT-23-3_SOT103P237X112-3N, symbol Personal_Projects:VS_STM1813LWX7F
- added Z3: Diode_BZX84C6V2-7-F, Personal_Project:Diode_BZX84C6V2_SOT96P240X110-3N, symbol Personal_Projects:Diode_BZX84C6V2-7-F
Connections:
- net +3.3V: now also C33.1, C34.2, C35.1, FB1.1, LDO2.1 (OUT), U3.5 (VCC), VS1.2 (VCC)
- net GND: now also C17.2, C2.2, C33.2, C34.1, C35.2, C36.2, C50.1, D1.2 (A), JST1.2 (PWR-), LDO2.4 (GND_1), LDO2.9 (GND_2), R7.2, U3.3 (GND), VS1.3 (VSS)
- net VBAT renamed VBAT+
- new net: C17.1, LDO2.3 (FB)
- new net *RST: U3.4, VS1.1 (~{RST})
- new net +3V3A: C36.1, C50.2, FB1.2
- new net PWR+: JST1.1 (PWR+), Q2.3 (D)
- new net PWR+_GATE: Q2.1 (G), R7.1, Z3.1 (A)
- new net PWR+_PP: J8.2 (Pin_2), Q2.2 (S), Z3.3 (K)
- new net PWR+_PS: C2.1, D1.1 (K), J8.1 (Pin_1), LDO2.5 (EN), LDO2.8 (IN)
- new net RST_PWR: JST1.3 (RST), U3.2
- new net USB_VBUS+: J8.3 (Pin_3)
- no-connect marks 9 -> 5
Other:
- note added: "Power can be sourced from USB or Power connector"
- note removed: "Input voltage range: 5V (Exact)"
- note removed: "ON/OFF Switch"
- note removed: "Pin 2 connects to one or three"
- note removed: "VOUT​=1.208⋅(1+31600/10000)≈5.0253 V"

Commit message: Update
Parts:
- removed C34, C50: 47u, Capacitor_SMD:C_0805_2012Metric, symbol Device:C_Polarized
- removed C35, C36: 10n_X7R, Capacitor_SMD:C_0805_2012Metric, symbol Device:C
- removed FB1: BLM21PG601SN1D_0805, Capacitor_SMD:C_0805_2012Metric, symbol Device:FerriteBead
- added C26, C39: 100n, Capacitor_SMD:C_0805_2012Metric, symbol Device:C
- added C45: 4u7, Capacitor_SMD:C_0805_2012Metric, symbol Device:C
- added FB2: BLM21AG121BH1D, Capacitor_SMD:C_0805_2012Metric, symbol Device:FerriteBead
Connections:
- net +3.3V: now also C26.1, FB2.2
- net GND: now also C26.2, C39.2, C45.2
- new net +3.3VA: C39.1, C45.1, FB2.1
Other:
- note added: "120Ohm@100MHz"
- note added: "Need further isolation of the digital domain VDD from the analog domain VDDA."
- note removed: "To generate 3V3"
- moved on the sheet: C17, C2, C33, LDO2, U3, VS1

Commit message: Update
Parts:
- added C34: 100n, Capacitor_SMD:C_0805_2012Metric, symbol Device:C
Connections:
- net GND: now also C34.2
- net PWR+_PP: now also J8.1 (Pin_1); no longer J8.2 (Pin_2)
- net PWR+_PS: now also J8.2 (Pin_2); no longer J8.1 (Pin_1)
- net RST_PWR: now also C34.1
Other:
- moved on the sheet: J8
Changed lines of the file:
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@@
 	)
 	(junction
+		(at 165.1 45.72)
+		(diameter 0)
+		(color 0 0 0 0)
+	)
+	(junction
 		(at 228.6 100.33)
 		(diameter 0)
@@
 	)
 	(junction
+		(at 176.53 139.7)
+		(diameter 0)
+		(color 0 0 0 0)
+	)
+	(junction
 		(at 86.36 118.11)
 		(diameter 0)
@@
 	)
 	(junction
-		(at 165.1 45.72)
+		(at 185.42 151.13)
 		(diameter 0)
 		(color 0 0 0 0)
@@
 	(wire
 		(pts
+			(xy 181.61 48.26) (xy 175.26 48.26)
+		)
+		(stroke
+			(width 0)
+			(type default)
+		)
+	)
+	(wire
+		(pts
+			(xy 185.42 151.13) (xy 185.42 152.4)
+		)
+		(stroke
+			(width 0)
+			(type default)
+		)
+	)
+	(wire
+		(pts
 			(xy 49.53 166.37) (xy 49.53 167.64)
 		)
@@
 	(wire
 		(pts
+			(xy 185.42 147.32) (xy 185.42 151.13)
+		)
+		(stroke
+			(width 0)
+			(type default)
+		)
+	)
+	(wire
+		(pts
 			(xy 40.64 100.33) (xy 76.2 100.33)
 		)
@@
 	(wire
 		(pts
-			(xy 175.26 36.83) (xy 194.31 36.83)
+			(xy 175.26 38.1) (xy 194.31 38.1)
 		)
 		(stroke
@@
 	(wire
 		(pts
+			(xy 165.1 45.72) (xy 181.61 45.72)
+		)
+		(stroke
+			(width 0)
+			(type default)
+		)
+	)
+	(wire
+		(pts
+			(xy 176.53 139.7) (xy 180.34 139.7)
+		)
+		(stroke
+			(width 0)
+			(type default)
+		)
+	)
+	(wire
+		(pts
 			(xy 114.3 100.33) (xy 130.81 100.33)
 		)
@@
 	(wire
 		(pts
-			(xy 175.26 43.18) (xy 175.26 36.83)
-		)
-		(stroke
-			(width 0)
-			(type default)
-		)
-	)
-	(wire
-		(pts
 			(xy 130.81 55.88) (xy 143.51 55.88)
 		)
@@
 	(wire
 		(pts
-			(xy 194.31 36.83) (xy 194.31 45.72)
-		)
-		(stroke
-			(width 0)
-			(type default)
-		)
-	)
-	(wire
-		(pts
-			(xy 185.42 147.32) (xy 185.42 148.59)
+			(xy 194.31 38.1) (xy 194.31 45.72)
 		)
 		(stroke
@@
 	(wire
 		(pts
-			(xy 171.45 139.7) (xy 180.34 139.7)
+			(xy 163.83 139.7) (xy 176.53 139.7)
 		)
 		(stroke
@@
 	(wire
 		(pts
-			(xy 181.61 43.18) (xy 175.26 43.18)
+			(xy 115.57 118.11) (xy 86.36 118.11)
 		)
 		(stroke
@@
 	(wire
 		(pts
-			(xy 115.57 118.11) (xy 86.36 118.11)
+			(xy 176.53 151.13) (xy 185.42 151.13)
 		)
 		(stroke
@@
 	(wire
 		(pts
-			(xy 130.81 55.88) (xy 130.81 59.69)
+			(xy 176.53 148.59) (xy 176.53 151.13)
 		)
 		(stroke
@@
 	(wire
 		(pts
-			(xy 228.6 113.03) (xy 228.6 110.49)
+			(xy 175.26 48.26) (xy 175.26 38.1)
 		)
 		(stroke
@@
 	(wire
 		(pts
-			(xy 165.1 45.72) (xy 181.61 45.72)
+			(xy 130.81 55.88) (xy 130.81 59.69)
+		)
+		(stroke
+			(width 0)
+			(type default)
+		)
+	)
+	(wire
+		(pts
+			(xy 228.6 113.03) (xy 228.6 110.49)
 		)
 		(stroke
@@
 	(wire
 		(pts
+			(xy 176.53 139.7) (xy 176.53 140.97)
+		)
+		(stroke
+			(width 0)
+			(type default)
+		)
+	)
+	(wire
+		(pts
 			(xy 118.11 55.88) (xy 130.81 55.88)
 		)
@@
 	(wire
 		(pts
-			(xy 170.18 48.26) (xy 181.61 48.26)
+			(xy 170.18 50.8) (xy 181.61 50.8)
 		)
 		(stroke
@@
 	)
 	(label "RST_PWR"
-		(at 171.45 139.7 0)
+		(at 163.83 139.7 0)
 		(fields_autoplaced yes)
 		(effects
@@
 	)
 	(symbol
+		(lib_id "Device:C")
+		(at 176.53 144.78 0)
+		(mirror y)
+		(unit 1)
+		(exclude_from_sim no)
+		(in_bom yes)
+		(on_board yes)
+		(dnp no)
+		(property "Reference" "C34"
+			(at 175.768 142.494 0)
+			(effects
+				(font
+					(size 1.27 1.27)
+				)
+				(justify left)
+			)
+		)
+		(property "Value" "100n"
+			(at 175.514 147.32 0)
+			(effects
+				(font
+					(size 1.27 1.27)
+				)
+				(justify left)
+			)
+		)
+		(property "Footprint" "Capacitor_SMD:C_0805_2012Metric"
+			(at 175.5648 148.59 0)
+			(effects
+				(font
+					(size 1.27 1.27)
+				)
+				(hide yes)
+			)
+		)
+		(property "Datasheet" "~"
+			(at 176.53 144.78 0)
+			(effects
+				(font
+					(size 1.27 1.27)
+				)
+				(hide yes)
+			)
+		)
+		(property "Description" "Unpolarized capacitor"
+			(at 176.53 144.78 0)
+			(effects
+				(font
+					(size 1.27 1.27)
+				)
+				(hide yes)
+			)
+		)
+		(pin "1"
+		)
+		(pin "2"
+		)
+		(instances
+			(project "LoRa_Board"
+				(path "/34ccaf76-212c-4f8e-9afa-bb7eea5015e3/c04c6a26-8055-4d4b-aa4b-63838eda4582"
+					(reference "C34")
+					(unit 1)
+				)
+			)
+		)
+	)
+	(symbol
 		(lib_id "power:GND")
 		(at 228.6 114.3 0)
@@
 	(symbol
 		(lib_id "power:GND")
-		(at 185.42 148.59 0)
+		(at 185.42 152.4 0)
 		(mirror y)
 		(unit 1)
@@
 		(dnp no)
 		(property "Reference" "#PWR028"
-			(at 185.42 154.94 0)
+			(at 185.42 158.75 0)
 			(effects
 				(font
@@
 		)
 		(property "Value" "GND"
-			(at 187.96 151.638 90)
+			(at 187.96 155.448 90)
 			(effects
 				(font
@@
 		)
 		(property "Footprint" ""
-			(at 185.42 148.59 0)
+			(at 185.42 152.4 0)
 			(effects
 				(font
@@
 		)
 		(property "Datasheet" ""
-			(at 185.42 148.59 0)
+			(at 185.42 152.4 0)
 			(effects
 				(font
@@
 		)
 		(property "Description" "Power symbol creates a global label with name \"GND\" , ground"
-			(at 185.42 148.59 0)
+			(at 185.42 152.4 0)
 			(effects
 				(font
@@
 	(symbol
 		(lib_id "power:+3.3V")
-		(at 170.18 48.26 90)
+		(at 170.18 50.8 90)
 		(unit 1)
 		(exclude_from_sim no)
@@
 		(dnp no)
 		(property "Reference" "#PWR081"
-			(at 173.99 48.26 0)
+			(at 173.99 50.8 0)
 			(effects
 				(font
@@
 		)
 		(property "Value" "USB_VBUS+"
-			(at 176.022 46.99 90)
+			(at 176.022 49.53 90)
 			(effects
 				(font
@@
 		)
 		(property "Footprint" ""
-			(at 170.18 48.26 0)
+			(at 170.18 50.8 0)
 			(effects
 				(font
@@
 		)
 		(property "Datasheet" ""
-			(at 170.18 48.26 0)
+			(at 170.18 50.8 0)
 			(effects
 				(font
@@
 		)
 		(property "Description" "Power symbol creates a global label with name \"+3.3V\""
-			(at 170.18 48.26 0)
+			(at 170.18 50.8 0)
 			(effects
 				(font
@@
 	(symbol
 		(lib_id "Connector_Generic:Conn_01x03")
-		(at 186.69 45.72 0)
+		(at 186.69 48.26 0)
 		(unit 1)
 		(exclude_from_sim no)
@@
 		(dnp no)
 		(property "Reference" "J8"
-			(at 184.912 40.132 0)
+			(at 184.912 42.672 0)
 			(effects
 				(font
@@
 		)
 		(property "Value" "PWR_SRC_JMP"
-			(at 178.562 51.562 0)
+			(at 178.562 54.102 0)
 			(effects
 				(font
@@
 		)
 		(property "Footprint" "Connector_PinHeader_2.54mm:PinHeader_1x03_P2.54mm_Vertical"
-			(at 186.69 45.72 0)
+			(at 186.69 48.26 0)
 			(effects
 				(font
@@
 		)
 		(property "Datasheet" "~"
-			(at 186.69 45.72 0)
+			(at 186.69 48.26 0)
 			(effects
 				(font
@@
 		)
 		(property "Description" "Generic connector, single row, 01x03, script generated (kicad-library-utils/schlib/autogen/connector/)"
-			(at 186.69 45.72 0)
+			(at 186.69 48.26 0)
 			(effects
 				(font

Commit message: Update
Parts:
- removed BH2: Battery_Holder_1060TR, Personal_Project:Battery_Holder_1060TR, symbol Personal_Projects:Battery_Holder_1060TR
- removed C9: 100n, Capacitor_SMD:C_0805_2012Metric, symbol Device:C
- removed J11: Coin Battery Jumper, Connector_PinHeader_2.54mm:PinHeader_1x03_P2.54mm_Vertical, symbol Connector_Generic:Conn_01x03
Connections:
- no-connect marks 5 -> 4
Other:
- note removed: "EP is optional adhesive zone"

Commit message: Update
Connections:
- net USB_VBUS+ renamed VBUS+
Changed lines of the file:
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@@
 	(wire
 		(pts
-			(xy 170.18 50.8) (xy 181.61 50.8)
+			(xy 171.45 50.8) (xy 181.61 50.8)
 		)
 		(stroke
@@
 	)
 	(symbol
+		(lib_id "power:+3.3V")
+		(at 171.45 50.8 90)
+		(unit 1)
+		(exclude_from_sim no)
+		(in_bom yes)
+		(on_board yes)
+		(dnp no)
+		(property "Reference" "#PWR045"
+			(at 175.26 50.8 0)
+			(effects
+				(font
+					(size 1.27 1.27)
+				)
+				(hide yes)
+			)
+		)
+		(property "Value" "VBUS+"
+			(at 174.244 49.53 90)
+			(effects
+				(font
+					(size 1.27 1.27)
+				)
+			)
+		)
+		(property "Footprint" ""
+			(at 171.45 50.8 0)
+			(effects
+				(font
+					(size 1.27 1.27)
+				)
+				(hide yes)
+			)
+		)
+		(property "Datasheet" ""
+			(at 171.45 50.8 0)
+			(effects
+				(font
+					(size 1.27 1.27)
+				)
+				(hide yes)
+			)
+		)
+		(property "Description" "Power symbol creates a global label with name \"+3.3V\""
+			(at 171.45 50.8 0)
+			(effects
+				(font
+					(size 1.27 1.27)
+				)
+				(hide yes)
+			)
+		)
+		(pin "1"
+		)
+		(instances
+			(project "LoRa_Board"
+				(path "/34ccaf76-212c-4f8e-9afa-bb7eea5015e3/c04c6a26-8055-4d4b-aa4b-63838eda4582"
+					(reference "#PWR045")
+					(unit 1)
+				)
+			)
+		)
+	)
+	(symbol
 		(lib_id "power:GND")
 		(at 86.36 119.38 0)
@@
 					(unit 1)
 				)
-			)
-		)
-	)
-	(symbol
-		(lib_id "power:+3.3V")
-		(at 170.18 50.8 90)
-		(unit 1)
-		(exclude_from_sim no)
-		(in_bom yes)
-		(on_board yes)
-		(dnp no)
-		(property "Reference" "#PWR081"
-			(at 173.99 50.8 0)
-			(effects
-				(font
-					(size 1.27 1.27)
-				)
-				(hide yes)
-			)
-		)
-		(property "Value" "USB_VBUS+"
-			(at 176.022 49.53 90)
-			(effects
-				(font
-					(size 1.27 1.27)
-				)
-			)
-		)
-		(property "Footprint" ""
-			(at 170.18 50.8 0)
-			(effects
-				(font
-					(size 1.27 1.27)
-				)
-				(hide yes)
-			)
-		)
-		(property "Datasheet" ""
-			(at 170.18 50.8 0)
-			(effects
-				(font
-					(size 1.27 1.27)
-				)
-				(hide yes)
-			)
-		)
-		(property "Description" "Power symbol creates a global label with name \"+3.3V\""
-			(at 170.18 50.8 0)
-			(effects
-				(font
-					(size 1.27 1.27)
-				)
-				(hide yes)
-			)
-		)
-		(pin "1"
-		)
-		(instances
-			(project "LoRa_Board"
-				(path "/34ccaf76-212c-4f8e-9afa-bb7eea5015e3/c04c6a26-8055-4d4b-aa4b-63838eda4582"
-					(reference "#PWR081")
-					(unit 1)
-				)

Commit message: Update Readme file
Other:
- company: (none) -> Peter Hancak
- title: (none) -> LoRa Board
Changed lines of the file:
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@@
 	(generator_version "8.0")
 	(paper "USLetter")
+	(title_block
+		(title "LoRa Board")
+		(date "2026-03-17")
+		(rev "B")
+		(company "Peter Hancak")
+	)
 	(junction
 		(at 137.16 100.33)
@@
 			)
 			(justify left top)
-		)
-	)
-	(text_box "Notes:\nThe plan for the popower input is to filter the USB VBUS using ferrite bead along with decoupling capacitors that will then supply a 3V3 LDO. The ouptut will supply VDD digital domain which will e filtered again using ferritte bead and decoupling capacitors before connecting to VDDA the annalog domain.\n\n- USB-C VBUS filtered using FB, C\n- LDO 3V3\n- Supply VDD  digital domain\n- Isolate digital domain switching from analog domain by filtering again using FB, C \n\nFerrite Beads\n- 600Ohm@100MHz Used for VBUS to isolate the voltage rail noise\n- 120Ohm@100MHz Used to isolate the VDD digital domain transients  "
-		(exclude_from_sim no)
-		(at 98.425 156.21 0)
-		(size 53.975 36.195)
-		(stroke
-			(width 0)
-			(type dash)
-		)
-		(fill
-			(type none)
-		)
-		(effects
-			(font
-				(size 1 1)
-			)
-			(justify left top)
