File: Power_Management.kicad_sch (KiCad schematic)
At the start: 24 parts, among them U3 SN74LVC1G07DBVR, U6 SMPS_TPS62740DSSR

Commit message: PCB Layout
Parts:
- removed EF2: EFUSE_TPS259531DSGR, Personal_Project:EFUSE_TPS259531DSGR, symbol Personal_Projects:EFUSE_TPS259531DSGR
- removed R47: 100R, Resistor_SMD:R_0603_1608Metric, symbol Device:R
- added EF1: EFUSE_TPS259531DSGR, Personal_Projects:EF_TPS259531DSGR, symbol Personal_Components:EFUSE_TPS259531DSGR
- C19, C26, C65: footprint Capacitor_SMD:C_0805_2012Metric -> Capacitor_SMD:C_0603_1608Metric
Connections:
- net +3.3VIO is gone; now on net +3.3V: C65.1, L7.2, R48.1, TP12.1, U6.5 (VOUT)
- net DVDT_1: now also EF1.1 (DVDT)
- net EN/UVLO_1: now also EF1.2 (EN/UVLO)
- net GND: now also EF1.8 (GND), EF1.9 (GND__1)
- net ILM: now also EF1.7 (ILM)
- net PWR+_EF: now also EF1.5 (OUT)
- net PWR+_PP: now also EF1.3 (IN), EF1.4 (IN__1)
- net ~{FLT}: now also EF1.6 (~{FLT})
- net SW: now reaches L7.1, U6.2 (SW)
Other:
- moved on the sheet: R50

Commit message: Power domain update
Parts:
- removed R48: 100R, Resistor_SMD:R_0603_1608Metric, symbol Device:R
Connections:
- net *RST renamed BFR_RST
- net BFR_RST: no longer U6.7 (PG)
- new net TPS62740_PG: U6.7 (PG)
Other:
- moved on the sheet: C34, U3
