File: Notes.kicad_sch (KiCad schematic)
At the start: 0 parts

Commit message: PCB Layout
Other:
- note added: "CONTROL LOGIC V1 V2 V3 RF2(LP) RF3(HP) RF4(IN) 0 0 1 ON OFF OFF 0 1 0 OFF ON OFF 0 1 1 OFF OFF ON"
- note added: "NX3L1T3157GM RF Ouputs S OUT CCT HIGH Y1 LP LOW Y0 HP"
- note added: "NX3L1T3157GM RFVCTRL Ouputs S OUT CCT HIGH Y1 LP LOW Y0 HP"
