File: STM32WL55CCU6_RF.kicad_sch (KiCad schematic)
At the start: 43 parts, among them IC2 RF_Switch_PE42440MLBB-Z, IC4 STM32WL55CCU6, J10 SMA PCB END LAUNCH JACK ROUND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, SW2 Switch_NX3L1T3157GMZ

Commit message: PCB Layout
Parts:
- removed C74, C76, C80: 10p, Capacitor_SMD:C_0805_2012Metric, symbol Device:C
- removed C75, C77, C81: 1n, Capacitor_SMD:C_0805_2012Metric, symbol Device:C
- removed IC2: RF_Switch_PE42440MLBB-Z, Personal_Project:RF_SWITCH_PE42440_QFN50P300X300X80-17N, symbol Personal_Projects:RF_Switch_PE42440MLBB-Z
- removed R1: 100R, Resistor_SMD:R_0805_2012Metric, symbol Device:R
- added C46: 100p, Capacitor_SMD:C_0603_1608Metric, symbol Device:C
- added C47, C73: 100n, Capacitor_SMD:C_0603_1608Metric, symbol Device:C
- added R3, R7: 1k2, Resistor_SMD:R_0603_1608Metric, symbol Device:R
- added U2: RFSW2_SKY13414-485LF, Personal_Project:RFSW2_SKY13414-485LF, symbol Personal_Components:RFSW2_SKY13414-485LF
- C10, C11, C12, C13, C15, C18, C20, C21, C22, C4, C40, C41, C42, C43, C5, C51, C6, C78, C79, C8: footprint Capacitor_SMD:C_0603_1608Metric_Pad1.08x0.95mm_HandSolder -> Capacitor_SMD:C_0603_1608Metric
- J10: MANUFACTURER (none) -> Wurth Elektronik; Manufacturer Wurth Elektronik -> (none)
- L12, L13, L19, L20, L21, L22, L23, L8: footprint Inductor_SMD:L_0603_1608Metric_Pad1.05x0.95mm_HandSolder -> Inductor_SMD:L_0603_1608Metric
- R2, R8: value 100R -> 1k; footprint Resistor_SMD:R_0805_2012Metric -> Resistor_SMD:R_0603_1608Metric
- renumbered IC4 to IC1
Connections:
- net +3.3V: now also C46.1, C47.1, C73.1, U2.4 (VDD)
- net GND: now also C46.2, C47.2, C73.2, R3.1, R7.1, U2.15 (GND), U2.7 (V1)
- net RF1: now also U2.10 (RF4)
- net RF1_1: now also U2.2 (RF3)
- net RF2_1: now also U2.9 (RF2)
- net PA5_INOUTRF renamed SKY13414_V3_R
- net SKY13414_V3_R: now also R3.2, U2.5 (V3)
- net PA7_HPLP_CTRL renamed NX3L1T3_RF_S
- net NX3L1T3_RF_S: no longer R8.1
- net RFIN renamed ANT
- net ANT: now also U2.13 (ANT)
- net V1 renamed SKY13414_V2
- net V2 renamed SKY13414_V3
- new net SKY13414_V2_R: R7.2, R8.1, U2.6 (V2)
Other:
- note added: "NX3L1T3157GM RF Ouputs S OUT CCT HIGH Y1 LP LOW Y0 HP"
- note removed: "NX3L1T3157GM,115 Ouputs S OUT CCT HIGH Y1 LP(Y0) LOW Y0 HP(Y1)"
- note removed: "RF_Switch_PE42440MLBB-Z V1 (PA7_HPLP_CTRL) V2 (PA5_INOUTRF) OUTPUT CCT 0 0 RFC - RF1 (PIN13) HP 1 0 RFC - RF2 (PIN15) NC 0 1 RFC - RF3 (PIN8) RFIN 1 1 RFC - RF4 (PIN6) LP"
- moved on the sheet: C51, C79, L23, R2, R8
