File: STM32WL55CCU6_GPIO.kicad_sch (KiCad schematic)
At the start: 15 parts, among them IC1 STM32WL55CCU6, J3 BOOT_JPR

Commit message: PCB Layout
Parts:
- removed C69: TBD, Capacitor_SMD:C_0805_2012Metric, symbol Device:C
- removed J3: BOOT_JPR, symbol Connector_Generic:Conn_01x02
- added J13: BOOT0_J, symbol Connector_Generic:Conn_02x03_Odd_Even
- added U16: (no value), Personal_Project:Button_SKSCLCE010, symbol Personal_Projects:BTN_SKSCLCE010
- C25, C28, C29, C31, C35, C71: footprint Capacitor_SMD:C_0805_2012Metric -> Capacitor_SMD:C_0603_1608Metric
- OS3: footprint Personal_Project:Oscillator_ECS327MVATX3CNTR -> Crystal:Crystal_SMD_3225-4Pin_3.2x2.5mm
- OS4: footprint Personal_Project:Oscillator_ECSTXO32CSMV320ANTR -> Crystal:Crystal_SMD_3225-4Pin_3.2x2.5mm
- R13, R4: footprint Resistor_SMD:R_0805_2012Metric -> Resistor_SMD:R_0603_1608Metric
Connections:
- net +3.3V: now also U16.3, U16.4
- net BOOT0: now also J13.2 (Pin_2), J13.4 (Pin_4), J13.6 (Pin_6)
- net BOOT0J: now also J13.5 (Pin_5), U16.1, U16.2
- net OSC_IN_1: now reaches C31.1, R13.2
- net OSC_IN_2: now reaches OS4.3 (OUTPUT), R13.1
- new net BOOT0_EXTCTR: J13.3 (Pin_3)
- new net BOOT0_GPIO: J13.1 (Pin_1)
Other:
- note removed: "OPTIONAL"
- moved on the sheet: C25, C28, C29, C31, C35, C71, FB5, IC1A, OS3, OS4, R13, R32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

Commit message: Power domain update
Parts:
- J13: footprint (none) -> Connector_PinHeader_2.54mm:PinHeader_2x03_P2.54mm_Vertical
Connections:
- net PA10_SPI2_MOSI: now also IC1.33 (PA10); no longer IC1.36 (PA13)
- net PA11_DEBUG_RF-NRESET: now also IC1.34 (PA11); no longer IC1.35 (PA12)
- net PA12_DEBUG_RF-BUSY: now also IC1.35 (PA12); no longer IC1.34 (PA11)
- net PA13_DEBUG_JTMS-SWDIO: now also IC1.36 (PA13); no longer IC1.33 (PA10)
Changed lines of the file:
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@@
-		)
-	)
-	(label "PA10_SPI2_MOSI"
-		(at 74.93 77.47 0)
-		(effects
-			(font
-				(size 1.27 1.27)
-			)
-			(justify left bottom)
 		)
 	)
@@
 		)
 	)
+	(label "PA13_DEBUG_JTMS-SWDIO"
+		(at 74.93 77.47 0)
+		(effects
+			(font
+				(size 1.27 1.27)
+			)
+			(justify left bottom)
+		)
+	)
+	(label "PA12_DEBUG_RF-BUSY"
+		(at 74.93 80.01 0)
+		(effects
+			(font
+				(size 1.27 1.27)
+			)
+			(justify left bottom)
+		)
+	)
 	(label "BOOT0"
 		(at 100.33 121.92 0)
@@
 		)
 	)
-	(label "PA12_DEBUG_RF-BUSY"
-		(at 74.93 82.55 0)
-		(effects
-			(font
-				(size 1.27 1.27)
-			)
-			(justify left bottom)
-		)
-	)
 	(label "NRST"
 		(at 156.21 120.65 180)
@@
 		)
 	)
+	(label "PA10_SPI2_MOSI"
+		(at 74.93 85.09 0)
+		(effects
+			(font
+				(size 1.27 1.27)
+			)
+			(justify left bottom)
+		)
+	)
 	(label "PH1-OSC_OUT"
 		(at 166.37 86.36 180)
@@
 	)
 	(label "PA11_DEBUG_RF-NRESET"
-		(at 74.93 80.01 0)
+		(at 74.93 82.55 0)
 		(effects
 			(font
@@
 		)
 	)
-	(label "PA13_DEBUG_JTMS-SWDIO"
-		(at 74.93 85.09 0)
-		(effects
-			(font
-				(size 1.27 1.27)
-			)
-			(justify left bottom)
-		)
-	)
 	(label "PA14_DEBUG_JTCK-SWCLK"
 		(at 74.93 87.63 0)
@@
 		)
 	)
+	(hierarchical_label "PA12_DEBUG_RF-BUSY"
+		(shape input)
+		(at 74.93 80.01 180)
+		(effects
+			(font
+				(size 1.27 1.27)
+			)
+			(justify right)
+		)
+	)
 	(hierarchical_label "PB12_SPI2_NSS"
 		(shape input)
@@
 		)
 	)
+	(hierarchical_label "PA11_DEBUG_RF-NRESET"
+		(shape input)
+		(at 74.93 82.55 180)
+		(effects
+			(font
+				(size 1.27 1.27)
+			)
+			(justify right)
+		)
+	)
 	(hierarchical_label "BOOT0_EXTCTR"
 		(shape input)
@@
 		)
 	)
-	(hierarchical_label "PA13_DEBUG_JTMS-SWDIO"
-		(shape input)
-		(at 74.93 85.09 180)
-		(effects
-			(font
-				(size 1.27 1.27)
-			)
-			(justify right)
-		)
-	)
 	(hierarchical_label "PA6"
 		(shape input)
@@
 		(shape input)
 		(at 74.93 52.07 180)
-		(effects
-			(font
-				(size 1.27 1.27)
-			)
-			(justify right)
-		)
-	)
-	(hierarchical_label "PA11_DEBUG_RF-NRESET"
-		(shape input)
-		(at 74.93 80.01 180)
 		(effects
 			(font
@@
 		)
 	)
+	(hierarchical_label "PA10_SPI2_MOSI"
+		(shape input)
+		(at 74.93 85.09 180)
+		(effects
+			(font
+				(size 1.27 1.27)
+			)
+			(justify right)
+		)
+	)
 	(hierarchical_label "PB7_I2C1_SDA"
 		(shape input)
@@
 		(shape input)
 		(at 74.93 57.15 180)
-		(effects
-			(font
-				(size 1.27 1.27)
-			)
-			(justify right)
-		)
-	)
-	(hierarchical_label "PA12_DEBUG_RF-BUSY"
-		(shape input)
-		(at 74.93 82.55 180)
 		(effects
 			(font
@@
 		)
 	)
+	(hierarchical_label "PA13_DEBUG_JTMS-SWDIO"
+		(shape input)
+		(at 74.93 77.47 180)
+		(effects
+			(font
+				(size 1.27 1.27)
+			)
+			(justify right)
+		)
+	)
 	(hierarchical_label "BOOT0_GPIO"
 		(shape input)
 		(at 57.15 116.84 180)
-		(effects
-			(font
-				(size 1.27 1.27)
-			)
-			(justify right)
-		)
-	)
-	(hierarchical_label "PA10_SPI2_MOSI"
-		(shape input)
-		(at 74.93 77.47 180)
 		(effects
 			(font
@@
 			)
 		)
-		(property "Footprint" ""
+		(property "Footprint" "Connector_PinHeader_2.54mm:PinHeader_2x03_P2.54mm_Vertical"
 			(at 87.63 119.38 0)
 			(hide yes)
