File: STM32WL55CCU6_PWR.kicad_sch (KiCad schematic)
At the start: 16 parts, among them IC3 STM32WL55CCU6, SW3 Switch_NX3L1T3157GMZ

Commit message: PCB Layout
Parts:
- added C74: 100n, Capacitor_SMD:C_0603_1608Metric, symbol Device:C
- C27, C30, C32, C72: footprint Capacitor_SMD:C_0805_2012Metric -> Capacitor_SMD:C_0603_1608Metric
- L3: footprint Inductor_SMD:L_0805_2012Metric_Pad1.15x1.40mm_HandSolder -> Inductor_SMD:L_0805_2012Metric
- renumbered IC3 to IC1
Connections:
- net +3.3V: now also C74.1
- net GND: now also C74.2
- net VDDA: now reaches C17.1, C36.1, FB6.1, IC1.41 (VDDA)
- net PB2_RFVCTRL renamed NX3L1T3_RFVCTRL_S
Other:
- note added: "NX3L1T3157GM RFVCTRL Ouputs S OUT CCT HIGH Y1 LP LOW Y0 HP"
- note removed: "CTRL LOGIC CTRL1=LOW, CTRL2=LOW VDDPA=VDDSMPS, RF_HP, ANT=RF_HP CTRL1=HIGH, CTRL2=LOW VDDPA=FBSMPS, RF_LP, ANT=RFI (RF3) CTRL1=HIGH, CTRL2=HIGH VDDPA=FBSMPS, RF_LP, ANT=RF_LP(RF4)"
- moved on the sheet: C16, C17, C23, C27, C30, C32, C36, C37, C57, C7, C70, C72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

Commit message: Power domain update
Changed lines of the file:
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@@
-	(wire
-		(pts
-			(xy 81.3562 19.1262) (xy 0.0762 19.1262)
-		)
-		(stroke
-			(width 0)
-			(type default)
-		)
-	)
 	(wire
 		(pts
@@
 	(wire
 		(pts
-			(xy 0.0762 19.1262) (xy 0.0762 0.0762)
-		)
-		(stroke
-			(width 0)
-			(type default)
-		)
-	)
-	(wire
-		(pts
 			(xy 69.85 83.82) (xy 90.17 83.82)
 		)
@@
 		(pts
 			(xy 182.88 100.33) (xy 182.88 102.87)
-		)
-		(stroke
-			(width 0)
-			(type default)
-		)
-	)
-	(wire
-		(pts
-			(xy 0.0762 0.0762) (xy 8.9662 0.0762)
 		)
 		(stroke
@@
 		)
 	)
-	(label "VDDSMPS"
-		(at 181.61 67.31 180)
-		(effects
-			(font
-				(size 1.27 1.27)
-			)
-			(justify right bottom)
-		)
-	)
